File: electronics/airsuspension_MCU.sch (KiCad schematic (older format))
At the start: 1 part, among them U10 Teensy3.1

Commit message: more footprints...
Parts:
- U10: farnell (none) -> 2430007; name (none) -> Teensy3.1
Changed lines of the file:
@@
 F 0 "U10" H 4900 5300 60  0000 C CNN
 F 1 "Teensy3.1" H 6100 5300 60  0000 C CNN
-F 2 "" H 5600 3400 60  0000 C CNN
-F 3 "" H 5600 3400 60  0000 C CNN
+F 2 "" H 5600 3400 60  0001 C CNN
+F 3 "https://www.pjrc.com/teensy/pinout.html" H 5600 3400 60  0001 C CNN
+F 4 "Teensy3.1" H 5450 3250 60  0001 C CNN "name"
+F 5 "2430007" H 5450 3250 60  0001 C CNN "farnell"
 	1    5450 3250
 	1    0    0    -1
 $EndComp
 $Comp
-L GND #PWR059
+L GND #PWR56
 U 1 1 550B9984
 P 4000 1300
-F 0 "#PWR059" H 4000 1050 60  0001 C CNN
+F 0 "#PWR56" H 4000 1050 60  0001 C CNN
 F 1 "GND" H 4000 1150 60  0000 C CNN
 F 2 "" H 4000 1300 60  0000 C CNN
@@
 +3.3V
 $Comp
-L GND #PWR060
+L GND #PWR57
 U 1 1 550B99C1
 P 7300 1550
-F 0 "#PWR060" H 7300 1300 60  0001 C CNN
+F 0 "#PWR57" H 7300 1300 60  0001 C CNN
 F 1 "GND" H 7300 1400 60  0000 C CNN
 F 2 "" H 7300 1550 60  0000 C CNN
@@
 RightSuck_ON
 $Comp
-L GND #PWR061
+L GND #PWR55
 U 1 1 550CFA12
 P 3400 4200
-F 0 "#PWR061" H 3400 3950 60  0001 C CNN
+F 0 "#PWR55" H 3400 3950 60  0001 C CNN
 F 1 "GND" H 3400 4050 60  0000 C CNN
 F 2 "" H 3400 4200 60  0000 C CNN
