File: electronics/airsuspension_outputs.sch (KiCad schematic (older format))
At the start: 51 parts, among them Q1 BSS138, Q2 BC847, U1 ITS5215L, U2 BTS6133D, U3 ITS5215L, U4 ITS5215L, U5 ITS5215L

Commit message: more footprints...
Parts:
- D1, D10, D11, D3, D6, D7, D8, D9: footprint LED-0805 -> LEDs:LED-0805
- Q1, Q2: footprint SOT-23 -> Housings_SOT-23_SOT-143_TSOT-6:SOT-23
- U1: farnell (none) -> 1426197; name (none) -> ITS5215L
- U2: footprint (none) -> SMD_Packages:DPAK-5
- U3, U4, U5: farnell (none) -> 1426197
