File: electronics/airsuspension_CAN.sch (KiCad schematic (older format))
At the start: 5 parts, among them U8 SN65HVD1050D

Commit message: Some more fottprints added to PCB
Parts:
- C17: footprint (none) -> Capacitors_SMD:C_0805; farnell (none) -> 1288261; name (none) -> C0805C224K5RACTU
- JP1: footprint (none) -> Oddities:NetTie-I_Connected_SMD
- JP2: footprint (none) -> Oddities:NetTie-I_SMD
- U8: footprint (none) -> Housings_SOIC:SOIC-8_3.9x4.9mm_Pitch1.27mm; farnell (none) -> 1220984; name (none) -> SN65HVD1050D
Changed lines of the file:
@@
 F 0 "U8" H 5350 3450 60  0000 C CNN
 F 1 "SN65HVD1050D" H 5300 2700 60  0000 C CNN
-F 2 "" H 5400 2950 60  0001 C CNN
-F 3 "" H 5400 2950 60  0000 C CNN
+F 2 "Housings_SOIC:SOIC-8_3.9x4.9mm_Pitch1.27mm" H 5400 2950 60  0001 C CNN
+F 3 "http://www.farnell.com/datasheets/1804905.pdf" H 5400 2950 60  0001 C CNN
+F 4 "1220984" H 5300 3100 60  0001 C CNN "farnell"
+F 5 "SN65HVD1050D" H 5300 3100 60  0001 C CNN "name"
 	1    5300 3100
 	1    0    0    -1
@@
 F 0 "C17" H 4400 3650 50  0000 L CNN
 F 1 "220nF" H 4400 3450 50  0000 L CNN
-F 2 "" H 4388 3400 30  0001 C CNN
+F 2 "Capacitors_SMD:C_0805" H 4388 3400 30  0001 C CNN
 F 3 "" H 4350 3550 60  0000 C CNN
+F 4 "1288261" H 4350 3550 60  0001 C CNN "farnell"
+F 5 "C0805C224K5RACTU" H 4350 3550 60  0001 C CNN "name"
 	1    4350 3550
 	1    0    0    -1
@@
 F 0 "JP2" H 6600 2600 50  0000 C CNN
 F 1 "CAN_Silent" H 6600 2370 50  0000 C CNN
-F 2 "" H 6600 2450 60  0001 C CNN
+F 2 "Oddities:NetTie-I_SMD" H 6600 2450 60  0001 C CNN
 F 3 "" H 6600 2450 60  0000 C CNN
 	1    6600 2450
@@
 F 0 "JP1" H 6000 2600 50  0000 C CNN
 F 1 "CAN_fullspeed" H 6000 2370 50  0000 C CNN
-F 2 "" H 6000 2450 60  0001 C CNN
+F 2 "Oddities:NetTie-I_Connected_SMD" H 6000 2450 60  0001 C CNN
 F 3 "" H 6000 2450 60  0000 C CNN
 	1    6000 2450

Commit message: some fottprints and BOM changes
Parts:
- R53: farnell (none) -> 2303452; name (none) -> ERJ6ENF1200V
Changed lines of the file:
@@
 F 2 "" V 6530 3150 30  0001 C CNN
 F 3 "" H 6600 3150 30  0000 C CNN
+F 4 "2303452" V 6600 3150 60  0001 C CNN "farnell"
+F 5 "ERJ6ENF1200V" V 6600 3150 60  0001 C CNN "name"
 	1    6600 3150
 	1    0    0    -1

Commit message: Some more footprints and beginning PCB work
Parts:
- R53: footprint (none) -> Resistors_SMD:R_0805_HandSoldering
Changed lines of the file:
@@
 F 0 "R53" V 6680 3150 50  0000 C CNN
 F 1 "120R" V 6607 3151 50  0000 C CNN
-F 2 "" V 6530 3150 30  0001 C CNN
-F 3 "" H 6600 3150 30  0000 C CNN
+F 2 "Resistors_SMD:R_0805_HandSoldering" V 6530 3150 30  0001 C CNN
+F 3 "http://www.farnell.com/datasheets/1678782.pdf" H 6600 3150 30  0001 C CNN
 F 4 "2303452" V 6600 3150 60  0001 C CNN "farnell"
 F 5 "ERJ6ENF1200V" V 6600 3150 60  0001 C CNN "name"

Commit message: Changed to a more stable powersupply (3Amps 5V and separate 3.3v) + some few cleanups due to updated kicad
Parts:
- removed JP1: CAN_fullspeed, Oddities:NetTie-I_Connected_SMD, symbol JUMPER
- added R?: 10k, Resistors_SMD:R_0805_HandSoldering, symbol R
Connections:
- net +5V: now also C17.1
- net CAN_HI: now also R53.1
- net CAN_LO: now also R53.2
- net GND: now also C17.2, R?.2
- net at JP2.1, U8.8 (S): now also R?.1
Other:
- note added: "Normal operation should see CAN_fullspeed (LOW)\nCAN_Silent mode is lowpower mode, should be open by default"
- note removed: "Normal operation should see CAN_fullspeed bridged\nCAN_Silent mode is lowpower mode, should be open by default"
Changed lines of the file:
@@
 EESchema Schematic File Version 2
+LIBS:airsuspension_controller-rescue
 LIBS:power
 LIBS:device
@@
 LIBS:memory
 LIBS:xilinx
-LIBS:special
 LIBS:microcontrollers
 LIBS:dsp
@@
 Sheet 4 6
 Title ""
-Date ""
+Date "3 aug 2015"
 Rev ""
 Comp ""
@@
 $EndComp
 $Comp
-L JUMPER JP1
-U 1 1 55069FDD
-P 6000 2450
-F 0 "JP1" H 6000 2600 50  0000 C CNN
-F 1 "CAN_fullspeed" H 6000 2370 50  0000 C CNN
-F 2 "Oddities:NetTie-I_Connected_SMD" H 6000 2450 60  0001 C CNN
-F 3 "" H 6000 2450 60  0000 C CNN
-	1    6000 2450
-	1    0    0    -1
-$EndComp
-$Comp
 L GND #PWR050
 U 1 1 5506A004
-P 5700 2500
-F 0 "#PWR050" H 5700 2250 60  0001 C CNN
-F 1 "GND" H 5700 2350 60  0000 C CNN
-F 2 "" H 5700 2500 60  0000 C CNN
-F 3 "" H 5700 2500 60  0000 C CNN
-	1    5700 2500
+P 5875 2500
+F 0 "#PWR050" H 5875 2250 60  0001 C CNN
+F 1 "GND" H 5875 2350 60  0000 C CNN
+F 2 "" H 5875 2500 60  0000 C CNN
+F 3 "" H 5875 2500 60  0000 C CNN
+	1    5875 2500
 	1    0    0    -1
 $EndComp
@@
 +5V
 Wire Wire Line
-	5800 2900 6150 2900
-Wire Wire Line
-	6150 2900 6150 2700
-Wire Wire Line
-	6150 2700 6300 2700
-Wire Wire Line
-	6300 2700 6300 2450
-Wire Wire Line
-	5700 2500 5700 2450
+	5800 2900 6200 2900
 Text Notes 4700 2000 0    60   ~ 0
-Normal operation should see CAN_fullspeed bridged\nCAN_Silent mode is lowpower mode, should be open by default
+Normal operation should see CAN_fullspeed (LOW)\nCAN_Silent mode is lowpower mode, should be open by default
 Text Notes 6850 3200 0    60   ~ 0
 Resistor is here only when Node is a end node\nThere should be exactly 2 endnodes in a CAN network\n
+Wire Wire Line
+	6600 2900 6600 3000
+Wire Wire Line
+	6600 3300 6600 3400
+Wire Wire Line
+	4350 3350 4350 3400
+Wire Wire Line
+	4350 3700 4350 3750
+$Comp
+L R R?
+U 1 1 56FA4041
+P 6025 2450
+F 0 "R?" V 5818 2450 50  0000 C CNN
+F 1 "10k" V 5909 2450 50  0000 C CNN
+F 2 "Resistors_SMD:R_0805_HandSoldering" V 5955 2450 50  0001 C CNN
+F 3 "" H 6025 2450 50  0000 C CNN
+F 4 "9332391" V 6025 2450 60  0001 C CNN "farnell"
+	1    6025 2450
+	0    1    1    0
+$EndComp
+Wire Wire Line
+	5875 2450 5875 2500
+Wire Wire Line
+	6175 2450 6300 2450
+Wire Wire Line
+	6200 2900 6200 2450
+Connection ~ 6200 2450
 $EndSCHEMATC

Commit message: First placement with a ModICE enclosure
Parts:
- gave numbers to parts that had none: 1
Changed lines of the file:
@@
 LIBS:power_switches
 LIBS:miscellaneous
+LIBS:cinch
 LIBS:airsuspension_controller-cache
 EELAYER 25 0
@@
 $EndComp
 $Comp
-L GND #PWR048
+L GND #PWR050
 U 1 1 55069D68
 P 4500 3050
-F 0 "#PWR048" H 4500 2800 60  0001 C CNN
+F 0 "#PWR050" H 4500 2800 60  0001 C CNN
 F 1 "GND" H 4500 2900 60  0000 C CNN
 F 2 "" H 4500 3050 60  0000 C CNN
@@
 $EndComp
 $Comp
-L GND #PWR049
+L GND #PWR051
 U 1 1 55069DAC
 P 4350 3750
-F 0 "#PWR049" H 4350 3500 60  0001 C CNN
+F 0 "#PWR051" H 4350 3500 60  0001 C CNN
 F 1 "GND" H 4350 3600 60  0000 C CNN
 F 2 "" H 4350 3750 60  0000 C CNN
@@
 $EndComp
 $Comp
-L GND #PWR050
+L GND #PWR052
 U 1 1 5506A004
 P 5875 2500
-F 0 "#PWR050" H 5875 2250 60  0001 C CNN
+F 0 "#PWR052" H 5875 2250 60  0001 C CNN
 F 1 "GND" H 5875 2350 60  0000 C CNN
 F 2 "" H 5875 2500 60  0000 C CNN
@@
 	4350 3700 4350 3750
 $Comp
-L R R?
+L R R55
 U 1 1 56FA4041
 P 6025 2450
-F 0 "R?" V 5818 2450 50  0000 C CNN
+F 0 "R55" V 5818 2450 50  0000 C CNN
 F 1 "10k" V 5909 2450 50  0000 C CNN
 F 2 "Resistors_SMD:R_0805_HandSoldering" V 5955 2450 50  0001 C CNN

Commit message: Some updates as some parts were not available
Parts:
- C17: name C0805C224K5RACTU -> (none); part (none) -> C0805C224K5RACTU
- JP2: farnell (none) -> (none); part (none) -> (none)
- R53: name ERJ6ENF1200V -> (none)
- U8: name SN65HVD1050D -> (none); part (none) -> SN65HVD1050D
Changed lines of the file:
@@
 F 3 "http://www.farnell.com/datasheets/1804905.pdf" H 5400 2950 60  0001 C CNN
 F 4 "1220984" H 5300 3100 60  0001 C CNN "farnell"
-F 5 "SN65HVD1050D" H 5300 3100 60  0001 C CNN "name"
+F 5 "SN65HVD1050D" H 5300 3100 60  0001 C CNN "part"
 	1    5300 3100
 	1    0    0    -1
@@
 F 3 "http://www.farnell.com/datasheets/1678782.pdf" H 6600 3150 30  0001 C CNN
 F 4 "2303452" V 6600 3150 60  0001 C CNN "farnell"
-F 5 "ERJ6ENF1200V" V 6600 3150 60  0001 C CNN "name"
 	1    6600 3150
 	1    0    0    -1
@@
 F 3 "" H 4350 3550 60  0000 C CNN
 F 4 "1288261" H 4350 3550 60  0001 C CNN "farnell"
-F 5 "C0805C224K5RACTU" H 4350 3550 60  0001 C CNN "name"
+F 5 "C0805C224K5RACTU" H 4350 3550 60  0001 C CNN "part"
 	1    4350 3550
 	1    0    0    -1
@@
 F 2 "Oddities:NetTie-I_SMD" H 6600 2450 60  0001 C CNN
 F 3 "" H 6600 2450 60  0000 C CNN
+F 4 " " H 6600 2450 60  0001 C CNN "part"
+F 5 " " H 6600 2450 60  0001 C CNN "farnell"
 	1    6600 2450
 	1    0    0    -1
