File: electronics/AirSuspension/Airsuspension_5V.sch (KiCad schematic (older format))
At the start: 28 parts, among them Q3 IPD50P04P4L-11, Q4 BC856, Q5 BC856, Q6 IPD060N03L G, U11 MC34063, U9 LD1117S33CTR

Commit message: Changed value of load sensing resistor for 5V switch do reduce system noise
Parts:
- R57: value 0.031 -> 0.1; farnell 1099911 -> 2008301; part LR1206-R033FW -> CRL1206-FW-R100ELF
- U11: symbol MC34063 -> MC34063-RESCUE-airsuspension_controller
Changed lines of the file:
@@
 $EndDescr
 $Comp
-L MC34063 U11
+L MC34063-RESCUE-airsuspension_controller U11
 U 1 1 56F98FC6
 P 5650 3725
+AR Path="/56F98FC6" Ref="U11"  Part="1"
+AR Path="/5507DD0F/56F98FC6" Ref="U11"  Part="1"
 F 0 "U11" H 5650 4292 50  0000 C CNN
 F 1 "MC34063" H 5650 4201 50  0000 C CNN
@@
 P 4850 3475
 F 0 "R57" H 4920 3521 50  0000 L CNN
-F 1 "0.031" H 4920 3430 50  0000 L CNN
+F 1 "0.1" H 4920 3430 50  0000 L CNN
 F 2 "Resistors_SMD:R_1206_HandSoldering" V 4780 3475 50  0001 C CNN
 F 3 "" H 4850 3475 50  0000 C CNN
-F 4 "1099911" H 4850 3475 60  0001 C CNN "farnell"
-F 5 "LR1206-R033FW" H 4850 3475 60  0001 C CNN "part"
+F 4 "2008301" H 4850 3475 60  0001 C CNN "farnell"
+F 5 "CRL1206-FW-R100ELF" H 4850 3475 60  0001 C CNN "part"
 	1    4850 3475
 	1    0    0    -1
