File: electronics/AirSuspension/airsuspension_controller.sch (KiCad schematic (older format))
At the start: 7 parts

Commit message: Added some documentation Schematic document
Other:
- note added: "Begins on L\nEnds on Y"
Changed lines of the file:
@@
 	1    0    0    -1
 $EndComp
+Text Notes 2700 1875 0    60   ~ 0
+Begins on L\nEnds on Y
 $EndSCHEMATC

Commit message: More fixes and chenged components eat less boardspace
Parts:
- Ha12: part 5810130028 -> 5810130029
Changed lines of the file:
@@
 F 2 "" H 775 2500 60  0000 C CNN
 F 3 "" H 775 2500 60  0000 C CNN
-F 4 "5810130028" H 775 2475 60  0001 C CNN "part"
+F 4 "5810130029" H 775 2475 60  0001 C CNN "part"
 F 5 "1282206" H 775 2475 60  0001 C CNN "farnell"
 	1    775  2475
