File: electronics/Parkbrake/Parkbrake.sch (KiCad schematic (older format))
At the start: 28 parts, among them P1 Conn48pin, Q1 BSS138, Q2 BSS138, Q3 P-ch -40V 0.0035ohm, Q4 P-ch -40V 0.0035ohm, Q5 BSS308, Q6 BSS308

Commit message: some more work on parkbrake pcb
Connections:
- net +12V_BatR: now also P1.13 (E1), P1.14 (E2), P1.15 (E3); no longer P1.1 (A1), P1.2 (A2), P1.3 (A3)
- net BrakeLights: now also P1.1 (A1); no longer P1.13 (E1)
- net LeftRearMotor+: now also P1.8 (C2), P1.9 (C3); no longer P1.11 (D2), P1.12 (D3)
- net LeftRearMotor-: now also P1.11 (D2), P1.12 (D3); no longer P1.14 (E2), P1.15 (E3)
- net ParkbrakeSwitch_non_invert: now also P1.4 (B1); no longer P1.7 (C1)
- net Parkbrake_indicator_lamp: now also P1.7 (C1); no longer P1.4 (B1)
- net RightRearMotor+: now also P1.2 (A2), P1.3 (A3); no longer P1.5 (B2), P1.6 (B3)
- net RightRearMotor-: now also P1.5 (B2), P1.6 (B3); no longer P1.8 (C2), P1.9 (C3)
Changed lines of the file:
@@
 $EndComp
 $Comp
-L GND #PWR8
+L GND #PWR01
 U 1 1 5708DE8A
 P 4750 7250
-F 0 "#PWR8" H 4750 7000 50  0001 C CNN
+F 0 "#PWR01" H 4750 7000 50  0001 C CNN
 F 1 "GND" H 4758 7077 50  0000 C CNN
 F 2 "" H 4750 7250 50  0000 C CNN
@@
 $EndComp
 $Comp
-L GNDPWR #PWR1
+L GNDPWR #PWR02
 U 1 1 57090A02
 P 1050 5775
-F 0 "#PWR1" H 1050 5575 50  0001 C CNN
+F 0 "#PWR02" H 1050 5575 50  0001 C CNN
 F 1 "GNDPWR" H 1057 5849 50  0001 C CNN
 F 2 "" H 1050 5725 50  0000 C CNN
@@
 $EndComp
 $Comp
-L GNDPWR #PWR3
+L GNDPWR #PWR03
 U 1 1 5701F17D
 P 1675 5075
-F 0 "#PWR3" H 1675 4875 50  0001 C CNN
+F 0 "#PWR03" H 1675 4875 50  0001 C CNN
 F 1 "GNDPWR" H 1682 5149 50  0001 C CNN
 F 2 "" H 1675 5025 50  0000 C CNN
@@
 $EndComp
 $Comp
-L GND #PWR9
+L GND #PWR04
 U 1 1 570200C5
 P 5375 7050
-F 0 "#PWR9" H 5375 6800 50  0001 C CNN
+F 0 "#PWR04" H 5375 6800 50  0001 C CNN
 F 1 "GND" H 5383 6877 50  0000 C CNN
 F 2 "" H 5375 7050 50  0000 C CNN
@@
 $EndComp
 $Comp
-L GNDPWR #PWR5
+L GNDPWR #PWR05
 U 1 1 570235BF
 P 2025 1075
-F 0 "#PWR5" H 2025 875 50  0001 C CNN
+F 0 "#PWR05" H 2025 875 50  0001 C CNN
 F 1 "GNDPWR" H 2032 1149 50  0000 C CNN
 F 2 "" H 2025 1025 50  0000 C CNN
@@
 Text GLabel 3100 1525 2    60   Input ~ 0
 RightFrontMotor-
+Text GLabel 3100 3375 2    60   Input ~ 0
+LeftRearMotor+
 Text GLabel 3100 3525 2    60   Input ~ 0
-LeftRearMotor+
-Text GLabel 3100 3675 2    60   Input ~ 0
 LeftRearMotor-
+Text GLabel 3100 3075 2    60   Input ~ 0
+RightRearMotor+
 Text GLabel 3100 3225 2    60   Input ~ 0
-RightRearMotor+
-Text GLabel 3100 3375 2    60   Input ~ 0
 RightRearMotor-
 Text GLabel 3125 2325 2    60   Input ~ 0
@@
 $EndSheet
 $Comp
-L GND #PWR7
+L GND #PWR06
 U 1 1 578E7EF2
-P 2075 2425
-F 0 "#PWR7" H 2075 2175 50  0001 C CNN
-F 1 "GND" H 2075 2275 50  0000 C CNN
-F 2 "" H 2075 2425 50  0000 C CNN
-F 3 "" H 2075 2425 50  0000 C CNN
-	1    2075 2425
+P 2075 2525
+F 0 "#PWR06" H 2075 2275 50  0001 C CNN
+F 1 "GND" H 2075 2375 50  0000 C CNN
+F 2 "" H 2075 2525 50  0000 C CNN
+F 3 "" H 2075 2525 50  0000 C CNN
+	1    2075 2525
 	1    0    0    -1
 $EndComp
@@
 Text GLabel 2050 2025 0    60   Input ~ 0
 RR_wheelsensor_in+
+Text GLabel 2025 3375 0    60   Input ~ 0
+Parkbrake_indicator_lamp
+Text GLabel 2025 3075 0    60   Input ~ 0
+BrakeLights
 Text GLabel 2025 3225 0    60   Input ~ 0
-Parkbrake_indicator_lamp
-Text GLabel 2025 3675 0    60   Input ~ 0
-BrakeLights
-Text GLabel 2025 3375 0    60   Input ~ 0
 ParkbrakeSwitch_non_invert
 Text GLabel 2025 3525 0    60   Input ~ 0
@@
 L_wheelsensor_out+
 $Comp
-L PWR_FLAG #FLG1
+L PWR_FLAG #FLG07
 U 1 1 578EA974
 P 1150 4575
-F 0 "#FLG1" H 1150 4670 50  0001 C CNN
+F 0 "#FLG07" H 1150 4670 50  0001 C CNN
 F 1 "PWR_FLAG" H 1150 4755 50  0000 C CNN
 F 2 "" H 1150 4575 50  0000 C CNN
@@
 $EndComp
 $Comp
-L PWR_FLAG #FLG8
+L PWR_FLAG #FLG08
 U 1 1 578EAB0E
 P 4425 6550
-F 0 "#FLG8" H 4425 6645 50  0001 C CNN
+F 0 "#FLG08" H 4425 6645 50  0001 C CNN
 F 1 "PWR_FLAG" H 4425 6730 50  0001 C CNN
 F 2 "" H 4425 6550 50  0000 C CNN
@@
 $EndComp
 $Comp
-L PWR_FLAG #FLG10
+L PWR_FLAG #FLG09
 U 1 1 578EAB3C
 P 5375 7050
-F 0 "#FLG10" H 5375 7145 50  0001 C CNN
+F 0 "#FLG09" H 5375 7145 50  0001 C CNN
 F 1 "PWR_FLAG" H 5375 7250 50  0001 C CNN
 F 2 "" H 5375 7050 50  0000 C CNN
 F 3 "" H 5375 7050 50  0000 C CNN
 	1    5375 7050
-	0    1    1    0
-$EndComp
-$Comp
-L PWR_FLAG #FLG4
-U 1 1 578EAC6F
-P 1675 5075
-F 0 "#FLG4" H 1675 5170 50  0001 C CNN
-F 1 "PWR_FLAG" H 1700 5275 50  0001 C CNN
-F 2 "" H 1675 5075 50  0000 C CNN
-F 3 "" H 1675 5075 50  0000 C CNN
-	1    1675 5075
 	0    1    1    0
 $EndComp
@@
 ParkbrakeSwitch_non_invert
 $Comp
-L PWR_FLAG #FLG7
+L PWR_FLAG #FLG010
 U 1 1 578F074A
 P 4425 6125
-F 0 "#FLG7" H 4425 6220 50  0001 C CNN
+F 0 "#FLG010" H 4425 6220 50  0001 C CNN
 F 1 "PWR_FLAG" H 4425 6305 50  0001 C CNN
 F 2 "" H 4425 6125 50  0000 C CNN
@@
 $EndComp
 $Comp
-L PWR_FLAG #FLG9
+L PWR_FLAG #FLG011
 U 1 1 5797B077
 P 5375 6550
-F 0 "#FLG9" H 5375 6645 50  0001 C CNN
+F 0 "#FLG011" H 5375 6645 50  0001 C CNN
 F 1 "PWR_FLAG" H 5375 6750 50  0001 C CNN
 F 2 "" H 5375 6550 50  0000 C CNN
@@
 $EndComp
 $Comp
-L PWR_FLAG #FLG3
+L PWR_FLAG #FLG012
 U 1 1 579735F3
 P 1675 4575
-F 0 "#FLG3" H 1675 4670 50  0001 C CNN
+F 0 "#FLG012" H 1675 4670 50  0001 C CNN
 F 1 "PWR_FLAG" H 1700 4775 50  0001 C CNN
 F 2 "" H 1675 4575 50  0000 C CNN
@@
 $EndComp
 $Comp
-L GNDPWR #PWR6
+L GNDPWR #PWR013
 U 1 1 579818E3
 P 2025 3825
-F 0 "#PWR6" H 2025 3625 50  0001 C CNN
+F 0 "#PWR013" H 2025 3625 50  0001 C CNN
 F 1 "GNDPWR" H 2025 3700 50  0000 C CNN
 F 2 "" H 2025 3775 50  0000 C CNN
@@
 	1    0    0    -1
 $EndComp
-Text Label 3100 3075 0    60   ~ 0
+Text Label 3100 3675 0    60   ~ 0
 +12V_BatR
 Wire Wire Line
@@
 Wire Wire Line
 	2250 3525 2025 3525
-Wire Wire Line
-	2500 3375 3100 3375
 Connection ~ 2750 3375
 Wire Wire Line
@@
 Wire Wire Line
 	2500 3225 3100 3225
-Wire Wire Line
-	2250 3075 3100 3075
 Connection ~ 2500 3825
 Connection ~ 2750 3225
 Connection ~ 2750 3075
-Wire Wire Line
-	2250 3375 2025 3375
 Wire Wire Line
 	2250 3225 2025 3225
@@
 $EndComp
 $Comp
-L GNDPWR #PWR2
+L GNDPWR #PWR014
 U 1 1 5798E6D1
 P 1050 7575
-F 0 "#PWR2" H 1050 7375 50  0001 C CNN
+F 0 "#PWR014" H 1050 7375 50  0001 C CNN
 F 1 "GNDPWR" H 1057 7649 50  0001 C CNN
 F 2 "" H 1050 7525 50  0000 C CNN
@@
 $EndComp
 $Comp
-L GNDPWR #PWR4
+L GNDPWR #PWR015
 U 1 1 5798E6F2
 P 1675 6875
-F 0 "#PWR4" H 1675 6675 50  0001 C CNN
+F 0 "#PWR015" H 1675 6675 50  0001 C CNN
 F 1 "GNDPWR" H 1682 6949 50  0001 C CNN
 F 2 "" H 1675 6825 50  0000 C CNN
@@
 Batt switch off and polarity protection
 $Comp
-L PWR_FLAG #FLG2
+L PWR_FLAG #FLG016
 U 1 1 5798E6F9
 P 1150 6375
-F 0 "#FLG2" H 1150 6470 50  0001 C CNN
+F 0 "#FLG016" H 1150 6470 50  0001 C CNN
 F 1 "PWR_FLAG" H 1150 6555 50  0000 C CNN
 F 2 "" H 1150 6375 50  0000 C CNN
@@
 $EndComp
 $Comp
-L PWR_FLAG #FLG6
+L PWR_FLAG #FLG017
 U 1 1 5798E6FF
 P 1675 6875
-F 0 "#FLG6" H 1675 6970 50  0001 C CNN
+F 0 "#FLG017" H 1675 6970 50  0001 C CNN
 F 1 "PWR_FLAG" H 1700 7075 50  0001 C CNN
 F 2 "" H 1675 6875 50  0000 C CNN
@@
 $EndComp
 $Comp
-L PWR_FLAG #FLG5
+L PWR_FLAG #FLG018
 U 1 1 5798E705
 P 1675 6375
-F 0 "#FLG5" H 1675 6470 50  0001 C CNN
+F 0 "#FLG018" H 1675 6470 50  0001 C CNN
 F 1 "PWR_FLAG" H 1700 6575 50  0001 C CNN
 F 2 "" H 1675 6375 50  0000 C CNN
@@
 Connection ~ 1350 6775
 Wire Wire Line
-	2500 3675 3100 3675
+	2250 3675 3100 3675
 Connection ~ 2750 3675
 Wire Wire Line
-	2250 3675 2025 3675
-Connection ~ 2500 3075
+	2500 3375 3100 3375
+Wire Wire Line
+	2250 3375 2025 3375
+Wire Wire Line
+	2500 3075 3100 3075
+Connection ~ 2500 3675
+Wire Wire Line
+	2250 3075 2025 3075
+Wire Wire Line
+	2075 2425 2075 2525
+Text GLabel 2050 2525 0    60   Input ~ 0
+SensorGND
+Wire Wire Line
+	2075 2525 2050 2525
 $EndSCHEMATC
