File: electronics/Parkbrake/H-Bridge_logic.sch (KiCad schematic (older format))
At the start: 29 parts

Commit message: Add currentlimit latching to avaoid current limit oscilation Start a mcu schema part
Parts:
- removed U? (x9): 74LS11, symbol 74LS11
- added U? (x8): 74LV08D, symbol 74LS08
- added U? (x4): CD74HC03M, symbol 7400
- U? (x4): value 74LS00 -> CD74HC03M
Connections:
- net labels added: LeftFront_Loosen, LeftRear_Loosen, RightFront_Loosen, RightRear_Loosen, ~LeftFront_CL, ~LeftFront_Reset, ~LeftRear_CL, ~LeftRear_Reset, ~RightFront_CL, ~RightFront_Reset, ~RightRear_CL, ~RightRear_Reset
- net labels removed: LeftFront_Enable, LeftRear_Enable, RightFront_Enable, RightRear_Enable
- wire segments 87 -> 118
- no-connect marks 1 -> 0
Other:
- note added: "~SR~ latch tripped by overcurrent, must be reset by software\nCurrentLimit triggers the SR latch, the xx_DIAG is the output \nof this latch, is high when the latch has triggered."
- moved on the sheet: U?A, U?B, U?C, U?D

Commit message: More work on parkbrake node
Parts:
- R? (x4): footprint (none) -> Resistors_SMD:R_0805; farnell (none) -> 9332383; part (none) -> MC01W080511K
Connections:
- net ~LeftRear_Reset is gone; now on net Bridge_Disable: U?.5
- net ~RightFront_Reset is gone; now on net Bridge_Disable: U?.12
- net ~RightRear_Reset is gone; now on net Bridge_Disable: U?.12
- net ~LeftFront_Reset renamed Bridge_Disable
Changed lines of the file:
@@
 LIBS:teensy
 LIBS:power_switches
+LIBS:stm32
 LIBS:Parkbrake-cache
 EELAYER 25 0
@@
 $Descr A4 11693 8268
 encoding utf-8
-Sheet 2 6
+Sheet 2 10
 Title ""
 Date ""
@@
 F 0 "R?" V 1457 1900 50  0000 C CNN
 F 1 "1k" V 1366 1900 50  0000 C CNN
-F 2 "" V 1180 1900 50  0000 C CNN
+F 2 "Resistors_SMD:R_0805" V 1180 1900 50  0001 C CNN
 F 3 "" H 1250 1900 50  0000 C CNN
+F 4 "9332383" V 1250 1900 60  0001 C CNN "farnell"
+F 5 "MC01W080511K" V 1250 1900 60  0001 C CNN "part"
 	1    1250 1900
 	0    -1   -1   0
@@
 F 0 "R?" V 1043 2850 50  0000 C CNN
 F 1 "1k" V 1134 2850 50  0000 C CNN
-F 2 "" V 1180 2850 50  0000 C CNN
+F 2 "Resistors_SMD:R_0805" V 1180 2850 50  0001 C CNN
 F 3 "" H 1250 2850 50  0000 C CNN
+F 4 "9332383" V 1250 2850 60  0001 C CNN "farnell"
+F 5 "MC01W080511K" V 1250 2850 60  0001 C CNN "part"
 	1    1250 2850
 	0    1    1    0
@@
 F 0 "R?" V 3293 2850 50  0000 C CNN
 F 1 "1k" V 3384 2850 50  0000 C CNN
-F 2 "" V 3430 2850 50  0000 C CNN
+F 2 "Resistors_SMD:R_0805" V 3430 2850 50  0001 C CNN
 F 3 "" H 3500 2850 50  0000 C CNN
+F 4 "9332383" V 3500 2850 60  0001 C CNN "farnell"
+F 5 "MC01W080511K" V 3500 2850 60  0001 C CNN "part"
 	1    3500 2850
 	0    1    1    0
@@
 F 0 "R?" V 3268 1900 50  0000 C CNN
 F 1 "1k" V 3359 1900 50  0000 C CNN
-F 2 "" V 3405 1900 50  0000 C CNN
+F 2 "Resistors_SMD:R_0805" V 3405 1900 50  0001 C CNN
 F 3 "" H 3475 1900 50  0000 C CNN
+F 4 "9332383" V 3475 1900 60  0001 C CNN "farnell"
+F 5 "MC01W080511K" V 3475 1900 60  0001 C CNN "part"
 	1    3475 1900
 	0    1    1    0
@@
 $EndComp
 Text GLabel 1375 5525 0    60   Input ~ 0
-~LeftFront_Reset
+Bridge_Disable
 Text Notes 7900 4225 0    60   ~ 0
 ~SR~ latch tripped by overcurrent, must be reset by software\nCurrentLimit triggers the SR latch, the xx_DIAG is the output \nof this latch, is high when the latch has triggered.
@@
 	3050 5350 2900 5350
 Wire Wire Line
-	2900 5350 2900 5775
-Wire Wire Line
-	2900 5775 2900 5950
+	2900 5350 2900 5950
 Wire Wire Line
 	2900 5775 3050 5775
@@
 	2900 4875 3050 4875
 Wire Wire Line
-	2900 4275 2900 4425
-Wire Wire Line
-	2900 4425 2900 4875
+	2900 4275 2900 4875
 Wire Wire Line
 	4800 5350 4925 5350
 Wire Wire Line
-	4925 5350 4925 5775
-Wire Wire Line
-	4925 5775 4925 5950
+	4925 5350 4925 5950
 Wire Wire Line
 	4925 5775 4800 5775
 Wire Wire Line
-	4925 4275 4925 4400
-Wire Wire Line
-	4925 4400 4925 4875
+	4925 4275 4925 4875
 Wire Wire Line
 	4925 4875 4800 4875
@@
 	4925 4400 4800 4400
 Wire Wire Line
-	9000 1475 9000 1650
-Wire Wire Line
-	9000 1650 9000 2075
+	9000 1475 9000 2075
 Wire Wire Line
 	9000 2075 8900 2075
@@
 	9000 1650 8900 1650
 Wire Wire Line
-	9000 2550 9000 2950
-Wire Wire Line
-	9000 2950 9000 3150
+	9000 2550 9000 3150
 Wire Wire Line
 	9000 2950 8900 2950
@@
 	9000 2550 8900 2550
 Wire Wire Line
-	6875 2550 6875 2950
-Wire Wire Line
-	6875 2950 6875 3150
+	6875 2550 6875 3150
 Wire Wire Line
 	6875 2950 7000 2950
@@
 	7000 2550 6875 2550
 Wire Wire Line
-	6875 1450 6875 1650
-Wire Wire Line
-	6875 1650 6875 2075
+	6875 1450 6875 2075
 Wire Wire Line
 	6875 2075 7000 2075
@@
 	7000 1650 6875 1650
 Wire Wire Line
-	1350 900  1425 900
-Wire Wire Line
-	1425 900  1900 900
-Wire Wire Line
-	1900 900  2275 900
-Wire Wire Line
-	2275 900  2700 900
-Wire Wire Line
-	2700 900  2825 900
+	1350 900  2825 900
 Connection ~ 1425 900
 Wire Wire Line
-	1425 1200 1900 1200
-Wire Wire Line
-	1900 1200 2275 1200
-Wire Wire Line
-	2275 1200 2700 1200
-Wire Wire Line
-	2700 1200 2850 1200
+	1425 1200 2850 1200
 Connection ~ 1900 900
 Connection ~ 2275 900
@@
 Connection ~ 2700 1200
 Wire Wire Line
-	3300 1800 3300 1900
-Wire Wire Line
-	3300 1900 3300 2025
+	3300 1800 3300 2025
 Wire Wire Line
 	3325 1900 3300 1900
 Connection ~ 3300 1900
 Wire Wire Line
-	2900 1800 2900 1900
-Wire Wire Line
-	2900 1900 2900 2025
+	2900 1800 2900 2025
 Wire Wire Line
 	2900 1900 2700 1900
 Connection ~ 2900 1900
 Wire Wire Line
-	1425 2725 1425 2850
-Wire Wire Line
-	1425 2850 1425 2950
+	1425 2725 1425 2950
 Wire Wire Line
 	1400 2850 1425 2850
 Connection ~ 1425 2850
 Wire Wire Line
-	1825 2725 1825 2850
-Wire Wire Line
-	1825 2850 1825 2950
+	1825 2725 1825 2950
 Wire Wire Line
 	1825 2850 1950 2850
 Connection ~ 1825 2850
 Wire Wire Line
-	1825 1800 1825 1900
-Wire Wire Line
-	1825 1900 1825 2025
+	1825 1800 1825 2025
 Wire Wire Line
 	1825 1900 1950 1900
 Connection ~ 1825 1900
 Wire Wire Line
-	1425 1800 1425 1900
-Wire Wire Line
-	1425 1900 1425 2025
+	1425 1800 1425 2025
 Wire Wire Line
 	1425 1900 1400 1900
 Connection ~ 1425 1900
 Wire Wire Line
-	3325 2725 3325 2850
-Wire Wire Line
-	3325 2850 3325 2950
+	3325 2725 3325 2950
 Wire Wire Line
 	3350 2850 3325 2850
 Connection ~ 3325 2850
 Wire Wire Line
-	2925 2725 2925 2850
-Wire Wire Line
-	2925 2850 2925 2950
+	2925 2725 2925 2950
 Wire Wire Line
 	2925 2850 2700 2850
@@
 	1375 5175 1375 5325
 Wire Wire Line
-	1375 5325 1375 5325
-Wire Wire Line
 	1375 4875 1375 5050
 Wire Wire Line
 	1375 5050 2675 5050
 Wire Wire Line
-	2675 4525 2675 5050
-Wire Wire Line
-	2675 5050 2675 5425
-Wire Wire Line
-	2675 5425 2675 5700
+	2675 4525 2675 5700
 Wire Wire Line
 	2675 5425 2575 5425
@@
 	6500 5075 5175 5075
 Wire Wire Line
-	5175 4525 5175 5075
-Wire Wire Line
-	5175 5075 5175 5400
-Wire Wire Line
-	5175 5400 5175 5700
+	5175 4525 5175 5700
 Wire Wire Line
 	5175 5400 5300 5400
@@
 Connection ~ 5175 5075
 Text GLabel 6500 5500 2    60   Input ~ 0
-~RightFront_Reset
+Bridge_Disable
 $Comp
 L 74LS08 U?
@@
 	5400 2275 6725 2275
 Wire Wire Line
-	6725 1700 6725 2275
-Wire Wire Line
-	6725 2275 6725 2600
-Wire Wire Line
-	6725 2600 6725 2900
+	6725 1700 6725 2900
 Wire Wire Line
 	6725 2600 6600 2600
@@
 Connection ~ 6875 1650
 Text GLabel 5400 2700 0    60   Input ~ 0
-~LeftRear_Reset
+Bridge_Disable
 Wire Wire Line
 	9175 2025 9175 2350
@@
 	10375 2275 9100 2275
 Wire Wire Line
-	9100 1750 9100 2275
-Wire Wire Line
-	9100 2275 9100 2600
-Wire Wire Line
-	9100 2600 9100 2900
+	9100 1750 9100 2900
 Wire Wire Line
 	9100 2600 9175 2600
@@
 Connection ~ 9000 1650
 Text GLabel 10375 2700 2    60   Input ~ 0
-~RightRear_Reset
+Bridge_Disable
 Text GLabel 1375 5175 0    60   Input ~ 0
 LeftFront_DIAG

Commit message: ordernr, type and footprints for all components
Parts:
- C? (x4): footprint (none) -> Capacitors_SMD:C_0805; farnell (none) -> 2496940; part (none) -> 0805B104J500CT
- D? (x4): footprint (none) -> LEDs:LED_0805; farnell (none) -> 2463991; part (none) -> KP-2012LSGC
- D? (x4): footprint (none) -> LEDs:LED_0805; farnell (none) -> 1318244; part (none) -> KP-2012SRC-PRV
Changed lines of the file:
@@
 F 0 "C?" H 1540 1096 50  0000 L CNN
 F 1 "100n" H 1550 1025 50  0000 L CNN
-F 2 "" H 1463 900 50  0000 C CNN
+F 2 "Capacitors_SMD:C_0805" H 1463 900 50  0001 C CNN
 F 3 "" H 1425 1050 50  0000 C CNN
+F 4 "0805B104J500CT" H 1425 1050 60  0001 C CNN "part"
+F 5 "2496940" H 1425 1050 60  0001 C CNN "farnell"
 	1    1425 1050
 	1    0    0    -1
@@
 F 0 "C?" H 2015 1096 50  0000 L CNN
 F 1 "100n" H 2015 1005 50  0000 L CNN
-F 2 "" H 1938 900 50  0000 C CNN
+F 2 "Capacitors_SMD:C_0805" H 1938 900 50  0001 C CNN
 F 3 "" H 1900 1050 50  0000 C CNN
+F 4 "0805B104J500CT" H 1900 1050 60  0001 C CNN "part"
+F 5 "2496940" H 1900 1050 60  0001 C CNN "farnell"
 	1    1900 1050
 	1    0    0    -1
@@
 F 0 "C?" H 2390 1096 50  0000 L CNN
 F 1 "100n" H 2390 1005 50  0000 L CNN
-F 2 "" H 2313 900 50  0000 C CNN
+F 2 "Capacitors_SMD:C_0805" H 2313 900 50  0001 C CNN
 F 3 "" H 2275 1050 50  0000 C CNN
+F 4 "0805B104J500CT" H 2275 1050 60  0001 C CNN "part"
+F 5 "2496940" H 2275 1050 60  0001 C CNN "farnell"
 	1    2275 1050
 	1    0    0    -1
@@
 F 0 "C?" H 2815 1096 50  0000 L CNN
 F 1 "100n" H 2825 1025 50  0000 L CNN
-F 2 "" H 2738 900 50  0000 C CNN
+F 2 "Capacitors_SMD:C_0805" H 2738 900 50  0001 C CNN
 F 3 "" H 2700 1050 50  0000 C CNN
+F 4 "0805B104J500CT" H 2700 1050 60  0001 C CNN "part"
+F 5 "2496940" H 2700 1050 60  0001 C CNN "farnell"
 	1    2700 1050
 	1    0    0    -1
@@
 F 0 "D?" H 1625 2015 50  0000 C CNN
 F 1 "LF_Release" H 1625 1924 50  0000 C CNN
-F 2 "" H 1625 1800 50  0000 C CNN
+F 2 "LEDs:LED_0805" H 1625 1800 50  0001 C CNN
 F 3 "" H 1625 1800 50  0000 C CNN
+F 4 "KP-2012LSGC" H 1625 1800 60  0001 C CNN "part"
+F 5 "2463991" H 1625 1800 60  0001 C CNN "farnell"
 	1    1625 1800
 	1    0    0    -1
@@
 F 0 "D?" H 1625 2225 50  0000 C CNN
 F 1 "LF_Tighten" H 1625 2150 50  0000 C CNN
-F 2 "" H 1625 2025 50  0000 C CNN
+F 2 "LEDs:LED_0805" H 1625 2025 50  0001 C CNN
 F 3 "" H 1625 2025 50  0000 C CNN
+F 4 "KP-2012SRC-PRV" H 1625 2025 60  0001 C CNN "part"
+F 5 "1318244" H 1625 2025 60  0001 C CNN "farnell"
 	1    1625 2025
 	-1   0    0    1
@@
 F 0 "D?" H 1625 2940 50  0000 C CNN
 F 1 "LR_Release" H 1625 2849 50  0000 C CNN
-F 2 "" H 1625 2725 50  0000 C CNN
+F 2 "LEDs:LED_0805" H 1625 2725 50  0001 C CNN
 F 3 "" H 1625 2725 50  0000 C CNN
+F 4 "KP-2012LSGC" H 1625 2725 60  0001 C CNN "part"
+F 5 "2463991" H 1625 2725 60  0001 C CNN "farnell"
 	1    1625 2725
 	1    0    0    -1
@@
 F 0 "D?" H 1625 3150 50  0000 C CNN
 F 1 "LR_Tighten" H 1625 3075 50  0000 C CNN
-F 2 "" H 1625 2950 50  0000 C CNN
+F 2 "LEDs:LED_0805" H 1625 2950 50  0001 C CNN
 F 3 "" H 1625 2950 50  0000 C CNN
+F 4 "KP-2012SRC-PRV" H 1625 2950 60  0001 C CNN "part"
+F 5 "1318244" H 1625 2950 60  0001 C CNN "farnell"
 	1    1625 2950
 	-1   0    0    1
@@
 F 0 "D?" H 3100 2015 50  0000 C CNN
 F 1 "RF_Release" H 3100 1924 50  0000 C CNN
-F 2 "" H 3100 1800 50  0000 C CNN
+F 2 "LEDs:LED_0805" H 3100 1800 50  0001 C CNN
 F 3 "" H 3100 1800 50  0000 C CNN
+F 4 "KP-2012LSGC" H 3100 1800 60  0001 C CNN "part"
+F 5 "2463991" H 3100 1800 60  0001 C CNN "farnell"
 	1    3100 1800
 	1    0    0    -1
@@
 F 0 "D?" H 3100 2225 50  0000 C CNN
 F 1 "RF_tighten" H 3100 2150 50  0000 C CNN
-F 2 "" H 3100 2025 50  0000 C CNN
+F 2 "LEDs:LED_0805" H 3100 2025 50  0001 C CNN
 F 3 "" H 3100 2025 50  0000 C CNN
+F 4 "KP-2012SRC-PRV" H 3100 2025 60  0001 C CNN "part"
+F 5 "1318244" H 3100 2025 60  0001 C CNN "farnell"
 	1    3100 2025
 	-1   0    0    1
@@
 F 0 "D?" H 3125 2940 50  0000 C CNN
 F 1 "RR_Release" H 3125 2849 50  0000 C CNN
-F 2 "" H 3125 2725 50  0000 C CNN
+F 2 "LEDs:LED_0805" H 3125 2725 50  0001 C CNN
 F 3 "" H 3125 2725 50  0000 C CNN
+F 4 "KP-2012LSGC" H 3125 2725 60  0001 C CNN "part"
+F 5 "2463991" H 3125 2725 60  0001 C CNN "farnell"
 	1    3125 2725
 	1    0    0    -1
@@
 F 0 "D?" H 3125 3150 50  0000 C CNN
 F 1 "RR_Tighten" H 3125 3075 50  0000 C CNN
-F 2 "" H 3125 2950 50  0000 C CNN
+F 2 "LEDs:LED_0805" H 3125 2950 50  0001 C CNN
 F 3 "" H 3125 2950 50  0000 C CNN
+F 4 "KP-2012SRC-PRV" H 3125 2950 60  0001 C CNN "part"
+F 5 "1318244" H 3125 2950 60  0001 C CNN "farnell"
 	1    3125 2950
 	-1   0    0    1

Commit message: Make it pass DRC rule check
Parts:
- gave numbers to parts that had none: 20
Changed lines of the file:
@@
 $EndDescr
 $Comp
-L 74LS00 U?
+L 74LS00 U1
 U 1 1 5704D186
 P 1975 4775
-F 0 "U?" H 1875 4875 50  0000 L CNN
+F 0 "U1" H 1875 4875 50  0000 L CNN
 F 1 "CD74HC03M" H 1750 4750 50  0000 L CNN
 F 2 "" H 1975 4775 50  0000 C CNN
@@
 $EndComp
 $Comp
-L 74LS00 U?
+L 74LS00 U1
 U 2 1 570532D4
 P 1975 5425
-F 0 "U?" H 1875 5525 50  0000 L CNN
+F 0 "U1" H 1875 5525 50  0000 L CNN
 F 1 "CD74HC03M" H 1750 5400 50  0000 L CNN
 F 2 "" H 1975 5425 50  0000 C CNN
@@
 $EndSheet
 $Comp
-L 74LS00 U?
+L 74LS00 U1
 U 3 1 570625EF
 P 5900 4825
-F 0 "U?" H 5850 4725 50  0000 L CNN
+F 0 "U1" H 5850 4725 50  0000 L CNN
 F 1 "CD74HC03M" H 5675 4875 50  0000 L CNN
 F 2 "" H 5900 4825 50  0000 C CNN
@@
 $EndComp
 $Comp
-L 74LS00 U?
+L 74LS00 U1
 U 4 1 5706623B
 P 5900 5400
-F 0 "U?" H 5850 5300 50  0000 L CNN
+F 0 "U1" H 5850 5300 50  0000 L CNN
 F 1 "CD74HC03M" H 5675 5450 50  0000 L CNN
 F 2 "" H 5900 5400 50  0000 C CNN
@@
 $EndComp
 $Comp
-L C C?
+L C C1
 U 1 1 5706DC6B
 P 1425 1050
-F 0 "C?" H 1540 1096 50  0000 L CNN
+F 0 "C1" H 1540 1096 50  0000 L CNN
 F 1 "100n" H 1550 1025 50  0000 L CNN
 F 2 "Capacitors_SMD:C_0805" H 1463 900 50  0001 C CNN
@@
 $EndComp
 $Comp
-L GND #PWR?
+L GND #PWR015
 U 1 1 5706E47E
 P 1425 1200
-F 0 "#PWR?" H 1425 950 50  0001 C CNN
+F 0 "#PWR015" H 1425 950 50  0001 C CNN
 F 1 "GND" H 1433 1027 50  0000 C CNN
 F 2 "" H 1425 1200 50  0000 C CNN
@@
 $EndSheet
 $Comp
-L C C?
+L C C2
 U 1 1 5707D112
 P 1900 1050
-F 0 "C?" H 2015 1096 50  0000 L CNN
+F 0 "C2" H 2015 1096 50  0000 L CNN
 F 1 "100n" H 2015 1005 50  0000 L CNN
 F 2 "Capacitors_SMD:C_0805" H 1938 900 50  0001 C CNN
@@
 $EndComp
 $Comp
-L C C?
+L C C3
 U 1 1 5707D1B4
 P 2275 1050
-F 0 "C?" H 2390 1096 50  0000 L CNN
+F 0 "C3" H 2390 1096 50  0000 L CNN
 F 1 "100n" H 2390 1005 50  0000 L CNN
 F 2 "Capacitors_SMD:C_0805" H 2313 900 50  0001 C CNN
@@
 $EndComp
 $Comp
-L C C?
+L C C4
 U 1 1 5707D256
 P 2700 1050
-F 0 "C?" H 2815 1096 50  0000 L CNN
+F 0 "C4" H 2815 1096 50  0000 L CNN
 F 1 "100n" H 2825 1025 50  0000 L CNN
 F 2 "Capacitors_SMD:C_0805" H 2738 900 50  0001 C CNN
@@
 $EndComp
 $Comp
-L LED D?
+L LED D4
 U 1 1 5707E22E
 P 1625 1800
-F 0 "D?" H 1625 2015 50  0000 C CNN
+F 0 "D4" H 1625 2015 50  0000 C CNN
 F 1 "LF_Release" H 1625 1924 50  0000 C CNN
 F 2 "LEDs:LED_0805" H 1625 1800 50  0001 C CNN
@@
 $EndComp
 $Comp
-L LED D?
+L LED D5
 U 1 1 5707E3F8
 P 1625 2025
-F 0 "D?" H 1625 2225 50  0000 C CNN
+F 0 "D5" H 1625 2225 50  0000 C CNN
 F 1 "LF_Tighten" H 1625 2150 50  0000 C CNN
 F 2 "LEDs:LED_0805" H 1625 2025 50  0001 C CNN
@@
 $EndComp
 $Comp
-L LED D?
+L LED D6
 U 1 1 5707E530
 P 1625 2725
-F 0 "D?" H 1625 2940 50  0000 C CNN
+F 0 "D6" H 1625 2940 50  0000 C CNN
 F 1 "LR_Release" H 1625 2849 50  0000 C CNN
 F 2 "LEDs:LED_0805" H 1625 2725 50  0001 C CNN
@@
 $EndComp
 $Comp
-L LED D?
+L LED D7
 U 1 1 5707E5E6
 P 1625 2950
-F 0 "D?" H 1625 3150 50  0000 C CNN
+F 0 "D7" H 1625 3150 50  0000 C CNN
 F 1 "LR_Tighten" H 1625 3075 50  0000 C CNN
 F 2 "LEDs:LED_0805" H 1625 2950 50  0001 C CNN
@@
 $EndComp
 $Comp
-L LED D?
+L LED D8
 U 1 1 5707E904
 P 3100 1800
-F 0 "D?" H 3100 2015 50  0000 C CNN
+F 0 "D8" H 3100 2015 50  0000 C CNN
 F 1 "RF_Release" H 3100 1924 50  0000 C CNN
 F 2 "LEDs:LED_0805" H 3100 1800 50  0001 C CNN
@@
 $EndComp
 $Comp
-L LED D?
+L LED D9
 U 1 1 5707E9DA
 P 3100 2025
-F 0 "D?" H 3100 2225 50  0000 C CNN
+F 0 "D9" H 3100 2225 50  0000 C CNN
 F 1 "RF_tighten" H 3100 2150 50  0000 C CNN
 F 2 "LEDs:LED_0805" H 3100 2025 50  0001 C CNN
@@
 $EndComp
 $Comp
-L LED D?
+L LED D10
 U 1 1 5707EB22
 P 3125 2725
-F 0 "D?" H 3125 2940 50  0000 C CNN
+F 0 "D10" H 3125 2940 50  0000 C CNN
 F 1 "RR_Release" H 3125 2849 50  0000 C CNN
 F 2 "LEDs:LED_0805" H 3125 2725 50  0001 C CNN
@@
 $EndComp
 $Comp
-L LED D?
+L LED D11
 U 1 1 5707EBD0
 P 3125 2950
-F 0 "D?" H 3125 3150 50  0000 C CNN
+F 0 "D11" H 3125 3150 50  0000 C CNN
 F 1 "RR_Tighten" H 3125 3075 50  0000 C CNN
 F 2 "LEDs:LED_0805" H 3125 2950 50  0001 C CNN
@@
 $EndComp
 $Comp
-L R R?
+L R R5
 U 1 1 5707ED69
 P 1250 1900
-F 0 "R?" V 1457 1900 50  0000 C CNN
+F 0 "R5" V 1457 1900 50  0000 C CNN
 F 1 "1k" V 1366 1900 50  0000 C CNN
 F 2 "Resistors_SMD:R_0805" V 1180 1900 50  0001 C CNN
@@
 $EndComp
 $Comp
-L R R?
+L R R6
 U 1 1 5707EF24
 P 1250 2850
-F 0 "R?" V 1043 2850 50  0000 C CNN
+F 0 "R6" V 1043 2850 50  0000 C CNN
 F 1 "1k" V 1134 2850 50  0000 C CNN
 F 2 "Resistors_SMD:R_0805" V 1180 2850 50  0001 C CNN
@@
 $EndComp
 $Comp
-L R R?
+L R R8
 U 1 1 5707F028
 P 3500 2850
-F 0 "R?" V 3293 2850 50  0000 C CNN
+F 0 "R8" V 3293 2850 50  0000 C CNN
 F 1 "1k" V 3384 2850 50  0000 C CNN
 F 2 "Resistors_SMD:R_0805" V 3430 2850 50  0001 C CNN
@@
 $EndComp
 $Comp
-L R R?
+L R R7
 U 1 1 5707F12F
 P 3475 1900
-F 0 "R?" V 3268 1900 50  0000 C CNN
+F 0 "R7" V 3268 1900 50  0000 C CNN
 F 1 "1k" V 3359 1900 50  0000 C CNN
 F 2 "Resistors_SMD:R_0805" V 3405 1900 50  0001 C CNN
@@
 RightRear_Tighten
 $Comp
-L 74LS08 U?
+L 74LS08 U2
 U 1 1 57135EB3
 P 2300 4275
-F 0 "U?" H 2275 4400 50  0000 C CNN
+F 0 "U2" H 2275 4400 50  0000 C CNN
 F 1 "74LV08D" H 2325 4275 50  0000 C CNN
 F 2 "" H 2300 4275 50  0000 C CNN
@@
 $EndComp
 $Comp
-L 74LS08 U?
+L 74LS08 U2
 U 2 1 5713618B
 P 2300 5950
-F 0 "U?" H 2300 6050 50  0000 C CNN
+F 0 "U2" H 2300 6050 50  0000 C CNN
 F 1 "74LV08D" H 2300 5925 50  0000 C CNN
 F 2 "" H 2300 5950 50  0000 C CNN
@@
 ~SR~ latch tripped by overcurrent, must be reset by software\nCurrentLimit triggers the SR latch, the xx_DIAG is the output \nof this latch, is high when the latch has triggered.
 $Comp
-L 74LS08 U?
+L 74LS08 U2
 U 3 1 5713C42D
 P 5525 4275
-F 0 "U?" H 5500 4175 50  0000 C CNN
+F 0 "U2" H 5500 4175 50  0000 C CNN
 F 1 "74LV08D" H 5500 4300 50  0000 C CNN
 F 2 "" H 5525 4275 50  0000 C CNN
@@
 $EndComp
 $Comp
-L 74LS08 U?
+L 74LS08 U2
 U 4 1 5713C5B9
 P 5525 5950
-F 0 "U?" H 5475 5825 50  0000 C CNN
+F 0 "U2" H 5475 5825 50  0000 C CNN
 F 1 "74LV08D" H 5475 5925 50  0000 C CNN
 F 2 "" H 5525 5950 50  0000 C CNN
@@
 Bridge_Disable
 $Comp
-L 74LS08 U?
+L 74LS08 U4
 U 1 1 5713F73F
 P 6275 1450
-F 0 "U?" H 6275 1600 50  0000 C CNN
+F 0 "U4" H 6275 1600 50  0000 C CNN
 F 1 "74LV08D" H 6250 1450 50  0000 C CNN
 F 2 "" H 6275 1450 50  0000 C CNN
@@
 $EndComp
 $Comp
-L 74LS08 U?
+L 74LS08 U4
 U 2 1 5713F923
 P 6275 3150
-F 0 "U?" H 6225 3275 50  0000 C CNN
+F 0 "U4" H 6225 3275 50  0000 C CNN
 F 1 "74LV08D" H 6200 3150 50  0000 C CNN
 F 2 "" H 6275 3150 50  0000 C CNN
@@
 $EndComp
 $Comp
-L 74LS08 U?
+L 74LS08 U4
 U 3 1 5713F9E5
 P 9600 1475
-F 0 "U?" H 9600 1350 50  0000 C CNN
+F 0 "U4" H 9600 1350 50  0000 C CNN
 F 1 "74LV08D" H 9625 1475 50  0000 C CNN
 F 2 "" H 9600 1475 50  0000 C CNN
@@
 $EndComp
 $Comp
-L 74LS08 U?
+L 74LS08 U4
 U 4 1 5713FB8D
 P 9600 3150
-F 0 "U?" H 9575 3025 50  0000 C CNN
+F 0 "U4" H 9575 3025 50  0000 C CNN
 F 1 "74LV08D" H 9575 3150 50  0000 C CNN
 F 2 "" H 9600 3150 50  0000 C CNN
@@
 $EndComp
 $Comp
-L 7400 U?
+L 7400 U3
 U 1 1 57141A30
 P 6000 2025
-F 0 "U?" H 5975 2150 50  0000 C CNN
+F 0 "U3" H 5975 2150 50  0000 C CNN
 F 1 "CD74HC03M" H 5975 2000 50  0000 C CNN
 F 2 "" H 6000 2025 50  0000 C CNN
@@
 $EndComp
 $Comp
-L 7400 U?
+L 7400 U3
 U 2 1 57141B42
 P 6000 2600
-F 0 "U?" H 5975 2725 50  0000 C CNN
+F 0 "U3" H 5975 2725 50  0000 C CNN
 F 1 "CD74HC03M" H 5975 2550 50  0000 C CNN
 F 2 "" H 6000 2600 50  0000 C CNN
@@
 $EndComp
 $Comp
-L 7400 U?
+L 7400 U3
 U 3 1 57141D9A
 P 9775 2025
-F 0 "U?" H 9750 1900 50  0000 C CNN
+F 0 "U3" H 9750 1900 50  0000 C CNN
 F 1 "CD74HC03M" H 9775 2025 50  0000 C CNN
 F 2 "" H 9775 2025 50  0000 C CNN
@@
 $EndComp
 $Comp
-L 7400 U?
+L 7400 U3
 U 4 1 57141F56
 P 9775 2600
-F 0 "U?" H 9750 2475 50  0000 C CNN
+F 0 "U3" H 9750 2475 50  0000 C CNN
 F 1 "CD74HC03M" H 9775 2625 50  0000 C CNN
 F 2 "" H 9775 2600 50  0000 C CNN
