File: electronics/Parkbrake/PowerRegulators.sch (KiCad schematic (older format))
At the start: 23 parts

Commit message: More work on parkbrake node
Parts:
- C?: farnell 2326228 -> 2507731; part EEEHAC681UAP -> EEEFK1E681SP
- D? (x2): footprint (none) -> Diodes_SMD:DO-214AB; farnell (none) -> 2353680; part (none) -> STPS3L40S
- L?: footprint (none) -> Inductors:Inductor_1212; farnell (none) -> 9522204; part (none) -> LQH32CN100K33L
- L?: value 17uH -> 33uH; footprint (none) -> Inductors:SELF-WE-PD-XXL; farnell (none) -> 2374128; part (none) -> SRR1260A-330M
- R? (x2): footprint (none) -> Resistors_SMD:R_0805; farnell (none) -> 9332839; part (none) -> MC01W08051220K
- R?: footprint (none) -> Resistors_SMD:R_0805; farnell (none) -> 9332502; part (none) -> MC01W0805112K
- R?: footprint (none) -> Resistors_SMD:R_0805; part (none) -> 9332391
- R?: footprint (none) -> Resistors_SMD:R_0805; farnell (none) -> 9332383; part (none) -> MC01W080511K
- R?: footprint (none) -> Resistors_SMD:R_0805; farnell (none) -> 9332995; part (none) -> MC01W080513K
- R?: value 0.073 -> 0.150 1/2W; footprint (none) -> Resistors_SMD:R_1206; farnell (none) -> 2503066; part (none) -> WW12PR150FTL
- U?: footprint (none) -> TO_SOT_Packages_SMD:SOT-23-6; farnell (none) -> 2509963; part (none) -> MIC2619YD6-TR
- U?: symbol MC34063 -> MC34063-RESCUE-Parkbrake
- U?: footprint SOT-223 -> TO_SOT_Packages_SMD:SOT-223; farnell (none) -> 1467779; part (none) -> LD1117S33CTR
Changed lines of the file:
@@
 LIBS:teensy
 LIBS:power_switches
+LIBS:stm32
 LIBS:Parkbrake-cache
 EELAYER 25 0
@@
 $Descr A4 11693 8268
 encoding utf-8
-Sheet 5 6
+Sheet 5 10
 Title ""
 Date ""
@@
 F 0 "U?" H 2125 6587 60  0000 C CNN
 F 1 "MIC2619" H 2125 6481 60  0000 C CNN
-F 2 "" H 2125 6150 60  0000 C CNN
+F 2 "TO_SOT_Packages_SMD:SOT-23-6" H 2125 6150 60  0001 C CNN
 F 3 "" H 2125 6150 60  0000 C CNN
+F 4 "MIC2619YD6-TR" H 2125 6150 60  0001 C CNN "part"
+F 5 "2509963" H 2125 6150 60  0001 C CNN "farnell"
 	1    2125 6150
 	1    0    0    -1
@@
 F 0 "L?" H 2125 5765 50  0000 C CNN
 F 1 "10uH" H 2125 5674 50  0000 C CNN
-F 2 "" H 2125 5550 50  0000 C CNN
+F 2 "Inductors:Inductor_1212" H 2125 5550 50  0001 C CNN
 F 3 "" H 2125 5550 50  0000 C CNN
+F 4 "LQH32CN100K33L" H 2125 5550 60  0001 C CNN "part"
+F 5 "9522204" H 2125 5550 60  0001 C CNN "farnell"
 	1    2125 5550
 	1    0    0    -1
@@
 F 0 "D?" H 2775 5795 50  0000 C CNN
 F 1 "40V 1A" H 2775 5886 50  0000 C CNN
-F 2 "" V 2775 6000 50  0000 C CNN
+F 2 "Diodes_SMD:DO-214AB" V 2775 6000 50  0001 C CNN
 F 3 "" V 2775 6000 50  0000 C CNN
+F 4 "STPS3L40S" H 2775 6000 60  0001 C CNN "part"
+F 5 "2353680" H 2775 6000 60  0001 C CNN "farnell"
 	1    2775 6000
 	-1   0    0    1
@@
 F 0 "R?" H 3145 6196 50  0000 L CNN
 F 1 "220k" H 3145 6105 50  0000 L CNN
-F 2 "" V 3005 6150 50  0000 C CNN
+F 2 "Resistors_SMD:R_0805" V 3005 6150 50  0001 C CNN
 F 3 "" H 3075 6150 50  0000 C CNN
+F 4 "MC01W08051220K" H 3075 6150 60  0001 C CNN "part"
+F 5 "9332839" H 3075 6150 60  0001 C CNN "farnell"
 	1    3075 6150
 	1    0    0    -1
@@
 F 0 "R?" H 3145 6571 50  0000 L CNN
 F 1 "12k" H 3145 6480 50  0000 L CNN
-F 2 "" V 3005 6525 50  0000 C CNN
+F 2 "Resistors_SMD:R_0805" V 3005 6525 50  0001 C CNN
 F 3 "" H 3075 6525 50  0000 C CNN
+F 4 "MC01W0805112K" H 3075 6525 60  0001 C CNN "part"
+F 5 "9332502" H 3075 6525 60  0001 C CNN "farnell"
 	1    3075 6525
 	1    0    0    -1
@@
 F 0 "R?" H 3420 6196 50  0000 L CNN
 F 1 "220k" H 3420 6105 50  0000 L CNN
-F 2 "" V 3280 6150 50  0000 C CNN
+F 2 "Resistors_SMD:R_0805" V 3280 6150 50  0001 C CNN
 F 3 "" H 3350 6150 50  0000 C CNN
+F 4 "MC01W08051220K" H 3350 6150 60  0001 C CNN "part"
+F 5 "9332839" H 3350 6150 60  0001 C CNN "farnell"
 	1    3350 6150
 	1    0    0    -1
@@
 F 0 "R?" H 3420 6571 50  0000 L CNN
 F 1 "10k" H 3420 6480 50  0000 L CNN
-F 2 "" V 3280 6525 50  0000 C CNN
+F 2 "Resistors_SMD:R_0805" V 3280 6525 50  0001 C CNN
 F 3 "" H 3350 6525 50  0000 C CNN
+F 4 "MC01W0805110K" H 3350 6525 60  0001 C CNN "part"
+F 5 "9332391" H 3350 6525 60  0001 C CNN "part"
 	1    3350 6525
 	1    0    0    -1
@@
 gate_drive_24V
 $Comp
-L MC34063 U?
+L MC34063-RESCUE-Parkbrake U?
 U 1 1 57089F7E
 P 3675 2425
+AR Path="/57089F7E" Ref="U?"  Part="1"
+AR Path="/57088F10/57089F7E" Ref="U?"  Part="1"
 F 0 "U?" H 3675 2992 50  0000 C CNN
 F 1 "MC34063" H 3675 2901 50  0000 C CNN
@@
 F 0 "R?" H 4145 3046 50  0000 L CNN
 F 1 "1k" H 4145 2955 50  0000 L CNN
-F 2 "" V 4005 3000 50  0000 C CNN
+F 2 "Resistors_SMD:R_0805" V 4005 3000 50  0001 C CNN
 F 3 "" H 4075 3000 50  0000 C CNN
+F 4 "MC01W080511K" H 4075 3000 60  0001 C CNN "part"
+F 5 "9332383" H 4075 3000 60  0001 C CNN "farnell"
 	1    4075 3000
 	1    0    0    -1
@@
 F 0 "R?" V 4550 2725 50  0000 C CNN
 F 1 "3k" V 4625 2725 50  0000 C CNN
-F 2 "" V 4555 2725 50  0000 C CNN
+F 2 "Resistors_SMD:R_0805" V 4555 2725 50  0001 C CNN
 F 3 "" H 4625 2725 50  0000 C CNN
+F 4 "MC01W080513K" V 4625 2725 60  0001 C CNN "part"
+F 5 "9332995" V 4625 2725 60  0001 C CNN "farnell"
 	1    4625 2725
 	0    1    1    0
@@
 P 2975 2175
 F 0 "R?" H 3045 2221 50  0000 L CNN
-F 1 "0.073" H 3045 2130 50  0000 L CNN
-F 2 "" V 2905 2175 50  0000 C CNN
+F 1 "0.150 1/2W" V 2875 2125 50  0000 L CNN
+F 2 "Resistors_SMD:R_1206" V 2905 2175 50  0001 C CNN
 F 3 "" H 2975 2175 50  0000 C CNN
+F 4 "WW12PR150FTL" H 2975 2175 60  0001 C CNN "part"
+F 5 "2503066" H 2975 2175 60  0001 C CNN "farnell"
 	1    2975 2175
 	1    0    0    -1
@@
 P 4600 2525
 F 0 "L?" H 4600 2740 50  0000 C CNN
-F 1 "17uH" H 4600 2649 50  0000 C CNN
-F 2 "" H 4600 2525 50  0000 C CNN
+F 1 "33uH" H 4600 2649 50  0000 C CNN
+F 2 "Inductors:SELF-WE-PD-XXL" H 4600 2525 50  0001 C CNN
 F 3 "" H 4600 2525 50  0000 C CNN
+F 4 "SRR1260A-330M" H 4600 2525 60  0001 C CNN "part"
+F 5 "2374128" H 4600 2525 60  0001 C CNN "farnell"
 	1    4600 2525
 	1    0    0    -1
@@
 F 0 "D?" V 4304 3079 50  0000 L CNN
 F 1 "D_Schottky" V 4395 3079 50  0000 L CNN
-F 2 "" H 4350 3000 50  0000 C CNN
+F 2 "Diodes_SMD:DO-214AB" H 4350 3000 50  0001 C CNN
 F 3 "" H 4350 3000 50  0000 C CNN
+F 4 "STPS3L40S" V 4350 3000 60  0001 C CNN "part"
+F 5 "2353680" V 4350 3000 60  0001 C CNN "farnell"
 	1    4350 3000
 	0    1    1    0
@@
 F 2 "Capacitors_SMD:c_elec_10x10.5" H 5113 2525 50  0001 C CNN
 F 3 "" H 5075 2675 50  0000 C CNN
-F 4 "EEEHAC681UAP" H 5075 2675 60  0001 C CNN "part"
-F 5 "2326228" H 5075 2675 60  0001 C CNN "farnell"
+F 4 "EEEFK1E681SP" H 5075 2675 60  0001 C CNN "part"
+F 5 "2507731" H 5075 2675 60  0001 C CNN "farnell"
 	1    5075 2675
 	1    0    0    -1
@@
 F 0 "U?" H 8450 2758 50  0000 C CNN
 F 1 "LD1117S33CTR" H 8450 2667 50  0000 C CNN
-F 2 "SOT-223" H 8450 2576 50  0000 C CNN
+F 2 "TO_SOT_Packages_SMD:SOT-223" H 8450 2576 50  0001 C CNN
 F 3 "" H 8450 2350 50  0000 C CNN
+F 4 "LD1117S33CTR" H 8450 2350 60  0001 C CNN "part"
+F 5 "1467779" H 8450 2350 60  0001 C CNN "farnell"
 	1    8450 2350
 	1    0    0    -1

Commit message: ordernr, type and footprints for all components
Parts:
- C?: footprint (none) -> Capacitors_SMD:C_1206; farnell (none) -> 2362126; part (none) -> GRM31MR71E105JA01L
- C? (x3): footprint (none) -> Capacitors_SMD:c_elec_5x5.3; symbol C -> CP; farnell (none) -> 1870621; part (none) -> MCESL35V106M5X5.2
- C? (x2): footprint (none) -> Capacitors_SMD:C_0805; farnell (none) -> 2496940; part (none) -> 0805B104J500CT
- C?: value 480p -> 470p; footprint (none) -> Capacitors_SMD:C_0805; farnell (none) -> 2497037; part (none) -> 0805N471J500CT
- C?: footprint (none) -> Capacitors_SMD:C_0805
Connections:
- net +12V_IGN_Safe renamed +12V_Feed
Changed lines of the file:
@@
 F 0 "C?" H 1540 6196 50  0000 L CNN
 F 1 "1u" H 1540 6105 50  0000 L CNN
-F 2 "" H 1463 6000 50  0000 C CNN
+F 2 "Capacitors_SMD:C_1206" H 1463 6000 50  0001 C CNN
 F 3 "" H 1425 6150 50  0000 C CNN
+F 4 "2362126" H 1425 6150 60  0001 C CNN "farnell"
+F 5 "GRM31MR71E105JA01L" H 1425 6150 60  0001 C CNN "part"
 	1    1425 6150
 	1    0    0    -1
@@
 $EndComp
 $Comp
-L C C?
+L CP C?
 U 1 1 57010AEF
 P 3725 6150
 F 0 "C?" V 3473 6150 50  0000 C CNN
 F 1 "10u" V 3564 6150 50  0000 C CNN
-F 2 "" H 3763 6000 50  0000 C CNN
+F 2 "Capacitors_SMD:c_elec_5x5.3" H 3763 6000 50  0001 C CNN
 F 3 "" H 3725 6150 50  0000 C CNN
+F 4 "MCESL35V106M5X5.2" V 3725 6150 60  0001 C CNN "part"
+F 5 "1870621" V 3725 6150 60  0001 C CNN "farnell"
 	1    3725 6150
 	-1   0    0    1
@@
 F 0 "C?" V 3898 6150 50  0000 C CNN
 F 1 "100n" V 3989 6150 50  0000 C CNN
-F 2 "" H 4188 6000 50  0000 C CNN
+F 2 "Capacitors_SMD:C_0805" H 4188 6000 50  0001 C CNN
 F 3 "" H 4150 6150 50  0000 C CNN
+F 4 "0805B104J500CT" V 4150 6150 60  0001 C CNN "part"
+F 5 "2496940" V 4150 6150 60  0001 C CNN "farnell"
 	1    4150 6150
 	-1   0    0    1
@@
 P 3125 3000
 F 0 "C?" H 3240 3046 50  0000 L CNN
-F 1 "480p" H 3240 2955 50  0000 L CNN
-F 2 "" H 3163 2850 50  0000 C CNN
+F 1 "470p" H 3240 2955 50  0000 L CNN
+F 2 "Capacitors_SMD:C_0805" H 3163 2850 50  0001 C CNN
 F 3 "" H 3125 3000 50  0000 C CNN
+F 4 "0805N471J500CT" H 3125 3000 60  0001 C CNN "part"
+F 5 "2497037" H 3125 3000 60  0001 C CNN "farnell"
 	1    3125 3000
 	1    0    0    -1
@@
 F 0 "C?" H 5590 2721 50  0000 L CNN
 F 1 "100n" H 5590 2630 50  0000 L CNN
-F 2 "" H 5513 2525 50  0000 C CNN
+F 2 "Capacitors_SMD:C_0805" H 5513 2525 50  0001 C CNN
 F 3 "" H 5475 2675 50  0000 C CNN
 F 4 "0805B104J500CT" H 5475 2675 60  0001 C CNN "part"
@@
 F 0 "C?" H 3090 2521 50  0000 L CNN
 F 1 "100n" H 3090 2430 50  0000 L CNN
-F 2 "" H 3013 2325 50  0000 C CNN
+F 2 "Capacitors_SMD:C_0805" H 3013 2325 50  0001 C CNN
 F 3 "" H 2975 2475 50  0000 C CNN
+F 4 "2496940" H 2975 2475 60  0001 C CNN "farnell"
+F 5 "0805B104J500CT" H 2975 2475 60  0001 C CNN "part"
 	1    2975 2475
 	1    0    0    -1
@@
 $EndComp
 Text GLabel 2800 2325 0    60   Input ~ 0
-+12V_IGN_Safe
++12V_Feed
 Text GLabel 5700 2525 2    60   Input ~ 0
 +5V
@@
 $EndComp
 $Comp
-L C C?
+L CP C?
 U 1 1 5708D4A0
 P 7875 2450
 F 0 "C?" H 7990 2496 50  0000 L CNN
 F 1 "10u" H 7990 2405 50  0000 L CNN
-F 2 "" H 7913 2300 50  0000 C CNN
+F 2 "Capacitors_SMD:c_elec_5x5.3" H 7913 2300 50  0001 C CNN
 F 3 "" H 7875 2450 50  0000 C CNN
+F 4 "MCESL35V106M5X5.2" H 7875 2450 60  0001 C CNN "part"
+F 5 "1870621" H 7875 2450 60  0001 C CNN "farnell"
 	1    7875 2450
 	1    0    0    -1
 $EndComp
 $Comp
-L C C?
+L CP C?
 U 1 1 5708D4FA
 P 9025 2450
 F 0 "C?" H 9140 2496 50  0000 L CNN
 F 1 "10u" H 9140 2405 50  0000 L CNN
-F 2 "" H 9063 2300 50  0000 C CNN
+F 2 "Capacitors_SMD:c_elec_5x5.3" H 9063 2300 50  0001 C CNN
 F 3 "" H 9025 2450 50  0000 C CNN
+F 4 "MCESL35V106M5X5.2" H 9025 2450 60  0001 C CNN "part"
+F 5 "1870621" H 9025 2450 60  0001 C CNN "farnell"
 	1    9025 2450
 	1    0    0    -1
