File: electronics/Parkbrake/PowerRegulators.sch (KiCad schematic (older format))
At the start: 23 parts, among them U21 MIC2619, U22 MC34063, U23 LD1117S33CTR

Commit message: traceroute finished although there probably is some errors
Connections:
- net +3.3V: now also C41.1
Changed lines of the file:
@@
 Connection ~ 7875 2300
-Wire Wire Line
-	8850 2300 9250 2300
 Wire Wire Line
 	8450 2600 8450 2775
@@
 $Comp
 L PWR_FLAG #FLG075
-U 1 1 57980F2B
-P 9025 2300
-F 0 "#FLG075" H 9025 2395 50  0001 C CNN
-F 1 "PWR_FLAG" H 9025 2480 50  0001 C CNN
-F 2 "" H 9025 2300 50  0000 C CNN
-F 3 "" H 9025 2300 50  0000 C CNN
-	1    9025 2300
-	1    0    0    -1
-$EndComp
-$Comp
-L PWR_FLAG #FLG076
 U 1 1 5798551D
 P 5075 2525
-F 0 "#FLG076" H 5075 2620 50  0001 C CNN
+F 0 "#FLG075" H 5075 2620 50  0001 C CNN
 F 1 "PWR_FLAG" H 5075 2705 50  0001 C CNN
 F 2 "" H 5075 2525 50  0000 C CNN
@@
 	1    0    0    -1
 $EndComp
+Wire Wire Line
+	8850 2300 9250 2300
+Connection ~ 9025 2300
 $EndSCHEMATC

Commit message: minor tweaks to pcb, had a cap on wrong polarity
Connections:
- net GNDPWR: now also C36.2; no longer C36.1
- net gate_drive_24V: now also C36.1; no longer C36.2
Changed lines of the file:
@@
 U 1 1 57010AEF
 P 3725 6150
-F 0 "C36" V 3473 6150 50  0000 C CNN
-F 1 "10u" V 3564 6150 50  0000 C CNN
+F 0 "C36" V 3950 6150 50  0000 C CNN
+F 1 "10u" V 3850 6150 50  0000 C CNN
 F 2 "Capacitors_Tantalum_SMD:TantalC_SizeC_EIA-6032_Wave" H 3763 6000 50  0001 C CNN
 F 3 "" H 3725 6150 50  0000 C CNN
@@
 F 5 "1457464" V 3725 6150 60  0001 C CNN "farnell"
 	1    3725 6150
-	-1   0    0    1
+	1    0    0    -1
 $EndComp
 $Comp

Commit message: reduce switching noise from 5v regulator circuit
Parts:
- added C100: 10u, myfootprints:CP_0805, symbol CP
- added C101: 1u, Capacitors_SMD:C_1206, symbol C
Connections:
- net +12V_Feed: now also C100.1, C101.1
- net GND: now also C100.2, C101.2
Changed lines of the file:
@@
 $EndComp
 $Comp
-L GNDPWR #PWR068
+L GNDPWR #PWR59
 U 1 1 57010C16
 P 1675 6425
-F 0 "#PWR068" H 1675 6225 50  0001 C CNN
+F 0 "#PWR59" H 1675 6225 50  0001 C CNN
 F 1 "GNDPWR" H 1675 6200 50  0001 C CNN
 F 2 "" H 1675 6375 50  0000 C CNN
@@
 $EndComp
 $Comp
-L GNDPWR #PWR069
+L GNDPWR #PWR61
 U 1 1 57011519
 P 3350 6700
-F 0 "#PWR069" H 3350 6500 50  0001 C CNN
+F 0 "#PWR61" H 3350 6500 50  0001 C CNN
 F 1 "GNDPWR" H 3357 6774 50  0001 C CNN
 F 2 "" H 3350 6650 50  0000 C CNN
@@
 $EndComp
 $Comp
-L GNDPWR #PWR070
+L GNDPWR #PWR63
 U 1 1 57011573
 P 3950 6300
-F 0 "#PWR070" H 3950 6100 50  0001 C CNN
+F 0 "#PWR63" H 3950 6100 50  0001 C CNN
 F 1 "GNDPWR" H 3957 6374 50  0001 C CNN
 F 2 "" H 3950 6250 50  0000 C CNN
@@
 $EndComp
 $Comp
-L GND #PWR071
+L GND #PWR62
 U 1 1 5708A002
 P 3675 3150
-F 0 "#PWR071" H 3675 2900 50  0001 C CNN
+F 0 "#PWR62" H 3675 2900 50  0001 C CNN
 F 1 "GND" H 3683 2977 50  0000 C CNN
 F 2 "" H 3675 3150 50  0000 C CNN
@@
 $EndComp
 $Comp
-L GND #PWR072
+L GND #PWR64
 U 1 1 5708ABA3
 P 5300 2850
-F 0 "#PWR072" H 5300 2600 50  0001 C CNN
+F 0 "#PWR64" H 5300 2600 50  0001 C CNN
 F 1 "GND" H 5308 2677 50  0000 C CNN
 F 2 "" H 5300 2850 50  0000 C CNN
@@
 $EndComp
 $Comp
-L GND #PWR073
+L GND #PWR60
 U 1 1 5708B974
 P 2975 2625
-F 0 "#PWR073" H 2975 2375 50  0001 C CNN
+F 0 "#PWR60" H 2975 2375 50  0001 C CNN
 F 1 "GND" H 2983 2452 50  0000 C CNN
 F 2 "" H 2975 2625 50  0000 C CNN
@@
 	1    0    0    -1
 $EndComp
-Text GLabel 2800 2325 0    60   Input ~ 0
+Text GLabel 2475 2225 0    60   Input ~ 0
 +12V_Feed
 Text GLabel 5700 2525 2    60   Input ~ 0
@@
 $EndComp
 $Comp
-L GND #PWR074
+L GND #PWR65
 U 1 1 5708D552
 P 8450 2775
-F 0 "#PWR074" H 8450 2525 50  0001 C CNN
+F 0 "#PWR65" H 8450 2525 50  0001 C CNN
 F 1 "GND" H 8458 2602 50  0000 C CNN
 F 2 "" H 8450 2775 50  0000 C CNN
@@
 	1    0    0    -1
 $EndComp
-Wire Wire Line
-	1675 5550 1675 6150
-Wire Wire Line
-	1675 6300 1675 6425
-Wire Wire Line
-	1675 6300 1425 6300
-Wire Wire Line
-	1675 6000 1425 6000
-Wire Wire Line
-	1675 5550 1875 5550
-Connection ~ 1675 6000
-Wire Wire Line
-	2375 5550 2575 5550
-Wire Wire Line
-	2575 5550 2575 6000
-Wire Wire Line
-	3075 6300 3075 6375
-Wire Wire Line
-	3350 6300 3350 6375
-Connection ~ 3075 6000
-Connection ~ 3350 6000
-Wire Wire Line
-	3075 6300 2800 6300
-Wire Wire Line
-	2800 6300 2800 6150
-Wire Wire Line
-	2800 6150 2575 6150
-Wire Wire Line
-	3350 6350 2575 6350
-Wire Wire Line
-	2575 6350 2575 6300
-Connection ~ 3350 6350
-Wire Wire Line
-	2575 6000 2675 6000
-Wire Wire Line
-	3350 6700 3350 6675
-Wire Wire Line
-	3350 6675 3075 6675
-Wire Wire Line
-	2875 6000 4500 6000
-Connection ~ 3725 6000
-Connection ~ 4150 6000
-Wire Wire Line
-	3725 6300 4150 6300
-Connection ~ 3950 6300
-Wire Wire Line
-	3125 3150 4350 3150
-Connection ~ 4075 3150
-Wire Wire Line
-	3125 2850 3125 2725
-Wire Wire Line
-	3125 2725 3275 2725
-Wire Wire Line
-	4075 2725 4075 2850
-Wire Wire Line
-	4075 2725 4475 2725
-Wire Wire Line
-	3675 2925 3675 3150
-Connection ~ 3675 3150
-Wire Wire Line
-	4350 2525 4075 2525
-Connection ~ 5075 2525
-Connection ~ 5475 2525
-Wire Wire Line
-	5075 2825 5475 2825
-Wire Wire Line
-	5300 2825 5300 2850
-Connection ~ 5300 2825
-Wire Wire Line
-	4100 2325 4075 2325
-Wire Wire Line
-	4100 1750 4100 2325
-Wire Wire Line
-	4100 2125 4075 2125
-Wire Wire Line
-	4100 1750 2975 1750
-Wire Wire Line
-	2975 1750 2975 2025
-Connection ~ 4100 2125
-Wire Wire Line
-	3275 2125 3275 1950
-Wire Wire Line
-	3275 1950 2975 1950
-Connection ~ 2975 1950
-Wire Wire Line
-	2800 2325 3275 2325
-Connection ~ 2975 2325
-Wire Wire Line
-	4850 2725 4850 2525
-Wire Wire Line
-	4850 2725 4775 2725
-Wire Wire Line
-	4350 2850 4350 2525
-Wire Wire Line
-	4850 2525 5700 2525
-Wire Wire Line
-	7750 2300 8050 2300
-Connection ~ 7875 2300
-Wire Wire Line
-	8450 2600 8450 2775
-Wire Wire Line
-	9025 2650 9025 2600
-Wire Wire Line
-	7875 2650 9025 2650
-Connection ~ 8450 2650
-Wire Wire Line
-	7875 2650 7875 2600
 Text GLabel 7750 2300 0    60   Input ~ 0
 +5V
@@
 +3.3V
 $Comp
-L PWR_FLAG #FLG075
+L PWR_FLAG #FLG10
 U 1 1 5798551D
 P 5075 2525
-F 0 "#FLG075" H 5075 2620 50  0001 C CNN
+F 0 "#FLG10" H 5075 2620 50  0001 C CNN
 F 1 "PWR_FLAG" H 5075 2705 50  0001 C CNN
 F 2 "" H 5075 2525 50  0000 C CNN
@@
 	1    0    0    -1
 $EndComp
+$Comp
+L CP C100
+U 1 1 5B5216F6
+P 2475 2475
+F 0 "C100" H 2200 2575 50  0000 L CNN
+F 1 "10u" H 2275 2375 50  0000 L CNN
+F 2 "myfootprints:CP_0805" H 2513 2325 50  0001 C CNN
+F 3 "" H 2475 2475 50  0000 C CNN
+F 4 "TMCP0J106KTRF" H 2475 2475 60  0001 C CNN "part"
+F 5 "2491430" H 2475 2475 60  0001 C CNN "farnell"
+	1    2475 2475
+	1    0    0    -1
+$EndComp
+$Comp
+L C C101
+U 1 1 5B521DEF
+P 2700 2475
+F 0 "C101" H 2725 2575 50  0000 L CNN
+F 1 "1u" H 2725 2400 50  0000 L CNN
+F 2 "Capacitors_SMD:C_1206" H 2738 2325 50  0001 C CNN
+F 3 "" H 2700 2475 50  0000 C CNN
+F 4 "2362126" H 2700 2475 60  0001 C CNN "farnell"
+F 5 "GRM31MR71E105JA01L" H 2700 2475 60  0001 C CNN "part"
+	1    2700 2475
+	1    0    0    -1
+$EndComp
+Wire Wire Line
+	1675 5550 1675 6150
+Wire Wire Line
+	1675 6300 1675 6425
+Wire Wire Line
+	1675 6300 1425 6300
+Wire Wire Line
+	1675 6000 1425 6000
+Wire Wire Line
+	1675 5550 1875 5550
+Connection ~ 1675 6000
+Wire Wire Line
+	2375 5550 2575 5550
+Wire Wire Line
+	2575 5550 2575 6000
+Wire Wire Line
+	3075 6300 3075 6375
+Wire Wire Line
+	3350 6300 3350 6375
+Connection ~ 3075 6000
+Connection ~ 3350 6000
+Wire Wire Line
+	3075 6300 2800 6300
+Wire Wire Line
+	2800 6300 2800 6150
+Wire Wire Line
+	2800 6150 2575 6150
+Wire Wire Line
+	3350 6350 2575 6350
+Wire Wire Line
+	2575 6350 2575 6300
+Connection ~ 3350 6350
+Wire Wire Line
+	2575 6000 2675 6000
+Wire Wire Line
+	3350 6700 3350 6675
+Wire Wire Line
+	3350 6675 3075 6675
+Wire Wire Line
+	2875 6000 4500 6000
+Connection ~ 3725 6000
+Connection ~ 4150 6000
+Wire Wire Line
+	3725 6300 4150 6300
+Connection ~ 3950 6300
+Wire Wire Line
+	3125 3150 4350 3150
+Connection ~ 4075 3150
+Wire Wire Line
+	3125 2850 3125 2725
+Wire Wire Line
+	3125 2725 3275 2725
+Wire Wire Line
+	4075 2725 4075 2850
+Wire Wire Line
+	4075 2725 4475 2725
+Wire Wire Line
+	3675 2925 3675 3150
+Connection ~ 3675 3150
+Wire Wire Line
+	4350 2525 4075 2525
+Connection ~ 5075 2525
+Connection ~ 5475 2525
+Wire Wire Line
+	5075 2825 5475 2825
+Wire Wire Line
+	5300 2825 5300 2850
+Connection ~ 5300 2825
+Wire Wire Line
+	4100 2325 4075 2325
+Wire Wire Line
+	4100 1750 4100 2325
+Wire Wire Line
+	4100 2125 4075 2125
+Wire Wire Line
+	4100 1750 2975 1750
+Wire Wire Line
+	2975 1750 2975 2025
+Connection ~ 4100 2125
+Wire Wire Line
+	3275 2125 3275 1950
+Wire Wire Line
+	3275 1950 2975 1950
+Connection ~ 2975 1950
+Wire Wire Line
+	2475 2325 3275 2325
+Connection ~ 2975 2325
+Wire Wire Line
+	4850 2725 4850 2525
+Wire Wire Line
+	4850 2725 4775 2725
+Wire Wire Line
+	4350 2850 4350 2525
+Wire Wire Line
+	4850 2525 5700 2525
+Wire Wire Line
+	7750 2300 8050 2300
+Connection ~ 7875 2300
+Wire Wire Line
+	8450 2600 8450 2775
+Wire Wire Line
+	9025 2650 9025 2600
+Wire Wire Line
+	7875 2650 9025 2650
+Connection ~ 8450 2650
+Wire Wire Line
+	7875 2650 7875 2600
 Wire Wire Line
 	8850 2300 9250 2300
 Connection ~ 9025 2300
+Wire Wire Line
+	2475 2625 2975 2625
+Connection ~ 2700 2325
+Connection ~ 2700 2625
+Wire Wire Line
+	2475 2325 2475 2225
 $EndSCHEMATC

Commit message: Warning in schematic
Other:
- note added: "wrong tantal voltage"
Changed lines of the file:
@@
 Wire Wire Line
 	2475 2325 2475 2225
+Text Notes 1400 2550 0    60   ~ 0
+wrong tantal voltage
 $EndSCHEMATC
