File: electronics/Parkbrake/Parkbrake.kicad_pcb (KiCad board)
At the start: 2 copper layers, 109.2 x 114.3 mm, 1 part, among them P1 Conn48pin

Commit message: More fixes and chenged components eat less boardspace
Parts:
- added C1: 100n, Capacitors_SMD:C_0805, F.Cu at (341.3, 147.5)
- added C10: 1u, Capacitors_SMD:C_1206, F.Cu at (217.8, 121.7)
- added C11: 100n, Capacitors_SMD:C_0805, F.Cu at (227.4, 120.7)
- added C12: 100n, Capacitors_SMD:C_0805, F.Cu at (242.1, 107.7)
- added C13: 100n, Capacitors_SMD:C_0805, F.Cu at (250.6, 101.0)
- added C14: 1u, Capacitors_SMD:C_1206, F.Cu at (236.2, 94.5)
- added C15: 220nF, Capacitors_SMD:C_1206, F.Cu at (225.2, 113.4)
- added C16: 100n, Capacitors_SMD:C_0805, F.Cu at (243.3, 121.3)
- added C17: 1u, Capacitors_SMD:C_1206, F.Cu at (246.1, 94.5)
- added C18: 100n, Capacitors_SMD:C_0805, F.Cu at (247.6, 121.3)
- added C19: 100n, Capacitors_SMD:C_0805, F.Cu at (247.7, 62.3)
- added C2: 100n, Capacitors_SMD:C_0805, F.Cu at (337.6, 141.2)
- added C20: 100n, Capacitors_SMD:C_0805, F.Cu at (256.2, 55.6)
- added C21: 1u, Capacitors_SMD:C_1206, F.Cu at (233.1, 64.4)
- added C22: 220nF, Capacitors_SMD:C_1206, F.Cu at (216.2, 81.0)
- added C23: 100n, Capacitors_SMD:C_0805, F.Cu at (261.4, 48.9)
- added C24: 1u, Capacitors_SMD:C_1206, F.Cu at (251.9, 49.1)
- added C25: 100n, Capacitors_SMD:C_0805, F.Cu at (235.4, 77.6)
- added C26: 100n, Capacitors_SMD:C_0805, F.Cu at (259.3, 61.9)
- added C27: 100n, Capacitors_SMD:C_0805, F.Cu at (234.8, 83.9)
- added C28: 1u, Capacitors_SMD:C_1206, F.Cu at (221.3, 81.4)
- added C29: 220nF, Capacitors_SMD:C_1206, F.Cu at (226.4, 81.4)
- added C3: 100n, Capacitors_SMD:C_0805, F.Cu at (345.6, 149.2)
- added C30: 100n, Capacitors_SMD:C_0805, F.Cu at (231.1, 77.6)
- added C31: 1u, Capacitors_SMD:C_1206, F.Cu at (238.0, 71.1)
- added C32: 100n, Capacitors_SMD:C_0805, F.Cu at (242.7, 71.4)
- added C33: 1u, Capacitors_SMD:C_1206, F.Cu at (296.4, 130.2)
- added C34: 100n, Capacitors_SMD:C_0805, F.Cu at (301.1, 130.0)
- added C35: 470p, Capacitors_SMD:C_0805, F.Cu at (295.3, 149.3)
- added C36: 10u, Capacitors_Tantalum_SMD:TantalC_SizeC_EIA-6032_Wave, F.Cu at (274.9, 131.2)
- added C37: 100n, Capacitors_SMD:C_0805, F.Cu at (275.8, 145.2)
- added C38: 680u, Capacitors_Tantalum_SMD:TantalC_SizeD_EIA-7343_Wave, F.Cu at (263.9, 131.2)
- added C39: 100n, Capacitors_SMD:C_0805, F.Cu at (287.4, 145.3)
- added C4: 100n, Capacitors_SMD:C_0805, F.Cu at (349.3, 141.9)
- added C40: 10u, myfootprints:CP_0805, F.Cu at (302.3, 142.5)
- added C41: 10u, myfootprints:CP_0805, F.Cu at (299.5, 149.2)
- added C42: 100n, Capacitors_SMD:C_0805, F.Cu at (348.0, 105.4)
- added C43: 1n, Capacitors_SMD:C_0805, F.Cu at (358.1, 92.4)
- added C44: 26p, Capacitors_SMD:C_0805, F.Cu at (354.1, 92.8)
- added C45: 26p, Capacitors_SMD:C_0805, F.Cu at (361.4, 86.1)
- added C46: 4.7u, myfootprints:CP_0805, F.Cu at (352.9, 99.0)
- added C47: 100n, Capacitors_SMD:C_0805, F.Cu at (348.8, 99.1)
- added C48: 100n, Capacitors_SMD:C_0805, F.Cu at (340.0, 105.4)
- added C49: 10n, Capacitors_SMD:C_0805, F.Cu at (357.3, 86.1)
- added C5: 100n, Capacitors_SMD:C_0805, F.Cu at (237.8, 127.0)
- added C50: 1u, Capacitors_SMD:C_1206, F.Cu at (352.8, 86.3)
- added C51: 10n, Capacitors_SMD:C_0805, F.Cu at (344.6, 99.1)
- added C52: 1u, Capacitors_SMD:C_1206, F.Cu at (347.7, 86.3)
- added C53: 10n, Capacitors_SMD:C_0805, F.Cu at (350.0, 92.8)
- added C54: 1u, Capacitors_SMD:C_1206, F.Cu at (341.4, 92.6)
- added C55: 10n, Capacitors_SMD:C_0805, F.Cu at (346.0, 92.8)
- added C56: 1u, Capacitors_SMD:C_1206, F.Cu at (335.3, 100.7)
- added C57: 100n, Capacitors_SMD:C_0805, F.Cu at (358.1, 56.7)
- added C58: 1n, Capacitors_SMD:C_0805, F.Cu at (373.2, 57.6)
- added C59: 100n, Capacitors_SMD:C_0805, F.Cu at (367.0, 51.3)
- added C6: 100n, Capacitors_SMD:C_0805, F.Cu at (245.8, 115.0)
- added C60: 100n, Capacitors_SMD:C_0805, F.Cu at (362.7, 50.4)
- added C61: 100n, Capacitors_SMD:C_0805, F.Cu at (196.9, 149.6)
- added C62: 100n, Capacitors_SMD:C_0805, F.Cu at (211.3, 138.5)
- added C63: 1n, Capacitors_SMD:C_0805, F.Cu at (205.5, 144.8)
- added C64: 100n, Capacitors_SMD:C_0805, F.Cu at (209.7, 144.8)
- added C65: 100n, Capacitors_SMD:C_0805, F.Cu at (291.5, 111.3)
- added C66: 100n, Capacitors_SMD:C_0805, F.Cu at (280.4, 118.6)
- added C67: 100n, Capacitors_SMD:C_0805, F.Cu at (287.2, 106.0)
- added C68: 100n, Capacitors_SMD:C_0805, F.Cu at (286.5, 112.3)
- added C69: 100n, Capacitors_SMD:C_0805, F.Cu at (297.8, 101.0)
- added C7: 1u, Capacitors_SMD:C_1206, F.Cu at (241.0, 101.2)
- added C70: 100n, Capacitors_SMD:C_0805, F.Cu at (303.0, 94.3)
- added C71: 100n, Capacitors_SMD:C_0805, F.Cu at (282.2, 111.9)
- added C72: 33uF, myfootprints:CP_1206, F.Cu at (298.3, 94.5)
- added C73: 33uF, myfootprints:CP_1206, F.Cu at (271.3, 118.8)
- added C74: 1u, Capacitors_SMD:C_1206, F.Cu at (301.1, 71.9)
- added C75: 1u, Capacitors_SMD:C_1206, F.Cu at (309.1, 64.9)
- added C76: 1u, Capacitors_SMD:C_1206, F.Cu at (296.0, 71.9)
- added C77: 1u, Capacitors_SMD:C_1206, F.Cu at (324.9, 42.4)
- added C78: 1u, Capacitors_SMD:C_1206, F.Cu at (304.0, 64.6)
- added C79: 1u, Capacitors_SMD:C_1206, F.Cu at (319.2, 49.1)
- added C8: 220nF, Capacitors_SMD:C_1206, F.Cu at (114.0, 115.5)
- added C80: 1u, Capacitors_SMD:C_1206, F.Cu at (309.1, 51.5)
- added C81: 1u, Capacitors_SMD:C_1206, F.Cu at (314.1, 48.7)
- added C82: 1u, Capacitors_SMD:C_1206, F.Cu at (309.1, 58.2)
- added C83: 47n, Capacitors_SMD:C_0805, F.Cu at (332.4, 48.5)
- added C84: 47n, Capacitors_SMD:C_0805, F.Cu at (313.6, 68.2)
- added C85: 47n, Capacitors_SMD:C_0805, F.Cu at (329.5, 42.2)
- added C86: 47n, Capacitors_SMD:C_0805, F.Cu at (333.5, 42.2)
- added C87: 1u, Capacitors_SMD:C_1206, F.Cu at (298.8, 65.2)
- added C88: 1u, Capacitors_SMD:C_1206, F.Cu at (314.1, 55.4)
- added C89: 1u, Capacitors_SMD:C_1206, F.Cu at (291.0, 70.5)
- added C9: 100n, Capacitors_SMD:C_0805, F.Cu at (231.7, 120.7)
- added C90: 1u, Capacitors_SMD:C_1206, F.Cu at (304.0, 57.9)
- added C91: 1u, Capacitors_SMD:C_1206, F.Cu at (319.9, 42.4)
- added C92: 10u, myfootprints:CP_0805, F.Cu at (332.0, 55.2)
- added C93: 10u, myfootprints:CP_0805, F.Cu at (326.1, 61.9)
- added C94: 100n, Capacitors_SMD:C_0805, F.Cu at (328.3, 48.9)
- added C95: 100n, Capacitors_SMD:C_0805, F.Cu at (323.1, 55.6)
- added C96: 1n, Capacitors_SMD:C_0805, F.Cu at (305.6, 71.4)
- added C97: 1n, Capacitors_SMD:C_0805, F.Cu at (313.6, 61.9)
- added C98: 100n, Capacitors_SMD:C_0805, F.Cu at (318.8, 55.6)
- added C99: 1n, Capacitors_SMD:C_0805, F.Cu at (317.7, 61.9)
- added D1: 10v, Diodes_SMD:SOD-323, F.Cu at (247.3, 138.3)
- added D10: RF_Release, LEDs:LED_0805, F.Cu at (322.1, 138.8)
- added D11: RF_tighten, LEDs:LED_0805, F.Cu at (339.4, 135.2)
- added D12: RR_Release, LEDs:LED_0805, F.Cu at (313.8, 148.0)
- added D13: RR_Tighten, LEDs:LED_0805, F.Cu at (330.9, 138.8)
- added D14: 1n4148W, Diodes_SMD:SOD-323, F.Cu at (229.9, 94.1)
- added D15: 1n4148W, Diodes_SMD:SOD-323, F.Cu at (221.6, 107.1)
- added D16: 1n4148W, Diodes_SMD:SOD-323, F.Cu at (214.0, 114.5)
- added D17: 1n4148W, Diodes_SMD:SOD-323, F.Cu at (221.6, 101.3)
- added D18: 1n4148W, Diodes_SMD:SOD-323, F.Cu at (204.9, 123.8)
- added D19: 1n4148W, Diodes_SMD:SOD-323, F.Cu at (229.9, 99.9)
- added D2: 10v, Diodes_SMD:SOD-323, F.Cu at (245.7, 143.3)
- added D20: 1n4148W, Diodes_SMD:SOD-323, F.Cu at (212.1, 68.9)
- added D21: 1n4148W, Diodes_SMD:SOD-323, F.Cu at (229.6, 58.1)
- added D22: 1n4148W, Diodes_SMD:SOD-323, F.Cu at (217.2, 74.7)
- added D23: 1n4148W, Diodes_SMD:SOD-323, F.Cu at (226.8, 68.4)
- added D24: 1n4148W, Diodes_SMD:SOD-323, F.Cu at (219.5, 68.9)
- added D25: 1n4148W, Diodes_SMD:SOD-323, F.Cu at (236.9, 58.1)
- added D26: min 40V 1A, Diodes_SMD:SOD-123, F.Cu at (273.6, 138.9)
- added D27: min 1.5A, Diodes_SMD:SOD-123, F.Cu at (288.8, 139.0)
- added D28: 3.3V, Diodes_SMD:SOD-323, F.Cu at (204.6, 150.9)
- added D29: 3.3V, Diodes_SMD:SOD-323, F.Cu at (200.9, 150.9)
- added D3: 1n4148w, Diodes_SMD:SOD-323, F.Cu at (220.7, 144.1)
- added D30: 1n4148w, Diodes_SMD:SOD-323, F.Cu at (184.5, 149.9)
- added D31: 3.3V, Diodes_SMD:SOD-323, F.Cu at (307.0, 100.4)
- added D32: 3.3V, Diodes_SMD:SOD-323, F.Cu at (267.3, 106.3)
- added D33: 3.3V, Diodes_SMD:SOD-323, F.Cu at (290.4, 117.3)
- added D34: 3.3V, Diodes_SMD:SOD-323, F.Cu at (300.0, 107.1)
- added D35: 1n4148w, Diodes_SMD:SOD-323, F.Cu at (284.8, 99.9)
- added D36: 1n4148w, Diodes_SMD:SOD-323, F.Cu at (269.0, 112.5)
- added D37: 1n4148w, Diodes_SMD:SOD-323, F.Cu at (284.8, 94.1)
- added D38: 1n4148w, Diodes_SMD:SOD-323, F.Cu at (292.0, 94.1)
- added D39: 1n4148w, Diodes_SMD:SOD-323, F.Cu at (265.0, 118.3)
- added D4: 1n4148w, Diodes_SMD:SOD-323, F.Cu at (220.7, 138.3)
- added D40: 1n4148w, Diodes_SMD:SOD-323, F.Cu at (276.3, 112.5)
- added D41: 1n4148w, Diodes_SMD:SOD-323, F.Cu at (281.3, 105.8)
- added D5: 10v, Diodes_SMD:SOD-323, F.Cu at (241.0, 144.6)
- added D6: LF_Release, LEDs:LED_0805, F.Cu at (322.7, 144.4)
- added D7: LF_Tighten, LEDs:LED_0805, F.Cu at (331.3, 144.4)
- added D8: LR_Release, LEDs:LED_0805, F.Cu at (338.7, 129.6)
- added D9: LR_Tighten, LEDs:LED_0805, F.Cu at (347.4, 129.6)
- added JP1: Jumper_NO_Small, Resistors_SMD:R_0805_HandSoldering, F.Cu at (338.3, 86.1)
- added JP10: RF_passth+, Resistors_SMD:R_0805_HandSoldering, F.Cu at (285.4, 48.5)
- added JP11: RF+_to_in, Resistors_SMD:R_0805_HandSoldering, F.Cu at (293.1, 57.7)
- added JP12: soft_R_out-, Resistors_SMD:R_0805_HandSoldering, F.Cu at (278.9, 42.2)
- added JP13: RF_passth-, Resistors_SMD:R_0805_HandSoldering, F.Cu at (275.8, 65.1)
- added JP14: RF-_to_in, Resistors_SMD:R_0805_HandSoldering, F.Cu at (313.3, 42.2)
- added JP2: Jumper_NO_Small, Resistors_SMD:R_0805_HandSoldering, F.Cu at (353.7, 50.4)
- added JP3: soft_L_out+, Resistors_SMD:R_0805_HandSoldering, F.Cu at (275.9, 58.8)
- added JP4: L_passth+, Resistors_SMD:R_0805_HandSoldering, F.Cu at (294.2, 51.4)
- added JP5: LF+_to_in, Resistors_SMD:R_0805_HandSoldering, F.Cu at (292.4, 64.0)
- added JP6: soft_L_out-, Resistors_SMD:R_0805_HandSoldering, F.Cu at (288.4, 42.2)
- added JP7: L_passth-, Resistors_SMD:R_0805_HandSoldering, F.Cu at (302.4, 51.4)
- added JP8: LF-_to_in, Resistors_SMD:R_0805_HandSoldering, F.Cu at (283.5, 74.2)
- added JP9: soft_R_out+, Resistors_SMD:R_0805_HandSoldering, F.Cu at (276.0, 52.5)
- added L1: 10uH, myfootprints:inductor_sd54, F.Cu at (270.2, 149.9)
- added L2: 33uH, myfootprints:inductor_sd54, F.Cu at (290.4, 131.2)
- added P2: JTAG, Socket_Strips:Socket_Strip_Straight_1x08, F.Cu at (348.7, 45.2)
- added P3: UART, Socket_Strips:Socket_Strip_Straight_1x03, F.Cu at (348.9, 59.7)
- added Q1: BSS138, TO_SOT_Packages_SMD:SOT-323, F.Cu at (220.4, 150.1)
- added Q10: IPD031N06L3 G, TO_SOT_Packages_SMD:TO-252-2Lead, F.Cu at (167.9, 71.2)
- added Q11: IPD031N06L3 G, TO_SOT_Packages_SMD:TO-252-2Lead, F.Cu at (167.9, 76.6)
- added Q12: NX3008CBKS, SOT363:SOT-363, F.Cu at (200.6, 109.7)
- added Q13: NX3008CBKS, SOT363:SOT-363, F.Cu at (197.7, 109.7)
- added Q14: IPD031N06L3 G, TO_SOT_Packages_SMD:TO-252-2Lead, F.Cu at (144.5, 76.7)
- added Q15: IPD031N06L3 G, TO_SOT_Packages_SMD:TO-252-2Lead, F.Cu at (144.5, 71.1)
- added Q16: IPD031N06L3 G, TO_SOT_Packages_SMD:TO-252-2Lead, F.Cu at (152.3, 71.1)
- added Q17: IPD031N06L3 G, TO_SOT_Packages_SMD:TO-252-2Lead, F.Cu at (152.3, 76.6)
- added Q18: NX3008CBKS, SOT363:SOT-363, F.Cu at (194.7, 109.7)
- added Q19: NX3008CBKS, SOT363:SOT-363, F.Cu at (222.4, 44.1)
- added Q2: BSS138, TO_SOT_Packages_SMD:SOT-323, F.Cu at (238.8, 138.4)
- added Q20: IPD031N06L3 G, TO_SOT_Packages_SMD:TO-252-2Lead, F.Cu at (199.5, 50.5)
- added Q21: IPD031N06L3 G, TO_SOT_Packages_SMD:TO-252-2Lead, F.Cu at (187.1, 50.5)
- added Q22: IPD031N06L3 G, TO_SOT_Packages_SMD:TO-252-2Lead, F.Cu at (187.1, 77.4)
- added Q23: IPD031N06L3 G, TO_SOT_Packages_SMD:TO-252-2Lead, F.Cu at (199.5, 64.0)
- added Q24: NX3008CBKS, SOT363:SOT-363, F.Cu at (219.4, 44.1)
- added Q25: NX3008CBKS, SOT363:SOT-363, F.Cu at (207.1, 71.1)
- added Q26: IPD031N06L3 G, TO_SOT_Packages_SMD:TO-252-2Lead, F.Cu at (211.8, 64.0)
- added Q27: IPD031N06L3 G, TO_SOT_Packages_SMD:TO-252-2Lead, F.Cu at (199.5, 77.4)
- added Q28: IPD031N06L3 G, TO_SOT_Packages_SMD:TO-252-2Lead, F.Cu at (211.8, 50.5)
- added Q29: IPD031N06L3 G, TO_SOT_Packages_SMD:TO-252-2Lead, F.Cu at (187.1, 64.0)
- added Q3: P-ch -40V 0.0035ohm, TO_SOT_Packages_SMD:TO-252-2Lead, F.Cu at (84.3, 69.7)
- added Q30: NX3008CBKS, SOT363:SOT-363, F.Cu at (225.3, 44.1)
- added Q31: BSS138, TO_SOT_Packages_SMD:SOT-323, F.Cu at (197.9, 138.4)
- added Q32: NTS4173, TO_SOT_Packages_SMD:SOT-323, F.Cu at (292.1, 100.1)
- added Q33: NX3008CBKS, SOT363:SOT-363, F.Cu at (272.7, 44.1)
- added Q4: P-ch -40V 0.0035ohm, TO_SOT_Packages_SMD:TO-252-2Lead, F.Cu at (130.1, 59.8)
- added Q5: BSS308, TO_SOT_Packages_SMD:SOT-23, F.Cu at (232.5, 138.7)
- added Q6: BSS308, TO_SOT_Packages_SMD:SOT-23, F.Cu at (227.6, 145.4)
- added Q7: NX3008CBKS, SOT363:SOT-363, F.Cu at (185.9, 108.5)
- added Q8: IPD031N06L3 G, TO_SOT_Packages_SMD:TO-252-2Lead, F.Cu at (160.1, 76.7)
- added Q9: IPD031N06L3 G, TO_SOT_Packages_SMD:TO-252-2Lead, F.Cu at (160.2, 71.1)
- added R1: 10k, Resistors_SMD:R_0805, F.Cu at (236.2, 149.6)
- added R10: 10k, Resistors_SMD:R_Array_Concave_4x0603, F.Cu at (345.3, 136.1)
- added R100: 10k, Resistors_SMD:R_0805, F.Cu at (203.3, 138.5)
- added R101: 1k, Resistors_SMD:R_0805, F.Cu at (190.4, 150.1)
- added R102: 560, Resistors_SMD:R_0805, F.Cu at (201.3, 144.8)
- added R103: 2.2k, Resistors_SMD:R_0805, F.Cu at (291.6, 105.0)
- added R104: 1k, Resistors_SMD:R_Array_Concave_4x0603, F.Cu at (259.3, 116.2)
- added R105: 100k, Resistors_SMD:R_0805, F.Cu at (303.0, 100.6)
- added R106: 1k, Resistors_SMD:R_0805, F.Cu at (296.0, 107.3)
- added R107: 2k, Resistors_SMD:R_0805, F.Cu at (284.7, 118.6)
- added R108: 1M, Resistors_SMD:R_0805, F.Cu at (307.3, 94.3)
- added R109: 1M, Resistors_SMD:R_0805, F.Cu at (276.0, 118.6)
- added R11: 10k, Resistors_SMD:R_0805, F.Cu at (239.3, 120.7)
- added R110: 1k, Resistors_SMD:R_Array_Concave_4x0603, F.Cu at (299.3, 58.2)
- added R111: 15k, Resistors_SMD:R_0805, F.Cu at (317.9, 68.2)
- added R112: 15k, Resistors_SMD:R_0805, F.Cu at (336.7, 48.5)
- added R113: 15k, Resistors_SMD:R_0805, F.Cu at (321.9, 61.9)
- added R114: 15k, Resistors_SMD:R_0805, F.Cu at (309.8, 74.5)
- added R115: 16.9k, Resistors_SMD:R_0805, F.Cu at (337.9, 42.2)
- added R116: 16.9k, Resistors_SMD:R_0805, F.Cu at (327.6, 55.2)
- added R117: 10k, Resistors_SMD:R_0805, F.Cu at (323.9, 48.9)
- added R12: 10k, Resistors_SMD:R_0805, F.Cu at (115.7, 124.5)
- added R13: 10k, Resistors_SMD:R_0805, F.Cu at (102.2, 107.9)
- added R14: 10, Resistors_SMD:R_1206, F.Cu at (211.1, 127.5)
- added R15: 10, Resistors_SMD:R_1206, F.Cu at (232.7, 107.9)
- added R16: 10k, Resistors_SMD:R_0805, F.Cu at (235.6, 120.7)
- added R17: 43, Resistors_SMD:R_0805, F.Cu at (249.7, 115.0)
- added R18: 10k, Resistors_SMD:R_0805, F.Cu at (108.9, 130.7)
- added R19: 100, Resistors_SMD:R_0805, F.Cu at (208.1, 88.6)
- added R2: 10k, Resistors_SMD:R_0805, F.Cu at (226.7, 150.5)
- added R20: 0.002, Resistors_SMD:R_1206, F.Cu at (166.0, 89.7)
- added R21: 0.002, Resistors_SMD:R_1206, F.Cu at (222.8, 121.7)
- added R22: 0.002, Resistors_SMD:R_1206, F.Cu at (115.8, 131.3)
- added R23: 100, Resistors_SMD:R_0805, F.Cu at (115.6, 110.3)
- added R24: 0.002, Resistors_SMD:R_1206, F.Cu at (101.3, 123.1)
- added R25: 10, Resistors_SMD:R_1206, F.Cu at (246.0, 101.2)
- added R26: 10, Resistors_SMD:R_1206, F.Cu at (237.5, 107.9)
- added R27: 10k, Resistors_SMD:R_0805, F.Cu at (229.6, 114.4)
- added R28: 10k, Resistors_SMD:R_0805, F.Cu at (223.8, 128.2)
- added R29: 10k, Resistors_SMD:R_0805, F.Cu at (247.5, 110.0)
- added R3: 1k, Resistors_SMD:R_0805, F.Cu at (232.6, 145.2)
- added R30: 10k, Resistors_SMD:R_0805, F.Cu at (232.5, 125.6)
- added R31: 10, Resistors_SMD:R_1206, F.Cu at (251.0, 94.5)
- added R32: 10, Resistors_SMD:R_1206, F.Cu at (212.9, 120.8)
- added R33: 10k, Resistors_SMD:R_0805, F.Cu at (220.2, 128.2)
- added R34: 43, Resistors_SMD:R_0805, F.Cu at (233.3, 114.4)
- added R35: 10k, Resistors_SMD:R_0805, F.Cu at (227.5, 127.0)
- added R36: 100, Resistors_SMD:R_0805, F.Cu at (241.8, 114.0)
- added R37: 0.002, Resistors_SMD:R_1206, F.Cu at (215.9, 128.4)
- added R38: 0.002, Resistors_SMD:R_1206, F.Cu at (236.1, 101.2)
- added R39: 0.002, Resistors_SMD:R_1206, F.Cu at (241.1, 94.5)
- added R4: 1k, Resistors_SMD:R_0805, F.Cu at (237.4, 143.3)
- added R40: 100, Resistors_SMD:R_0805, F.Cu at (247.5, 106.3)
- added R41: 0.002, Resistors_SMD:R_1206, F.Cu at (204.7, 129.1)
- added R42: 10, Resistors_SMD:R_1206, F.Cu at (220.2, 115.0)
- added R43: 10, Resistors_SMD:R_1206, F.Cu at (227.8, 106.2)
- added R44: 10k, Resistors_SMD:R_0805, F.Cu at (236.9, 114.4)
- added R45: 10k, Resistors_SMD:R_0805, F.Cu at (260.2, 55.6)
- added R46: 10k, Resistors_SMD:R_0805, F.Cu at (246.7, 74.9)
- added R47: 10k, Resistors_SMD:R_0805, F.Cu at (255.3, 68.2)
- added R48: 10, Resistors_SMD:R_1206, F.Cu at (264.5, 42.4)
- added R49: 10, Resistors_SMD:R_1206, F.Cu at (259.7, 42.4)
- added R5: 10k, Resistors_SMD:R_0805, F.Cu at (243.7, 138.5)
- added R50: 10k, Resistors_SMD:R_0805, F.Cu at (238.7, 84.0)
- added R51: 43, Resistors_SMD:R_0805, F.Cu at (255.3, 61.9)
- added R52: 10k, Resistors_SMD:R_0805, F.Cu at (239.4, 77.7)
- added R53: 100, Resistors_SMD:R_0805, F.Cu at (259.0, 68.2)
- added R54: 0.002, Resistors_SMD:R_1206, F.Cu at (246.9, 49.1)
- added R55: 0.002, Resistors_SMD:R_1206, F.Cu at (245.1, 42.4)
- added R56: 0.002, Resistors_SMD:R_1206, F.Cu at (243.1, 58.2)
- added R57: 100, Resistors_SMD:R_0805, F.Cu at (242.4, 84.0)
- added R58: 0.002, Resistors_SMD:R_1206, F.Cu at (254.8, 42.4)
- added R59: 10, Resistors_SMD:R_1206, F.Cu at (242.1, 51.5)
- added R6: 1k, Resistors_SMD:R_0805, F.Cu at (337.3, 147.5)
- added R60: 10, Resistors_SMD:R_1206, F.Cu at (237.2, 51.5)
- added R61: 10k, Resistors_SMD:R_0805, F.Cu at (265.4, 48.9)
- added R62: 10k, Resistors_SMD:R_0805, F.Cu at (263.8, 55.2)
- added R63: 10k, Resistors_SMD:R_0805, F.Cu at (250.3, 74.9)
- added R64: 10k, Resistors_SMD:R_0805, F.Cu at (252.2, 55.6)
- added R65: 10, Resistors_SMD:R_1206, F.Cu at (256.8, 49.1)
- added R66: 10, Resistors_SMD:R_1206, F.Cu at (200.0, 82.8)
- added R67: 10k, Resistors_SMD:R_0805, F.Cu at (250.8, 68.6)
- added R68: 43, Resistors_SMD:R_0805, F.Cu at (243.0, 77.7)
- added R69: 10k, Resistors_SMD:R_0805, F.Cu at (247.2, 68.6)
- added R7: 1k, Resistors_SMD:R_0805, F.Cu at (341.6, 141.2)
- added R70: 100, Resistors_SMD:R_0805, F.Cu at (251.7, 62.3)
- added R71: 0.002, Resistors_SMD:R_1206, F.Cu at (225.7, 74.7)
- added R72: 0.002, Resistors_SMD:R_1206, F.Cu at (238.1, 64.4)
- added R73: 0.002, Resistors_SMD:R_1206, F.Cu at (248.0, 55.8)
- added R74: 100, Resistors_SMD:R_0805, F.Cu at (230.8, 83.9)
- added R75: 0.002, Resistors_SMD:R_1206, F.Cu at (250.0, 42.4)
- added R76: 10, Resistors_SMD:R_1206, F.Cu at (233.0, 71.1)
- added R77: 10, Resistors_SMD:R_1206, F.Cu at (242.9, 64.9)
- added R78: 10k, Resistors_SMD:R_0805, F.Cu at (263.8, 61.5)
- added R79: 0.150 1/2W, Resistors_SMD:R_1206, F.Cu at (262.0, 148.8)
- added R8: 1k, Resistors_SMD:R_0805, F.Cu at (348.9, 135.6)
- added R80: 220k, Resistors_SMD:R_0805, F.Cu at (298.2, 143.0)
- added R81: 12k, Resistors_SMD:R_0805, F.Cu at (291.3, 145.3)
- added R82: 220k, Resistors_SMD:R_0805, F.Cu at (301.9, 136.3)
- added R83: 10k, Resistors_SMD:R_0805, F.Cu at (297.9, 136.7)
- added R84: 1k, Resistors_SMD:R_0805, F.Cu at (279.8, 147.0)
- added R85: 3k, Resistors_SMD:R_0805, F.Cu at (294.3, 138.9)
- added R86: 10k, Resistors_SMD:R_0805, F.Cu at (340.7, 99.1)
- added R87: 255, Resistors_SMD:R_0805, F.Cu at (344.0, 105.4)
- added R88: 10k, Resistors_SMD:R_0805, F.Cu at (381.9, 54.8)
- added R89: 120, Resistors_SMD:R_0805, F.Cu at (386.2, 42.2)
- added R9: 1k, Resistors_SMD:R_0805, F.Cu at (345.2, 142.9)
- added R90: 10k, Resistors_SMD:R_0805, F.Cu at (378.3, 51.3)
- added R91: 10k, Resistors_SMD:R_0805, F.Cu at (374.6, 51.3)
- added R92: 330, Resistors_SMD:R_0805, F.Cu at (382.5, 42.2)
- added R93: 330, Resistors_SMD:R_0805, F.Cu at (369.4, 57.6)
- added R94: 10k, Resistors_SMD:R_0805, F.Cu at (382.5, 48.5)
- added R95: 10k, Resistors_SMD:R_0805, F.Cu at (365.7, 57.6)
- added R96: 10k, Resistors_SMD:R_0805, F.Cu at (371.0, 51.3)
- added R97: 10k, Resistors_SMD:R_0805, F.Cu at (362.1, 56.7)
- added R98: 10k, Resistors_SMD:R_0805, F.Cu at (207.3, 138.5)
- added R99: 1k, Resistors_SMD:R_0805, F.Cu at (196.6, 143.3)
- added U1: 74LVC00, Housings_SSOP:TSSOP-14_4.4x5mm_Pitch0.65mm, F.Cu at (313.4, 131.4)
- added U10: IRS2304, Housings_SOIC:SOIC-8_3.9x4.9mm_Pitch1.27mm, F.Cu at (206.1, 109.2)
- added U11: ZXCT1082, TO_SOT_Packages_SMD:SOT-23-5, F.Cu at (197.3, 127.6)
- added U12: IRS2304, Housings_SOIC:SOIC-8_3.9x4.9mm_Pitch1.27mm, F.Cu at (197.2, 119.5)
- added U13: LM2903, Housings_SSOP:TSSOP-8_4.4x3mm_Pitch0.65mm, F.Cu at (185.1, 83.0)
- added U14: IRS2304, Housings_SOIC:SOIC-8_3.9x4.9mm_Pitch1.27mm, F.Cu at (238.7, 43.6)
- added U15: ZXCT1082, TO_SOT_Packages_SMD:SOT-23-5, F.Cu at (230.9, 51.8)
- added U16: IRS2304, Housings_SOIC:SOIC-8_3.9x4.9mm_Pitch1.27mm, F.Cu at (209.6, 80.8)
- added U17: LM2903, Housings_SSOP:TSSOP-8_4.4x3mm_Pitch0.65mm, F.Cu at (193.4, 83.0)
- added U18: IRS2304, Housings_SOIC:SOIC-8_3.9x4.9mm_Pitch1.27mm, F.Cu at (230.8, 43.6)
- added U19: ZXCT1082, TO_SOT_Packages_SMD:SOT-23-5, F.Cu at (222.0, 62.1)
- added U2: 74LVC08, Housings_SSOP:TSSOP-14_4.4x5mm_Pitch0.65mm, F.Cu at (330.1, 131.4)
- added U20: IRS2304, Housings_SOIC:SOIC-8_3.9x4.9mm_Pitch1.27mm, F.Cu at (221.9, 53.9)
- added U21: MIC2619, TO_SOT_Packages_SMD:SOT-23-6, F.Cu at (281.7, 139.9)
- added U22: MC34063, Housings_SOIC:SOIC-8_3.9x4.9mm_Pitch1.27mm, F.Cu at (283.0, 131.4)
- added U23: LD1117S33CTR, TO_SOT_Packages_SMD:SOT-223, F.Cu at (263.0, 140.6)
- added U24: CAT25160_EEPROM, Housings_SSOP:TSSOP-8_4.4x3mm_Pitch0.65mm, F.Cu at (325.4, 103.0)
- added U25: STM32F373RBTx, Housings_QFP:LQFP-64_10x10mm_Pitch0.5mm, F.Cu at (324.8, 91.2)
- added U26: SN65HVD1050D, Housings_SOIC:SOIC-8_3.9x4.9mm_Pitch1.27mm, F.Cu at (374.6, 43.6)
- added U27: SN74LVC245ADBR, Housings_SSOP:SSOP-20_5.3x7.2mm_Pitch0.65mm, F.Cu at (187.8, 141.2)
- added U28: SN74HC20, Housings_SSOP:TSSOP-14_4.4x5mm_Pitch0.65mm, F.Cu at (273.6, 105.0)
- added U29: SN74HC02, Housings_SSOP:TSSOP-14_4.4x5mm_Pitch0.65mm, F.Cu at (261.3, 108.0)
- added U3: 74LVC00, Housings_SSOP:TSSOP-14_4.4x5mm_Pitch0.65mm, F.Cu at (321.7, 131.4)
- added U30: SN74HC132, Housings_SSOP:TSSOP-14_4.4x5mm_Pitch0.65mm, F.Cu at (276.6, 95.8)
- added U31: MAX232, Housings_SSOP:TSSOP-16_4.4x5mm_Pitch0.65mm, F.Cu at (275.4, 72.9)
- added U32: MAX232, Housings_SSOP:TSSOP-16_4.4x5mm_Pitch0.65mm, F.Cu at (297.2, 43.7)
- added U33: NCV1124, Housings_SOIC:SOIC-8_3.9x4.9mm_Pitch1.27mm, F.Cu at (305.3, 43.6)
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Connections:
- P1 pad 1: Net-(P1-Pad1) -> /+12V_BatR
- P1 pad 10: Net-(P1-Pad10) -> ~ParkbrakeSwitch_inverted
- P1 pad 11: Net-(P1-Pad11) -> LeftRearMotor+
- P1 pad 12: Net-(P1-Pad12) -> LeftRearMotor+
- P1 pad 13: Net-(P1-Pad13) -> BrakeLights
- P1 pad 14: Net-(P1-Pad14) -> LeftRearMotor-
- P1 pad 15: Net-(P1-Pad15) -> LeftRearMotor-
- P1 pad 16: Net-(P1-Pad16) -> GNDPWR
- P1 pad 17: Net-(P1-Pad17) -> GNDPWR
- P1 pad 18: Net-(P1-Pad18) -> GNDPWR
- P1 pad 19: Net-(P1-Pad19) -> GNDPWR
- P1 pad 2: Net-(P1-Pad2) -> /+12V_BatR
- P1 pad 20: Net-(P1-Pad20) -> GNDPWR
- P1 pad 21: Net-(P1-Pad21) -> GNDPWR
- P1 pad 22: Net-(P1-Pad22) -> /+12V_BatF
- P1 pad 23: Net-(P1-Pad23) -> /+12V_BatF
- P1 pad 24: Net-(P1-Pad24) -> /+12V_BatF
- P1 pad 25: Net-(P1-Pad25) -> L_wheelsensor_out+
- P1 pad 26: Net-(P1-Pad26) -> LeftFrontMotor-
- P1 pad 27: Net-(P1-Pad27) -> LeftFrontMotor-
- P1 pad 28: Net-(P1-Pad28) -> L_wheelsensor_out-
- P1 pad 29: Net-(P1-Pad29) -> RightFrontMotor-
- P1 pad 3: Net-(P1-Pad3) -> /+12V_BatR
- P1 pad 30: Net-(P1-Pad30) -> RightFrontMotor-
- P1 pad 31: Net-(P1-Pad31) -> RF_wheelsensor_in+
- P1 pad 32: Net-(P1-Pad32) -> LeftFrontMotor+
- P1 pad 33: Net-(P1-Pad33) -> LeftFrontMotor+
- P1 pad 34: Net-(P1-Pad34) -> RF_wheelsensor_in-
- P1 pad 35: Net-(P1-Pad35) -> RightFrontMotor+
- P1 pad 36: Net-(P1-Pad36) -> RightFrontMotor+
- P1 pad 37: Net-(P1-Pad37) -> LF_wheelsensor_in-
- P1 pad 38: Net-(P1-Pad38) -> LF_wheelsensor_in+
- P1 pad 39: Net-(P1-Pad39) -> R_wheelsensor_out+
- P1 pad 4: Net-(P1-Pad4) -> Parkbrake_indicator_lamp
- P1 pad 40: Net-(P1-Pad40) -> LR_wheelsensor_in-
- P1 pad 41: Net-(P1-Pad41) -> RR_wheelsensor_in+
- P1 pad 42: Net-(P1-Pad42) -> R_wheelsensor_out-
- P1 pad 43: Net-(P1-Pad43) -> LR_wheelsensor_in-
- P1 pad 44: Net-(P1-Pad44) -> LR_wheelsensor_in+
- P1 pad 45: Net-(P1-Pad45) -> CAN_HI
- P1 pad 46: Net-(P1-Pad46) -> LR_wheelsensor_in-
- P1 pad 47: Net-(P1-Pad47) -> +12V_ign_in
- P1 pad 48: Net-(P1-Pad48) -> CAN_LO
- P1 pad 5: Net-(P1-Pad5) -> RightRearMotor+
- P1 pad 6: Net-(P1-Pad6) -> RightRearMotor+
- P1 pad 7: Net-(P1-Pad7) -> ParkbrakeSwitch_non_invert
- P1 pad 8: Net-(P1-Pad8) -> RightRearMotor-
- P1 pad 9: Net-(P1-Pad9) -> RightRearMotor-
Other:
- board size 109.2 x 114.3 mm -> 101.6 x 114.3 mm

Commit message: some more work on parkbrake pcb
Parts:
- C8, D15, Q10, Q14, Q16, Q4, Q8, R11, R21, R22, R38, R39, U5, VR2: moved to B.Cu
- R14, R15, R25, R26, R31, R32, R42, R43, R48, R49, R59, R60, R65, R66, R76, R77: footprint Resistors_SMD:R_1206 -> Resistors_SMD:R_0805
- moved R17 116.7 mm to (143.5, 66.8), turned to 180 degrees
- moved R31 115.8 mm to (145.5, 142.2)
- moved D2 114.8 mm to (171.7, 55.6)
- moved R4 113.9 mm to (165.6, 54.9), turned to 180 degrees
- moved R2 110.8 mm to (169.4, 55.6), turned to 270 degrees
- moved R11 109.8 mm to (143.5, 67.1), turned to 180 degrees
- moved C6 109.4 mm to (146.3, 69.3)
- moved C15 100.5 mm to (143.5, 54.9), turned to 180 degrees
- moved R27 97.9 mm to (148.8, 59.2)
- moved C5 97.0 mm to (150.1, 85.3), turned to 270 degrees
- moved VR2 94.3 mm to (172.7, 71.4)
- moved C11 93.2 mm to (150.1, 68.6), turned to 90 degrees
- moved R25 91.7 mm to (161.8, 64.8), turned to 90 degrees
- moved R16 91.0 mm to (158.2, 72.9)
- moved R24 89.4 mm to (174.2, 71.4), turned to 0 degrees
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Connections:
- C11 pad 2: +12V_Feed -> +12V_powerRear
- C12 pad 1: +12V_Feed -> +12V_powerRear
- C16 pad 1: LR_wheelsensor_in- -> GNDPWR
- C18 pad 2: +12V_Feed -> +12V_powerRear
- C19 pad 1: +12V_Feed -> +12V_powerFront
- C23 pad 1: LR_wheelsensor_in- -> GNDPWR
- C25 pad 2: +12V_Feed -> +12V_powerFront
- C26 pad 1: +12V_Feed -> +12V_powerFront
- C30 pad 1: LR_wheelsensor_in- -> GNDPWR
- C32 pad 2: +12V_Feed -> +12V_powerFront
- C5 pad 1: +12V_Feed -> +12V_powerRear
- C9 pad 1: LR_wheelsensor_in- -> GNDPWR
- D14 pad 1: Net-(D14-Pad1) -> Net-(C7-Pad2)
- D14 pad 2: +12V_Feed -> +12V_powerRear
- D16 pad 2: +12V_Feed -> +12V_powerRear
- D17 pad 2: +12V_Feed -> +12V_powerRear
- D19 pad 2: +12V_Feed -> +12V_powerRear
- D20 pad 2: +12V_Feed -> +12V_powerFront
- D22 pad 2: +12V_Feed -> +12V_powerFront
- D23 pad 2: +12V_Feed -> +12V_powerFront
- D25 pad 2: +12V_Feed -> +12V_powerFront
- P1 pad 1: /+12V_BatR -> BrakeLights
- P1 pad 11: LeftRearMotor+ -> LeftRearMotor-
- P1 pad 12: LeftRearMotor+ -> LeftRearMotor-
- P1 pad 13: BrakeLights -> /+12V_BatR
- P1 pad 14: LeftRearMotor- -> /+12V_BatR
- P1 pad 15: LeftRearMotor- -> /+12V_BatR
- P1 pad 2: /+12V_BatR -> RightRearMotor+
- P1 pad 3: /+12V_BatR -> RightRearMotor+
- P1 pad 4: Parkbrake_indicator_lamp -> ParkbrakeSwitch_non_invert
- P1 pad 5: RightRearMotor+ -> RightRearMotor-
- P1 pad 6: RightRearMotor+ -> RightRearMotor-
- P1 pad 7: ParkbrakeSwitch_non_invert -> Parkbrake_indicator_lamp
- P1 pad 8: RightRearMotor- -> LeftRearMotor+
- P1 pad 9: RightRearMotor- -> LeftRearMotor+
- Q10 pad 2: LeftRearMotor- -> Net-(Q10-Pad2)
- Q10 pad 3: Net-(Q10-Pad3) -> LeftRearMotor-
- Q11 pad 2: Net-(Q11-Pad2) -> LeftRearMotor-
- Q11 pad 3: LeftRearMotor- -> Net-(Q11-Pad3)
- Q16 pad 2: RightRearMotor- -> Net-(Q14-Pad2)
- Q16 pad 3: Net-(Q14-Pad2) -> RightRearMotor-
- Q17 pad 2: Net-(Q15-Pad3) -> RightRearMotor-
- Q17 pad 3: RightRearMotor- -> Net-(Q15-Pad3)
- Q22 pad 2: LeftFrontMotor- -> Net-(Q20-Pad2)
- Q22 pad 3: Net-(Q20-Pad2) -> LeftFrontMotor-
- Q23 pad 2: Net-(Q21-Pad3) -> LeftFrontMotor-
- Q23 pad 3: LeftFrontMotor- -> Net-(Q21-Pad3)
- Q28 pad 2: RightFrontMotor- -> Net-(Q26-Pad2)
- Q28 pad 3: Net-(Q26-Pad2) -> RightFrontMotor-
- Q29 pad 2: Net-(Q27-Pad3) -> RightFrontMotor-
- Q29 pad 3: RightFrontMotor- -> Net-(Q27-Pad3)
- Q7 pad 3: Net-(D14-Pad1) -> Net-(C7-Pad2)
- Q8 pad 2: Net-(Q10-Pad3) -> Net-(Q10-Pad2)
- Q9 pad 3: Net-(Q11-Pad2) -> Net-(Q11-Pad3)
- R14 pad 2: Net-(D14-Pad1) -> Net-(R14-Pad2)
- R16 pad 2: Net-(Q11-Pad2) -> Net-(Q11-Pad3)
- R18 pad 2: LR_wheelsensor_in- -> GNDPWR
- R19 pad 2: Net-(Q10-Pad3) -> Net-(Q10-Pad2)
- R20 pad 1: Net-(Q11-Pad2) -> Net-(Q11-Pad3)
- R21 pad 2: Net-(Q10-Pad3) -> Net-(Q10-Pad2)
- R22 pad 2: Net-(Q10-Pad3) -> Net-(Q10-Pad2)
- R24 pad 1: Net-(Q11-Pad2) -> Net-(Q11-Pad3)
- R35 pad 2: LR_wheelsensor_in- -> GNDPWR
- R52 pad 2: LR_wheelsensor_in- -> GNDPWR
- R69 pad 2: LR_wheelsensor_in- -> GNDPWR
- U10 pad 3: +12V_Feed -> +12V_powerRear
- U11 pad 2: LR_wheelsensor_in- -> GNDPWR
- U12 pad 3: +12V_Feed -> +12V_powerRear
- U14 pad 3: +12V_Feed -> +12V_powerFront
- U15 pad 2: LR_wheelsensor_in- -> GNDPWR
- U16 pad 3: +12V_Feed -> +12V_powerFront
- U18 pad 3: +12V_Feed -> +12V_powerFront
- U19 pad 2: LR_wheelsensor_in- -> GNDPWR
- U20 pad 3: +12V_Feed -> +12V_powerFront
- U6 pad 3: +12V_Feed -> +12V_powerRear
- U6 pad 7: Net-(D14-Pad1) -> Net-(R14-Pad2)
- U7 pad 2: LR_wheelsensor_in- -> GNDPWR
- U8 pad 3: +12V_Feed -> +12V_powerRear
Routing:
- net GNDPWR: track 0.00 -> 182.4 mm, vias 0 -> 5
- net RightRearMotor+: track 0.00 -> 170.3 mm, vias 0 -> 10
- net +12V_powerRear: track 0.00 -> 168.3 mm, vias 0 -> 7
- net LeftRearMotor+: track 0.00 -> 159.4 mm, vias 0 -> 10
- net RightRearMotor-: track 0.00 -> 136.6 mm, vias 0 -> 10
- net LeftRearMotor-: track 0.00 -> 59.9 mm, vias 0 -> 5
- net /H-Bridge_logic/H-BridgeRear/LeftRearLo+: track 0.00 -> 59.7 mm
- net /H-Bridge_logic/H-BridgeRear/LeftRearHI+: track 0.00 -> 59.1 mm
- net Net-(Q10-Pad2): track 0.00 -> 36.4 mm, vias 0 -> 1
- net Net-(Q14-Pad2): track 0.00 -> 35.2 mm
- net Net-(Q11-Pad3): track 0.00 -> 34.2 mm
- net /+12V_BatR: track 0.00 -> 24.3 mm
- net ~LeftRear_CL: track 0.00 -> 24.1 mm, vias 0 -> 1
- net LeftRear_CS: track 0.00 -> 22.9 mm, vias 0 -> 1
- net Net-(Q15-Pad3): track 0.00 -> 22.4 mm
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Other:
- net class highpwr added: clearance 0.2, trace_width 2.5, via_dia 2.5, via_drill 2
- net class pwr added: clearance 0.2, trace_width 1.5, via_dia 1.8, via_drill 1.5
- net class subpwr added: clearance 0.2, trace_width 0.8, via_dia 1, via_drill 0.8
- net class tiny added: clearance 0.2, trace_width 0.25, via_dia 0.6, via_drill 0.4

Commit message: more work on parkbrake ecu Rear H-bridge more or less finished
Parts:
- removed R103: 2.2k, Resistors_SMD:R_0805
- added R118: 10k, Resistors_SMD:R_0805, F.Cu at (130.0, 128.3)
- added R119: 10k, Resistors_SMD:R_0805, B.Cu at (142.7, 91.9)
- added R120: 10k, Resistors_SMD:R_0805, B.Cu at (142.7, 95.2)
- C3, C4, D18, Q3, R28, R34, R7, U9, VR1: moved to B.Cu
- R10: footprint Resistors_SMD:R_Array_Concave_4x0603 -> Resistors_SMD:R_0805
- moved R10 225.4 mm to (120.9, 114.8)
- moved C4 215.3 mm to (142.5, 82.0)
- moved R9 211.9 mm to (152.1, 55.6), turned to 270 degrees
- moved C3 211.6 mm to (142.5, 89.9)
- moved R7 201.3 mm to (159.3, 55.9), turned to 90 degrees
- moved D9 200.4 mm to (160.8, 56.6), turned to 180 degrees
- moved D13 199.6 mm to (148.8, 56.9), turned to 180 degrees
- moved D8 193.0 mm to (160.8, 54.9)
- moved D12 189.4 mm to (148.8, 54.9)
- moved D1 184.6 mm to (82.3, 55.4), turned to 270 degrees
- moved U3 183.0 mm to (142.7, 93.5), turned to 180 degrees
- moved U4 179.2 mm to (142.7, 85.9), turned to 180 degrees
- moved R1 178.3 mm to (84.8, 55.4), turned to 270 degrees
- moved R3 168.3 mm to (89.4, 56.6)
- moved VR1 159.8 mm to (81.5, 72.4), turned to 180 degrees
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Connections:
- D36 pad 1: Net-(D36-Pad1) -> (no net)
- R104 pad 2: LR_wheelsensor_in- -> BRAKELIGHTS_ON_SIGNAL
- R104 pad 3: (no net) -> PARKBRAKE_NON_INVERT_SIGNAL
- R104 pad 4: (no net) -> ~PARKBRAKE_INVERT_SIGNAL
- R104 pad 5: (no net) -> LR_wheelsensor_in-
- R104 pad 6: (no net) -> LR_wheelsensor_in-
- R104 pad 7: (no net) -> LR_wheelsensor_in-
- R104 pad 8: (no net) -> LR_wheelsensor_in-
- R110 pad 2: /Wheelsensors/L_sensor_interpolated_out+ -> LR_wheelsensor_in-
- R110 pad 3: (no net) -> LR_wheelsensor_in-
- R110 pad 4: (no net) -> LR_wheelsensor_in-
- R110 pad 5: (no net) -> /Wheelsensors/R_sensor_interpolated_out-
- R110 pad 6: (no net) -> /Wheelsensors/R_sensor_interpolated_out+
- R110 pad 7: (no net) -> /Wheelsensors/L_sensor_interpolated_out-
- R110 pad 8: (no net) -> /Wheelsensors/L_sensor_interpolated_out+
- U10 pad 1: /H-Bridge_logic/H-BridgeRear/RightRearHI+ -> /H-Bridge_logic/H-BridgeRear/RightRearHi-
- U12 pad 1: /H-Bridge_logic/H-BridgeRear/RightRearHi- -> /H-Bridge_logic/H-BridgeRear/RightRearHI+
- U4 pad 11: /H-Bridge_logic/H-BridgeRear/RightRearHI+ -> /H-Bridge_logic/H-BridgeRear/RightRearHi-
- U4 pad 8: /H-Bridge_logic/H-BridgeRear/RightRearHi- -> /H-Bridge_logic/H-BridgeRear/RightRearHI+
Routing:
- net GNDPWR: track 182.4 -> 392.1 mm, vias 5 -> 15
- net +12V_powerFront: track 0.00 -> 79.3 mm
- net +12V_powerRear: track 168.3 -> 223.9 mm, vias 7 -> 11
- net gate_drive_24V: track 11.0 -> 65.0 mm, vias 0 -> 4
- net +3.3V: track 4.68 -> 58.4 mm, vias 0 -> 4
- net /H-Bridge_logic/H-BridgeRear/RightRearHI+: track 0.00 -> 48.8 mm, vias 0 -> 3
- net /H-Bridge_logic/H-BridgeRear/RightRearHi-: track 0.00 -> 46.0 mm, vias 0 -> 3
- net LR_wheelsensor_in-: track 0.00 -> 37.7 mm, vias 0 -> 3
- net RightRearMotor-: track 136.6 -> 166.7 mm
- net LeftRear_Loosen: track 0.00 -> 28.5 mm
- net RightRearMotor+: track 170.3 -> 198.7 mm
- net RightRear_CS: track 0.00 -> 26.5 mm, vias 0 -> 1
- net Net-(Q2-Pad3): track 0.00 -> 25.7 mm
- net LeftRear_Tighten: track 0.00 -> 25.4 mm
- net /+12V_BatF: track 0.00 -> 24.5 mm
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
Commit message: Front motors H-bridge finished
Parts:
- C27, D21, JP6, JP7, JP8, Q21, Q23, Q27, Q29, R49, R50, R51, R54, R58, R65, R66, R67, R71, R75, R76, R77, U31, U32: moved to B.Cu
- Q3, VR1: moved to F.Cu
- moved C77 267.5 mm to (57.9, 57.9), turned to 90 degrees
- moved C79 259.1 mm to (60.5, 62.5), turned to 90 degrees
- moved R8 258.6 mm to (103.1, 55.4), turned to 270 degrees
- moved R6 255.3 mm to (99.1, 55.6), turned to 270 degrees
- moved C75 254.6 mm to (54.6, 57.1)
- moved C2 254.4 mm to (83.3, 134.9), turned to 270 degrees
- moved D7 251.3 mm to (95.8, 56.9)
- moved C80 248.7 mm to (60.5, 57.9), turned to 270 degrees
- moved C74 246.2 mm to (55.1, 60.7), turned to 90 degrees
- moved C78 246.1 mm to (58.2, 54.6)
- moved D11 245.9 mm to (106.4, 56.6)
- moved C1 245.4 mm to (96.0, 138.7)
- moved D6 244.0 mm to (95.8, 54.9), turned to 180 degrees
- moved U2 242.7 mm to (87.4, 133.1), turned to 90 degrees
- moved U32 242.0 mm to (57.4, 75.9)
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Connections:
- D20 pad 1: Net-(D20-Pad1) -> Net-(C21-Pad2)
- P1 pad 29: RightFrontMotor- -> LeftFrontMotor+
- P1 pad 30: RightFrontMotor- -> LeftFrontMotor+
- P1 pad 31: RF_wheelsensor_in+ -> LF_wheelsensor_in+
- P1 pad 32: LeftFrontMotor+ -> RightFrontMotor-
- P1 pad 33: LeftFrontMotor+ -> RightFrontMotor-
- P1 pad 34: RF_wheelsensor_in- -> LF_wheelsensor_in-
- P1 pad 37: LF_wheelsensor_in- -> RF_wheelsensor_in-
- P1 pad 38: LF_wheelsensor_in+ -> RF_wheelsensor_in+
- Q19 pad 3: Net-(D20-Pad1) -> Net-(C21-Pad2)
- R48 pad 2: Net-(D20-Pad1) -> Net-(R48-Pad2)
- U14 pad 7: Net-(D20-Pad1) -> Net-(R48-Pad2)
Routing:
- net +12V_powerFront: track 79.3 -> 259.6 mm, vias 0 -> 11
- net GNDPWR: track 392.1 -> 567.4 mm, vias 15 -> 27
- net RightFrontMotor+: track 0.00 -> 160.4 mm, vias 0 -> 12
- net RightFrontMotor-: track 0.00 -> 139.2 mm, vias 0 -> 11
- net LeftFrontMotor+: track 0.00 -> 116.3 mm, vias 0 -> 10
- net +3.3V: track 58.4 -> 157.4 mm, vias 4 -> 9
- net LR_wheelsensor_in-: track 37.7 -> 135.1 mm, vias 3 -> 7
- net /H-Bridge_logic/H-BridgeFront/LeftFrontHI+: track 0.00 -> 96.6 mm, vias 0 -> 3
- net /H-Bridge_logic/H-BridgeFront/LeftFrontLo+: track 0.00 -> 96.1 mm, vias 0 -> 3
- net LeftFrontMotor-: track 0.00 -> 86.0 mm, vias 0 -> 10
- net ~LeftFront_CL: track 0.00 -> 75.5 mm, vias 0 -> 2
- net LeftFront_CS: track 0.00 -> 75.0 mm, vias 0 -> 2
- net gate_drive_24V: track 65.0 -> 136.2 mm, vias 4 -> 8
- net /H-Bridge_logic/H-BridgeFront/RightFrontHi-: track 0.00 -> 56.3 mm, vias 0 -> 3
- net /H-Bridge_logic/H-BridgeFront/RightFrontHI+: track 0.00 -> 48.3 mm, vias 0 -> 3
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
Commit message: More work on inputs and 5 volt
Parts:
- added R103: 2.2k, Resistors_SMD:R_Array_Concave_4x0603, F.Cu at (127.7, 60.4)
- C35, C37, C39, C65, C66, C67, C68, C71, C74, C75, C76, C77, C79, C83, C84, C85, C86, C87, C90, D30, D31, D32, D33, D5, JP12, JP13, JP14, Q31, Q5, Q6, R102, R104, R110, R115, R116, R5, R80, R81, R82, R83, U21, U27, U29, U30, U33, U34, U35, VR3: moved to B.Cu
- U31: moved to F.Cu
- moved R88 275.2 mm to (110.8, 101.9), turned to 90 degrees
- moved R89 273.0 mm to (118.7, 96.9), turned to 270 degrees
- moved U26 266.7 mm to (114.9, 103.9), turned to 90 degrees
- moved R82 254.0 mm to (51.4, 94.1)
- moved C59 253.2 mm to (118.7, 100.9), turned to 270 degrees
- moved C57 252.1 mm to (110.7, 105.5), turned to 90 degrees
- moved R80 252.0 mm to (51.5, 91.8)
- moved JP2 248.7 mm to (112.1, 109.7)
- moved R83 246.0 mm to (55.0, 98.0), turned to 180 degrees
- moved R81 244.4 mm to (51.1, 100.5), turned to 180 degrees
- moved C33 238.9 mm to (59.7, 98.0)
- moved U21 234.4 mm to (51.2, 97.2), turned to 90 degrees
- moved R115 229.1 mm to (110.0, 65.7), turned to 90 degrees
- moved C37 225.2 mm to (55.1, 100.4)
- moved L1 224.8 mm to (54.5, 86.6)
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Connections:
- C41 pad 1: (no net) -> Net-(C41-Pad1)
- C69 pad 1: 3.3V -> +3.3V
- C70 pad 1: 3.3V -> +3.3V
- C71 pad 1: 3.3V -> +3.3V
- C72 pad 1: 3.3V -> +3.3V
- C73 pad 1: 3.3V -> +3.3V
- D35 pad 1: (no net) -> Net-(D35-Pad1)
- D36 pad 1: (no net) -> Net-(D36-Pad1)
- D37 pad 1: (no net) -> Net-(D37-Pad1)
- D38 pad 1: (no net) -> Net-(D38-Pad1)
- P1 pad 1: BrakeLights -> ParkbrakeSwitch_non_invert
- P1 pad 10: ~ParkbrakeSwitch_inverted -> Parkbrake_indicator_lamp
- P1 pad 4: ParkbrakeSwitch_non_invert -> ~ParkbrakeSwitch_inverted
- P1 pad 7: Parkbrake_indicator_lamp -> BrakeLights
- R104 pad 3: PARKBRAKE_NON_INVERT_SIGNAL -> ~PARKBRAKE_INVERT_SIGNAL
- R104 pad 4: ~PARKBRAKE_INVERT_SIGNAL -> PARKBRAKE_NON_INVERT_SIGNAL
- R110 pad 5: /Wheelsensors/R_sensor_interpolated_out- -> /Wheelsensors/L_sensor_interpolated_out-
- R110 pad 6: /Wheelsensors/R_sensor_interpolated_out+ -> /Wheelsensors/L_sensor_interpolated_out+
- R110 pad 7: /Wheelsensors/L_sensor_interpolated_out- -> /Wheelsensors/R_sensor_interpolated_out-
- R110 pad 8: /Wheelsensors/L_sensor_interpolated_out+ -> /Wheelsensors/R_sensor_interpolated_out+
- R86 pad 1: 3.3V -> +3.3V
- U25 pad 1: (no net) -> Net-(U25-Pad1)
- U27 pad 17: (no net) -> Net-(U27-Pad17)
- U27 pad 3: (no net) -> Net-(U27-Pad3)
- U31 pad 10: L_speed_out+ -> L_speed_out-
- U31 pad 11: L_speed_out- -> L_speed_out+
- U31 pad 12: (no net) -> Net-(U31-Pad12)
- U31 pad 14: Net-(C80-Pad1) -> Net-(C78-Pad1)
- U31 pad 7: Net-(C78-Pad1) -> Net-(C80-Pad1)
- U31 pad 9: (no net) -> Net-(U31-Pad9)
- U32 pad 12: (no net) -> Net-(U32-Pad12)
- U32 pad 9: (no net) -> Net-(U32-Pad9)
- U35 pad 1: /Wheelsensors/LF_5to3.3 -> /Wheelsensors/RF_5to3.3
- U35 pad 10: /Wheelsensors/LR_5to3.3 -> /Wheelsensors/RR_5to3.3
- U35 pad 11: RR_speed_in -> LR_speed_in
- U35 pad 12: /Wheelsensors/RR_5to3.3 -> /Wheelsensors/LR_5to3.3
- U35 pad 13: /Wheelsensors/RR_5to3.3 -> /Wheelsensors/LR_5to3.3
- U35 pad 2: /Wheelsensors/LF_5to3.3 -> /Wheelsensors/RF_5to3.3
- U35 pad 3: LF_speed_in -> RF_speed_in
- U35 pad 4: /Wheelsensors/RF_5to3.3 -> /Wheelsensors/LF_5to3.3
- U35 pad 5: /Wheelsensors/RF_5to3.3 -> /Wheelsensors/LF_5to3.3
- U35 pad 6: RF_speed_in -> LF_speed_in
- U35 pad 8: LR_speed_in -> RR_speed_in
- U35 pad 9: /Wheelsensors/LR_5to3.3 -> /Wheelsensors/RR_5to3.3
Routing:
- net LR_wheelsensor_in-: track 135.1 -> 577.0 mm, vias 7 -> 23
- net +5V: track 0.00 -> 151.1 mm, vias 0 -> 7
- net +3.3V: track 157.4 -> 278.8 mm, vias 9 -> 14
- net ~PARKBRAKE_INVERT_SIGNAL: track 0.00 -> 69.0 mm, vias 0 -> 3
- net CAN_LO: track 0.00 -> 63.5 mm
- net CAN_HI: track 0.00 -> 62.3 mm
- net IGN_ON_SIGNAL: track 0.00 -> 61.7 mm, vias 0 -> 2
- net BRAKELIGHTS_ON_SIGNAL: track 0.00 -> 61.6 mm, vias 0 -> 1
- net PARKBRAKE_NON_INVERT_SIGNAL: track 0.00 -> 61.4 mm, vias 0 -> 3
- net +12V_Feed: track 0.00 -> 59.4 mm, vias 0 -> 8
- net LF_speed_in: track 0.00 -> 57.6 mm
- net PARKBRAKE_INVERT_CHECK_SIGNAL: track 0.00 -> 57.4 mm, vias 0 -> 2
- net RF_speed_in: track 0.00 -> 55.5 mm
- net RR_speed_in: track 0.00 -> 49.3 mm
- net LR_speed_in: track 0.00 -> 47.1 mm
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