File: electronics/Parkbrake/buttonlogic.sch (KiCad schematic (older format))
At the start: 33 parts, among them Q32 NTS4173, U28 SN74HC20, U29 SN74HC02, U30 SN74HC132

Commit message: More work on inputs and 5 volt
Parts:
- R103: footprint (none) -> Resistors_SMD:R_Array_Concave_4x0603
Connections:
- net BRAKELIGHTS_ON_SIGNAL: now also R103.6; no longer R103.7
- net GND: now also R104.5, R104.6; no longer R104.5, R104.6
- net IGN_ON_SIGNAL: now also R103.5; no longer R103.8
- net PARKBRAKE_NON_INVERT_SIGNAL: now also R103.8, R104.4; no longer R103.6, R104.3
- net ~PARKBRAKE_INVERT_SIGNAL: now also R103.7, R104.3; no longer R103.5, R104.4
- net at D35.1 (K): now also R103.4; no longer R103.1
- net at D36.1 (K): now also R103.3; no longer R103.2
- net at D37.1 (K): now also R103.1; no longer R103.3
- net at D38.1 (K): now also R103.2; no longer R103.4
- net 3.3V renamed +3.3V
Changed lines of the file:
@@
 	5825 4400 5825 4650
 Text GLabel 6125 4100 1    60   Input ~ 0
-3.3V
++3.3V
 Wire Wire Line
 	5825 3250 5825 3450
@@
 	6125 3250 6125 3450
 Text GLabel 6125 2950 1    60   Input ~ 0
-3.3V
++3.3V
 Wire Wire Line
 	6425 3250 6425 3450
@@
 $EndComp
 Text GLabel 4700 5775 1    60   Input ~ 0
-3.3V
++3.3V
 Wire Wire Line
 	4350 5775 4975 5775
@@
 $Comp
 L Rnet4 R103
-U 2 1 57948BBF
+U 3 1 57948BBF
 P 1100 4000
 F 0 "R103" H 1100 4080 50  0000 C CNN
 F 1 "2.2k" H 1100 4000 50  0000 C CNN
-F 2 "" H 1100 3930 50  0000 C CNN
+F 2 "Resistors_SMD:R_Array_Concave_4x0603" H 1100 3930 50  0001 C CNN
 F 3 "" V 1100 4000 50  0000 C CNN
 F 4 "EXB38V222JV" H 1100 4000 60  0001 C CNN "part"
 F 5 "2060102" H 1100 4000 60  0001 C CNN "farnell"
-	2    1100 4000
+	3    1100 4000
 	0    1    1    0
 $EndComp
 $Comp
 L Rnet4 R103
-U 3 1 579490A2
+U 1 1 579490A2
 P 1100 5000
 F 0 "R103" H 1100 5080 50  0000 C CNN
 F 1 "2.2k" H 1100 5000 50  0000 C CNN
-F 2 "" H 1100 4930 50  0000 C CNN
+F 2 "Resistors_SMD:R_Array_Concave_4x0603" H 1100 4930 50  0001 C CNN
 F 3 "" V 1100 5000 50  0000 C CNN
-	3    1100 5000
+	1    1100 5000
 	0    1    1    0
 $EndComp
 $Comp
 L Rnet4 R103
-U 1 1 579493FA
+U 4 1 579493FA
 P 1100 2750
 F 0 "R103" H 1100 2830 50  0000 C CNN
@@
 F 4 "EXB38V222JV" H 1100 2750 60  0001 C CNN "part"
 F 5 "2060102" H 1100 2750 60  0001 C CNN "farnell"
-	1    1100 2750
+	4    1100 2750
 	0    1    1    0
 $EndComp
 $Comp
 L Rnet4 R103
-U 4 1 579498BE
+U 2 1 579498BE
 P 1100 6000
 F 0 "R103" H 1100 6080 50  0000 C CNN
 F 1 "2.2k" H 1100 6000 50  0000 C CNN
-F 2 "" H 1100 5930 50  0000 C CNN
+F 2 "Resistors_SMD:R_Array_Concave_4x0603" H 1100 5930 50  0001 C CNN
 F 3 "" V 1100 6000 50  0000 C CNN
-	4    1100 6000
+	2    1100 6000
 	0    1    1    0
 $EndComp
@@
 $Comp
 L Rnet4 R104
-U 3 1 5794AC57
+U 4 1 5794AC57
 P 1100 5325
 F 0 "R104" H 1100 5405 50  0000 C CNN
@@
 F 2 "" H 1100 5255 50  0000 C CNN
 F 3 "" V 1100 5325 50  0000 C CNN
-	3    1100 5325
+	4    1100 5325
 	0    1    1    0
 $EndComp
 $Comp
 L Rnet4 R104
-U 4 1 5794B091
+U 3 1 5794B091
 P 1100 6325
 F 0 "R104" H 1100 6405 50  0000 C CNN
@@
 F 2 "" H 1100 6255 50  0000 C CNN
 F 3 "" V 1100 6325 50  0000 C CNN
-	4    1100 6325
-	0    1    1    0
-$EndComp
+	3    1100 6325
+	0    1    1    0
+$EndComp
