File: electronics/Parkbrake/communication_and_debug.sch (KiCad schematic (older format))
At the start: 18 parts, among them P2 JTAG, P3 UART, U26 SN65HVD1050D

Commit message: traceroute finished although there probably is some errors
Connections:
- net USART_RX: now also R92.2; no longer R93.1
- net USART_TX: now also R93.1; no longer R92.2
Changed lines of the file:
@@
 $EndComp
 $Comp
-L GND #PWR086
+L GND #PWR085
 U 1 1 5791E9C0
 P 3125 3550
-F 0 "#PWR086" H 3125 3300 50  0001 C CNN
+F 0 "#PWR085" H 3125 3300 50  0001 C CNN
 F 1 "GND" H 3125 3400 50  0001 C CNN
 F 2 "" H 3125 3550 50  0000 C CNN
@@
 	2700 3600 2450 3600
 $Comp
-L GND #PWR087
+L GND #PWR086
 U 1 1 5791EA76
 P 2450 3600
-F 0 "#PWR087" H 2450 3350 50  0001 C CNN
+F 0 "#PWR086" H 2450 3350 50  0001 C CNN
 F 1 "GND" H 2450 3450 50  0001 C CNN
 F 2 "" H 2450 3600 50  0000 C CNN
@@
 +5V
 $Comp
-L GND #PWR088
+L GND #PWR087
 U 1 1 5791EABC
 P 2400 3975
-F 0 "#PWR088" H 2400 3725 50  0001 C CNN
+F 0 "#PWR087" H 2400 3725 50  0001 C CNN
 F 1 "GND" H 2400 3825 50  0001 C CNN
 F 2 "" H 2400 3975 50  0000 C CNN
@@
 $EndComp
 $Comp
-L GND #PWR089
+L GND #PWR088
 U 1 1 5791EB6A
 P 3425 4575
-F 0 "#PWR089" H 3425 4325 50  0001 C CNN
+F 0 "#PWR088" H 3425 4325 50  0001 C CNN
 F 1 "GND" H 3425 4425 50  0001 C CNN
 F 2 "" H 3425 4575 50  0000 C CNN
@@
 $EndComp
 $Comp
-L GND #PWR090
+L GND #PWR089
 U 1 1 57920F20
 P 7100 2975
-F 0 "#PWR090" H 7100 2725 50  0001 C CNN
+F 0 "#PWR089" H 7100 2725 50  0001 C CNN
 F 1 "GND" H 7100 2825 50  0000 C CNN
 F 2 "" H 7100 2975 50  0000 C CNN
@@
 	1    0    0    -1
 $EndComp
+Text GLabel 7400 2875 2    60   Input ~ 0
+USART_TX
 Text GLabel 7400 2775 2    60   Input ~ 0
-USART_TX
-Text GLabel 7400 2875 2    60   Input ~ 0
 USART_RX
 Text Notes 6575 3375 0    60   ~ 0
@@
 	6475 3425 6475 2425
 $Comp
-L GND #PWR091
+L GND #PWR090
 U 1 1 579225C8
 P 6875 4250
-F 0 "#PWR091" H 6875 4000 50  0001 C CNN
+F 0 "#PWR090" H 6875 4000 50  0001 C CNN
 F 1 "GND" H 6875 4100 50  0001 C CNN
 F 2 "" H 6875 4250 50  0000 C CNN
@@
 $EndComp
 $Comp
-L GND #PWR092
+L GND #PWR091
 U 1 1 579264FD
 P 7875 5250
-F 0 "#PWR092" H 7875 5000 50  0001 C CNN
+F 0 "#PWR091" H 7875 5000 50  0001 C CNN
 F 1 "GND" H 7875 5100 50  0001 C CNN
 F 2 "" H 7875 5250 50  0000 C CNN
