File: electronics/Parkbrake/microcontroller.sch (KiCad schematic (older format))
At the start: 4 parts

Commit message: More work on parkbrake node
Parts:
- removed C?: 100n, symbol C
- removed D?: 3.3V, symbol ZENERsmall
- removed R?: 10k, symbol R
- removed R?: 1k, symbol R
- added C? (x3): 100n, symbol C
- added C?: 4.7u, symbol C
- added C? (x4): 10n, symbol C
- added C? (x4): 1u, symbol C
- added C? (x2): 26p, symbol C
- added C?: 1n, symbol C
- added JP?: Jumper_NO_Small, symbol Jumper_NO_Small
- added R?: 255, symbol R
- added R?: 10k, Resistors_SMD:R_0805, symbol R
- added U?: CAT250_EEPROM, Housings_SSOP:TSSOP-8_4.4x3mm_Pitch0.65mm, symbol CAT250_EEPROM
- added U?: STM32F373RBTx, Housings_QFP:LQFP-64_10x10mm_Pitch0.5mm, symbol STM32F373RBTx
- added Y?: 24Mhz, Crystals:Crystal_HC49-SD_SMD, symbol Crystal
Connections:
- net GND: now also C?.2, C?.2, C?.2, C?.2, C?.2, C?.2, C?.2, C?.2, C?.2, C?.2, C?.2, C?.2, C?.2, C?.2, C?.2, JP?.1, U?.12 (VSSA), U?.31 (VSSSD), U?.4 (GND), U?.63 (VSS)
- new net: C?.1, R?.2, Y?.2
- new net +3.3V: C?.1, C?.1, U?.3 (~WP), U?.7 (~HOLD), U?.8 (Vcc)
- new net 3.3V: C?.1, C?.1, C?.1, C?.1, C?.1, C?.1, C?.1, C?.1, C?.1, C?.1, C?.1, R?.1, U?.13 (VDDA), U?.17 (VREF+), U?.32 (VDDSD), U?.33 (VREFSD+), U?.64 (VDD)
- new net BOOT0: JP?.2, R?.2, U?.60 (BOOT0)
- new net BUTTON_INV_SIG: U?.30 (PE9/DAC1_EXTI9/DAC2_EXTI9/SDADC1_AIN7P/SDADC1_AIN8M/SDADC2_AIN7P/SDADC2_AIN8M)
- new net BUTTON_SIG: U?.29 (PE8/SDADC1_AIN8P/SDADC2_AIN8P)
- new net Bridge_Disable: U?.57 (I2C1_SMBA/I2S1_SD/I2S3_SD/SPI1_MOSI/SPI3_MOSI/TIM16_BKIN/TIM17_CH1/TIM19_ETR/TIM3_CH2/USART2_CK/PB5)
- new net CAN_TX: U?.45 (CAN_TX/COMP2_OUT/I2S1_CK/SPI1_SCK/TIM16_CH1/TIM4_CH2/TIM5_CH3/USART1_DE/USART1_RTS/USB_DP/PA12)
- new net Feed_voltsense: U?.8 (PC0/ADC1_IN10/TIM5_CH1/TIM5_ETR)
- new net IGN_ON_SIG: U?.54 (PD2/TIM3_ETR)
- new net JTCLK: U?.49 (I2C1_SDA/SYS_JTCK-SWCLK/TIM12_CH1/TSC_G4_IO4/PA14)
- new net JTDI: U?.50 (ADC1_EXTI15/I2C1_SCL/I2S1_WS/I2S3_WS/SDADC1_EXTI15/SDADC2_EXTI15/SDADC3_EXTI15/SPI1_NSS/SPI3_NSS/SYS_JTDI/TIM12_CH2/TIM2_CH1/TIM2_ETR/TSC_SYNC/PA15)
- new net JTDO: U?.55 (I2S1_CK/I2S3_CK/SPI1_SCK/SPI3_SCK/SYS_JTDO-TRACESWO/TIM13_CH1/TIM2_CH2/TIM3_ETR/TIM4_ETR/TSC_G5_IO1/USART2_TX/PB3)
- new net JTMS: U?.46 (I2S1_MCK/IR_OUT/SPI1_MISO/SYS_JTMS-SWDIO/TIM16_CH1N/TIM4_CH3/TIM5_CH4/TSC_G4_IO3/USART3_CTS/PA13)
- new net JTNRST: U?.56 (I2S1_MCK/I2S3_MCK/SPI1_MISO/SPI3_MISO/SYS_NJTRST/TIM15_CH1N/TIM16_CH1/TIM17_BKIN/TIM3_CH1/TSC_G5_IO2/USART2_RX/PB4)
- new net LF_speed_in: U?.22 (ADC1_IN6/COMP1_OUT/DAC2_OUT1/I2S1_MCK/SPI1_MISO/TIM13_CH1/TIM16_CH1/TIM3_CH1/TSC_G2_IO3/PA6)
- new net LIGHTS_ON_SIG: U?.36 (PD8/I2S2_CK/SDADC3_AIN6P/SPI2_SCK/TSC_G6_IO3/USART3_TX)
- new net LR_speed_in: U?.20 (ADC1_IN4/DAC1_OUT1/I2S1_WS/I2S3_WS/SPI1_NSS/SPI3_NSS/TIM12_CH1/TIM3_CH2/TSC_G2_IO1/USART2_CK/PA4)
- new net L_speed_out+: U?.61 (CAN_RX/CEC/COMP1_OUT/I2C1_SCL/I2S2_CK/SPI2_SCK/TIM16_CH1/TIM19_CH3/TIM4_CH3/TSC_SYNC/USART3_TX/PB8)
- new net L_speed_out-: U?.62 (CAN_TX/COMP2_OUT/DAC1_EXTI9/DAC2_EXTI9/I2C1_SDA/I2S2_WS/IR_OUT/SPI2_NSS/TIM17_CH1/TIM19_CH4/TIM4_CH4/USART3_RX/PB9)
- new net LeftFront_CS: U?.16 (ADC1_IN2/COMP2_INM/COMP2_OUT/I2S3_MCK/SPI3_MISO/TIM15_CH1/TIM19_CH3/TIM2_CH3/TIM5_CH3/TSC_G1_IO3/USART2_TX/PA2)
- new net LeftFront_DIAG: U?.27 (ADC1_IN9/SDADC1_AIN5P/SDADC1_AIN6M/TIM3_CH4/TSC_G3_IO4/PB1)
- new net LeftFront_Loosen: U?.11 (PC3/ADC1_IN13/I2S2_SD/SPI2_MOSI/TIM5_CH4)
- new net LeftFront_Tighten: U?.10 (PC2/ADC1_IN12/I2S2_MCK/SPI2_MISO/TIM5_CH3)
- new net LeftRear_CS: U?.14 (ADC1_IN0/COMP1_INM/COMP1_OUT/RTC_TAMP2/SYS_WKUP1/TIM19_CH1/TIM2_CH1/TIM2_ETR/TIM5_CH1/TIM5_ETR/TSC_G1_IO1/USART2_CTS/PA0)
- new net LeftRear_DIAG: U?.41 (I2C2_SMBA/I2S2_CK/RCC_MCO/SPI2_SCK/TIM4_ETR/TIM5_CH1/TIM5_ETR/USART1_CK/PA8)
- new net LeftRear_Loosen: U?.52 (PC11/ADC1_EXTI11/I2S3_MCK/SDADC1_EXTI11/SDADC2_EXTI11/SDADC3_EXTI11/SPI3_MISO/TIM19_CH2/USART3_RX)
- new net LeftRear_Tighten: U?.51 (PC10/I2S3_CK/SPI3_SCK/TIM19_CH1/USART3_TX)
- new net NRST: U?.7 (NRST)
- new net OSC_IN: C?.1, U?.5 (PF0/I2C2_SDA/RCC_OSC_IN), Y?.1
- new net OSC_OUT: R?.1, U?.6 (PF1/I2C2_SCL/RCC_OSC_OUT)
- new net PWR_ENABLED_SIG: U?.43 (I2C2_SDA/I2S2_SD/SPI2_MOSI/TIM14_CH1/TIM17_BKIN/TIM2_CH4/TSC_G4_IO2/USART1_RX/PA10)
- new net PWR_voltsense: U?.26 (ADC1_IN8/I2S1_SD/SDADC1_AIN6P/SPI1_MOSI/TIM3_CH2/TIM3_CH3/TSC_G3_IO3/PB0)
- new net RELEASE_CMD_SIG: U?.48 (PF7/I2C2_SDA/USART2_CK)
- new net RF_speed_in: U?.23 (ADC1_IN7/COMP2_OUT/I2S1_SD/SPI1_MOSI/TIM14_CH1/TIM17_CH1/TIM3_CH2/TSC_G2_IO4/PA7)
- new net RR_speed_in: U?.21 (ADC1_IN5/CEC/DAC1_OUT2/I2S1_CK/SPI1_SCK/TIM12_CH2/TIM14_CH1/TIM2_CH1/TIM2_ETR/TSC_G2_IO2/PA5)
- new net R_speed_out+: U?.34 (I2S2_MCK/SDADC3_AIN8P/SPI2_MISO/TIM12_CH1/TIM15_CH1/TSC_G6_IO1/USART3_DE/USART3_RTS/PB14)
- new net R_speed_out-: U?.35 (ADC1_EXTI15/I2S2_SD/RTC_REFIN/SDADC1_EXTI15/SDADC2_EXTI15/SDADC3_AIN7P/SDADC3_AIN8M/SDADC3_EXTI15/SPI2_MOSI/TIM12_CH2/TIM15_CH1N/TIM15_CH2/TSC_G6_IO2/PB15)
- new net RightFront_CS: U?.18 (ADC1_IN3/COMP2_INP/I2S3_SD/SPI3_MOSI/TIM15_CH2/TIM19_CH4/TIM2_CH4/TIM5_CH4/TSC_G1_IO4/USART2_RX/PA3)
- new net RightFront_DIAG: U?.28 (SDADC1_AIN4P/SDADC2_AIN6P/PB2)
- new net RightFront_Loosen: U?.25 (PC5/ADC1_IN15/TSC_G3_IO2/USART1_RX)
- new net RightFront_Tighten: U?.24 (PC4/ADC1_IN14/TIM13_CH1/TSC_G3_IO1/USART1_TX)
- new net RightRear_CS: U?.15 (ADC1_IN1/COMP1_INP/I2S3_CK/RTC_REFIN/SPI3_SCK/TIM15_CH1N/TIM19_CH2/TIM2_CH2/TIM5_CH2/TSC_G1_IO2/USART2_DE/USART2_RTS/PA1)
- new net RightRear_DIAG: U?.42 (DAC1_EXTI9/DAC2_EXTI9/I2C2_SCL/I2S2_MCK/SPI2_MISO/TIM13_CH1/TIM15_BKIN/TIM2_CH3/TSC_G4_IO1/USART1_TX/PA9)
- new net RightRear_Loosen: U?.2 (PC13/RTC_OUT_ALARM/RTC_OUT_CALIB/RTC_TAMP1/RTC_TS/SYS_WKUP2)
- new net RightRear_Tighten: U?.53 (PC12/I2S3_SD/SPI3_MOSI/TIM19_CH3/USART3_CK)
- new net SPI_CS: U?.1 (~CS), U?.37 (PC6/I2S1_WS/SPI1_NSS/TIM3_CH1)
- new net SPI_MISO: U?.2 (MISO), U?.39 (PC8/I2S1_MCK/SPI1_MISO/TIM3_CH3)
- new net SPI_MOSI: U?.40 (PC9/DAC1_EXTI9/DAC2_EXTI9/I2S1_SD/SPI1_MOSI/TIM3_CH4), U?.5 (MOSI)
- new net SPI_SCK: U?.38 (PC7/I2S1_CK/SPI1_SCK/TIM3_CH2), U?.6 (SCK)
- new net TIGHTEN_CMD_SIG: U?.47 (PF6/I2C2_SCL/I2S1_SD/SPI1_MOSI/TIM4_CH4/USART3_DE/USART3_RTS)
- new net USART_RX: U?.59 (I2C1_SDA/TIM15_CH2/TIM17_CH1N/TIM19_CH2/TIM3_CH4/TIM4_CH2/TSC_G5_IO4/USART1_RX/PB7)
- new net USART_TX: U?.58 (I2C1_SCL/TIM15_CH1/TIM16_CH1N/TIM19_CH1/TIM3_CH3/TIM4_CH1/TSC_G5_IO3/USART1_TX/PB6)
- new net VDD_2: U?.19 (VDD)
- new net VR_diag_test: U?.4 (PC15/ADC1_EXTI15/RCC_OSC32_OUT/SDADC1_EXTI15/SDADC2_EXTI15/SDADC3_EXTI15)
- new net ~uC_SET_POWER: U?.3 (PC14/RCC_OSC32_IN)
- no-connect marks 0 -> 1
Other:
- note added: "4.7u near pin 47-48"
- note added: "Boot selection\nBridge for built\nin bootloader"
- note added: "Decoupling"
- note added: "EEPROM"
- note added: "Oscillator"
- note removed: "12V->1.2V \n24V->2.4V\nmax around 30v"

Commit message: ordernr, type and footprints for all components
Parts:
- C? (x2): footprint (none) -> Capacitors_SMD:C_0805; farnell (none) -> 2496940; part (none) -> 0805B104J500CT
- C?: part (none) -> 0805B104J500CT
- C?: footprint (none) -> Capacitors_SMD:c_elec_4x5.3; symbol C -> CP; farnell (none) -> 2068670; part (none) -> EDK475M035A9BAA
- C? (x4): footprint (none) -> Capacitors_SMD:C_0805; farnell (none) -> 2496936; part (none) -> 0805B103J500CT
- C? (x4): footprint (none) -> Capacitors_SMD:C_1206; farnell (none) -> 2362126; part (none) -> GRM31MR71E105JA01L
- C? (x2): footprint (none) -> Capacitors_SMD:C_0805; farnell (none) -> 2497027; part (none) -> 0805N270J500CT
- C?: farnell (none) -> 2494247; part (none) -> GRM2165C1H102JA01D
- R?: footprint (none) -> Resistors_SMD:R_0805; farnell (none) -> 2303484; part (none) -> ERJ6ENF2550V
Connections:
- net INDICATOR_ON: now reaches U?.9 (PC1/ADC1_IN11/TIM5_CH2)
- no-connect marks 1 -> 0
Changed lines of the file:
@@
 F 0 "C?" H 7900 6275 50  0000 L CNN
 F 1 "100n" H 7900 6075 50  0000 L CNN
-F 2 "" H 7913 6025 50  0000 C CNN
+F 2 "Capacitors_SMD:C_0805" H 7913 6025 50  0001 C CNN
 F 3 "" H 7875 6175 50  0000 C CNN
+F 4 "0805B104J500CT" H 7875 6175 60  0001 C CNN "part"
+F 5 "2496940" H 7875 6175 60  0001 C CNN "farnell"
 	1    7875 6175
 	1    0    0    -1
@@
 F 2 "" H 8163 6025 50  0000 C CNN
 F 3 "" H 8125 6175 50  0000 C CNN
+F 4 "0805B104J500CT" H 8125 6175 60  0001 C CNN "part"
 	1    8125 6175
 	1    0    0    -1
 $EndComp
 $Comp
-L C C?
+L CP C?
 U 1 1 579154AB
 P 7600 6175
 F 0 "C?" H 7625 6275 50  0000 L CNN
 F 1 "4.7u" H 7625 6075 50  0000 L CNN
-F 2 "" H 7638 6025 50  0000 C CNN
+F 2 "Capacitors_SMD:c_elec_4x5.3" H 7638 6025 50  0001 C CNN
 F 3 "" H 7600 6175 50  0000 C CNN
+F 4 "EDK475M035A9BAA" H 7600 6175 60  0001 C CNN "part"
+F 5 "2068670" H 7600 6175 60  0001 C CNN "farnell"
 	1    7600 6175
 	1    0    0    -1
@@
 F 0 "C?" H 8700 6275 50  0000 L CNN
 F 1 "10n" H 8700 6075 50  0000 L CNN
-F 2 "" H 8713 6025 50  0000 C CNN
+F 2 "Capacitors_SMD:C_0805" H 8713 6025 50  0001 C CNN
 F 3 "" H 8675 6175 50  0000 C CNN
+F 4 "0805B103J500CT" H 8675 6175 60  0001 C CNN "part"
+F 5 "2496936" H 8675 6175 60  0001 C CNN "farnell"
 	1    8675 6175
 	1    0    0    -1
@@
 F 0 "C?" H 8950 6275 50  0000 L CNN
 F 1 "1u" H 8950 6075 50  0000 L CNN
-F 2 "" H 8963 6025 50  0000 C CNN
+F 2 "Capacitors_SMD:C_1206" H 8963 6025 50  0001 C CNN
 F 3 "" H 8925 6175 50  0000 C CNN
+F 4 "GRM31MR71E105JA01L" H 8925 6175 60  0001 C CNN "part"
+F 5 "2362126" H 8925 6175 60  0001 C CNN "farnell"
 	1    8925 6175
 	1    0    0    -1
@@
 F 0 "C?" H 9475 6275 50  0000 L CNN
 F 1 "10n" H 9475 6075 50  0000 L CNN
-F 2 "" H 9488 6025 50  0000 C CNN
+F 2 "Capacitors_SMD:C_0805" H 9488 6025 50  0001 C CNN
 F 3 "" H 9450 6175 50  0000 C CNN
+F 4 "0805B103J500CT" H 9450 6175 60  0001 C CNN "part"
+F 5 "2496936" H 9450 6175 60  0001 C CNN "farnell"
 	1    9450 6175
 	1    0    0    -1
@@
 F 0 "C?" H 9725 6275 50  0000 L CNN
 F 1 "1u" H 9725 6075 50  0000 L CNN
-F 2 "" H 9738 6025 50  0000 C CNN
+F 2 "Capacitors_SMD:C_1206" H 9738 6025 50  0001 C CNN
 F 3 "" H 9700 6175 50  0000 C CNN
+F 4 "GRM31MR71E105JA01L" H 9700 6175 60  0001 C CNN "part"
+F 5 "2362126" H 9700 6175 60  0001 C CNN "farnell"
 	1    9700 6175
 	1    0    0    -1
@@
 F 0 "C?" H 10750 6275 50  0000 L CNN
 F 1 "10n" H 10750 6075 50  0000 L CNN
-F 2 "" H 10763 6025 50  0000 C CNN
+F 2 "Capacitors_SMD:C_0805" H 10763 6025 50  0001 C CNN
 F 3 "" H 10725 6175 50  0000 C CNN
+F 4 "0805B103J500CT" H 10725 6175 60  0001 C CNN "part"
+F 5 "2496936" H 10725 6175 60  0001 C CNN "farnell"
 	1    10725 6175
 	1    0    0    -1
@@
 F 0 "C?" H 11000 6275 50  0000 L CNN
 F 1 "1u" H 11000 6075 50  0000 L CNN
-F 2 "" H 11013 6025 50  0000 C CNN
+F 2 "Capacitors_SMD:C_1206" H 11013 6025 50  0001 C CNN
 F 3 "" H 10975 6175 50  0000 C CNN
+F 4 "GRM31MR71E105JA01L" H 10975 6175 60  0001 C CNN "part"
+F 5 "2362126" H 10975 6175 60  0001 C CNN "farnell"
 	1    10975 6175
 	1    0    0    -1
@@
 F 0 "C?" H 6025 7475 50  0000 L CNN
 F 1 "26p" H 6025 7275 50  0000 L CNN
-F 2 "" H 6038 7225 50  0000 C CNN
+F 2 "Capacitors_SMD:C_0805" H 6038 7225 50  0001 C CNN
 F 3 "" H 6000 7375 50  0000 C CNN
+F 4 "0805N270J500CT" H 6000 7375 60  0001 C CNN "part"
+F 5 "2497027" H 6000 7375 60  0001 C CNN "farnell"
 	1    6000 7375
 	1    0    0    -1
@@
 F 0 "C?" H 6425 7475 50  0000 L CNN
 F 1 "26p" H 6425 7275 50  0000 L CNN
-F 2 "" H 6438 7225 50  0000 C CNN
+F 2 "Capacitors_SMD:C_0805" H 6438 7225 50  0001 C CNN
 F 3 "" H 6400 7375 50  0000 C CNN
+F 4 "0805N270J500CT" H 6400 7375 60  0001 C CNN "part"
+F 5 "2497027" H 6400 7375 60  0001 C CNN "farnell"
 	1    6400 7375
 	1    0    0    -1
@@
 F 0 "R?" V 6480 6925 50  0000 C CNN
 F 1 "255" V 6400 6925 50  0000 C CNN
-F 2 "" V 6330 6925 50  0000 C CNN
+F 2 "Resistors_SMD:R_0805" V 6330 6925 50  0001 C CNN
 F 3 "" H 6400 6925 50  0000 C CNN
+F 4 "ERJ6ENF2550V" V 6400 6925 60  0001 C CNN "part"
+F 5 "2303484" V 6400 6925 60  0001 C CNN "farnell"
 	1    6400 6925
 	1    0    0    -1
@@
 F 2 "" H 4313 6575 50  0000 C CNN
 F 3 "" H 4275 6725 50  0000 C CNN
+F 4 "GRM2165C1H102JA01D" H 4275 6725 60  0001 C CNN "part"
+F 5 "2494247" H 4275 6725 60  0001 C CNN "farnell"
 	1    4275 6725
 	1    0    0    -1
@@
 F 0 "C?" H 4050 6825 50  0000 L CNN
 F 1 "100n" H 4050 6625 50  0000 L CNN
-F 2 "" H 4063 6575 50  0000 C CNN
+F 2 "Capacitors_SMD:C_0805" H 4063 6575 50  0001 C CNN
 F 3 "" H 4025 6725 50  0000 C CNN
+F 4 "0805B104J500CT" H 4025 6725 60  0001 C CNN "part"
+F 5 "2496940" H 4025 6725 60  0001 C CNN "farnell"
 	1    4025 6725
 	1    0    0    -1
@@
 F 0 "C?" H 10125 6275 50  0000 L CNN
 F 1 "10n" H 10125 6075 50  0000 L CNN
-F 2 "" H 10138 6025 50  0000 C CNN
+F 2 "Capacitors_SMD:C_0805" H 10138 6025 50  0001 C CNN
 F 3 "" H 10100 6175 50  0000 C CNN
+F 4 "0805B103J500CT" H 10100 6175 60  0001 C CNN "part"
+F 5 "2496936" H 10100 6175 60  0001 C CNN "farnell"
 	1    10100 6175
 	1    0    0    -1
@@
 F 0 "C?" H 10375 6275 50  0000 L CNN
 F 1 "1u" H 10375 6075 50  0000 L CNN
-F 2 "" H 10388 6025 50  0000 C CNN
+F 2 "Capacitors_SMD:C_1206" H 10388 6025 50  0001 C CNN
 F 3 "" H 10350 6175 50  0000 C CNN
+F 4 "GRM31MR71E105JA01L" H 10350 6175 60  0001 C CNN "part"
+F 5 "2362126" H 10350 6175 60  0001 C CNN "farnell"
 	1    10350 6175
 	1    0    0    -1
@@
 Wire Wire Line
 	1350 4050 1300 4050
-NoConn ~ 1375 3200
+Text GLabel 1375 3200 0    60   Input ~ 0
+INDICATOR_ON
 $EndSCHEMATC

Commit message: Make it pass DRC rule check
Parts:
- gave numbers to parts that had none: 21
Connections:
- net VDD_2 is gone; now on net +3.3V: U25.19 (VDD)
- net +3.3V: now also C46.1, C47.1, C48.1, C49.1, C50.1, C51.1, C52.1, C53.1, C54.1, C55.1, C56.1, U25.13 (VDDA), U25.17 (VREF+), U25.32 (VDDSD), U25.33 (VREFSD+), U25.64 (VDD)
- net 3.3V: no longer C46.1, C47.1, C48.1, C49.1, C50.1, C51.1, C52.1, C53.1, C54.1, C55.1, C56.1, U25.13 (VDDA), U25.17 (VREF+), U25.32 (VDDSD), U25.33 (VREFSD+), U25.64 (VDD)
- net CAN_RX: now also U25.44 (ADC1_EXTI11/CAN_RX/COMP1_OUT/I2S1_WS/I2S2_WS/SDADC1_EXTI11/SDADC2_EXTI11/SDADC3_EXTI11/SPI1_NSS/SPI2_NSS/TIM4_CH1/TIM5_CH2/USART1_CTS/USB_DM/PA11)
- no-connect marks 0 -> 1
Changed lines of the file:
@@
 $EndDescr
 Text GLabel 7875 5975 1    60   Input ~ 0
-3.3V
-$Comp
-L C C?
++3.3V
+$Comp
+L C C47
 U 1 1 57915417
 P 7875 6175
-F 0 "C?" H 7900 6275 50  0000 L CNN
+F 0 "C47" H 7900 6275 50  0000 L CNN
 F 1 "100n" H 7900 6075 50  0000 L CNN
 F 2 "Capacitors_SMD:C_0805" H 7913 6025 50  0001 C CNN
@@
 $EndComp
 $Comp
-L C C?
+L C C48
 U 1 1 57915474
 P 8125 6175
-F 0 "C?" H 8150 6275 50  0000 L CNN
+F 0 "C48" H 8150 6275 50  0000 L CNN
 F 1 "100n" H 8150 6075 50  0000 L CNN
 F 2 "" H 8163 6025 50  0000 C CNN
@@
 $EndComp
 $Comp
-L CP C?
+L CP C46
 U 1 1 579154AB
 P 7600 6175
-F 0 "C?" H 7625 6275 50  0000 L CNN
+F 0 "C46" H 7625 6275 50  0000 L CNN
 F 1 "4.7u" H 7625 6075 50  0000 L CNN
 F 2 "Capacitors_SMD:c_elec_4x5.3" H 7638 6025 50  0001 C CNN
@@
 $EndComp
 $Comp
-L C C?
+L C C49
 U 1 1 579154E4
 P 8675 6175
-F 0 "C?" H 8700 6275 50  0000 L CNN
+F 0 "C49" H 8700 6275 50  0000 L CNN
 F 1 "10n" H 8700 6075 50  0000 L CNN
 F 2 "Capacitors_SMD:C_0805" H 8713 6025 50  0001 C CNN
@@
 $EndComp
 $Comp
-L GND #PWR?
+L GND #PWR073
 U 1 1 57915825
 P 7875 6325
-F 0 "#PWR?" H 7875 6075 50  0001 C CNN
+F 0 "#PWR073" H 7875 6075 50  0001 C CNN
 F 1 "GND" H 7875 6175 50  0001 C CNN
 F 2 "" H 7875 6325 50  0000 C CNN
@@
 Connection ~ 7600 6025
 $Comp
-L C C?
+L C C50
 U 1 1 57915C80
 P 8925 6175
-F 0 "C?" H 8950 6275 50  0000 L CNN
+F 0 "C50" H 8950 6275 50  0000 L CNN
 F 1 "1u" H 8950 6075 50  0000 L CNN
 F 2 "Capacitors_SMD:C_1206" H 8963 6025 50  0001 C CNN
@@
 $EndComp
 $Comp
-L C C?
+L C C51
 U 1 1 57915CD6
 P 9450 6175
-F 0 "C?" H 9475 6275 50  0000 L CNN
+F 0 "C51" H 9475 6275 50  0000 L CNN
 F 1 "10n" H 9475 6075 50  0000 L CNN
 F 2 "Capacitors_SMD:C_0805" H 9488 6025 50  0001 C CNN
@@
 $EndComp
 $Comp
-L GND #PWR?
+L GND #PWR074
 U 1 1 57915D33
 P 8925 6325
-F 0 "#PWR?" H 8925 6075 50  0001 C CNN
+F 0 "#PWR074" H 8925 6075 50  0001 C CNN
 F 1 "GND" H 8925 6175 50  0001 C CNN
 F 2 "" H 8925 6325 50  0000 C CNN
@@
 	8925 6325 8675 6325
 $Comp
-L C C?
+L C C52
 U 1 1 5791614E
 P 9700 6175
-F 0 "C?" H 9725 6275 50  0000 L CNN
+F 0 "C52" H 9725 6275 50  0000 L CNN
 F 1 "1u" H 9725 6075 50  0000 L CNN
 F 2 "Capacitors_SMD:C_1206" H 9738 6025 50  0001 C CNN
@@
 Wire Wire Line
 	7500 6025 7875 6025
-Text Label 8125 5950 1    60   ~ 0
+Text Label 8125 5975 1    60   ~ 0
 VDD_2
 Wire Wire Line
@@
 VSSSD
 Text GLabel 8925 6025 1    60   Input ~ 0
-3.3V
-$Comp
-L GND #PWR?
++3.3V
+$Comp
+L GND #PWR075
 U 1 1 57918611
 P 9700 6325
-F 0 "#PWR?" H 9700 6075 50  0001 C CNN
+F 0 "#PWR075" H 9700 6075 50  0001 C CNN
 F 1 "GND" H 9700 6175 50  0001 C CNN
 F 2 "" H 9700 6325 50  0000 C CNN
@@
 	9700 6025 9450 6025
 Text GLabel 9700 6025 1    60   Input ~ 0
-3.3V
++3.3V
 Text Label 9450 6025 1    60   ~ 0
 VREFSD+
@@
 VSSSD
 $Comp
-L C C?
+L C C55
 U 1 1 5791910A
 P 10725 6175
-F 0 "C?" H 10750 6275 50  0000 L CNN
+F 0 "C55" H 10750 6275 50  0000 L CNN
 F 1 "10n" H 10750 6075 50  0000 L CNN
 F 2 "Capacitors_SMD:C_0805" H 10763 6025 50  0001 C CNN
@@
 $EndComp
 $Comp
-L C C?
+L C C56
 U 1 1 57919110
 P 10975 6175
-F 0 "C?" H 11000 6275 50  0000 L CNN
+F 0 "C56" H 11000 6275 50  0000 L CNN
 F 1 "1u" H 11000 6075 50  0000 L CNN
 F 2 "Capacitors_SMD:C_1206" H 11013 6025 50  0001 C CNN
@@
 $EndComp
 $Comp
-L GND #PWR?
+L GND #PWR076
 U 1 1 57919116
 P 10975 6325
-F 0 "#PWR?" H 10975 6075 50  0001 C CNN
+F 0 "#PWR076" H 10975 6075 50  0001 C CNN
 F 1 "GND" H 10975 6175 50  0001 C CNN
 F 2 "" H 10975 6325 50  0000 C CNN
@@
 	10975 6025 10725 6025
 Text GLabel 10975 6025 1    60   Input ~ 0
-3.3V
++3.3V
 Text Label 10725 6025 1    60   ~ 0
 VDDA
@@
 VREFSD+
 $Comp
-L C C?
+L C C44
 U 1 1 5791A5CD
 P 6000 7375
-F 0 "C?" H 6025 7475 50  0000 L CNN
+F 0 "C44" H 6025 7475 50  0000 L CNN
 F 1 "26p" H 6025 7275 50  0000 L CNN
 F 2 "Capacitors_SMD:C_0805" H 6038 7225 50  0001 C CNN
@@
 $EndComp
 $Comp
-L C C?
+L C C45
 U 1 1 5791A6BF
 P 6400 7375
-F 0 "C?" H 6425 7475 50  0000 L CNN
+F 0 "C45" H 6425 7475 50  0000 L CNN
 F 1 "26p" H 6425 7275 50  0000 L CNN
 F 2 "Capacitors_SMD:C_0805" H 6438 7225 50  0001 C CNN
@@
 $EndComp
 $Comp
-L GND #PWR?
+L GND #PWR077
 U 1 1 5791A808
 P 6000 7525
-F 0 "#PWR?" H 6000 7275 50  0001 C CNN
+F 0 "#PWR077" H 6000 7275 50  0001 C CNN
 F 1 "GND" H 6000 7375 50  0001 C CNN
 F 2 "" H 6000 7525 50  0000 C CNN
@@
 	6400 7075 6400 7225
 $Comp
-L Crystal Y?
+L Crystal Y1
 U 1 1 5791AC33
 P 6200 7075
-F 0 "Y?" H 6200 7225 50  0000 C CNN
+F 0 "Y1" H 6200 7225 50  0000 C CNN
 F 1 "24Mhz" H 6200 6925 50  0000 C CNN
 F 2 "Crystals:Crystal_HC49-SD_SMD" H 6200 7075 50  0001 C CNN
@@
 $EndComp
 $Comp
-L R R?
+L R R89
 U 1 1 5791AD48
 P 6400 6925
-F 0 "R?" V 6480 6925 50  0000 C CNN
+F 0 "R89" V 6480 6925 50  0000 C CNN
 F 1 "255" V 6400 6925 50  0000 C CNN
 F 2 "Resistors_SMD:R_0805" V 6330 6925 50  0001 C CNN
@@
 OSC_OUT
 $Comp
-L R R?
+L R R88
 U 1 1 5791C2AA
 P 2825 7075
-F 0 "R?" V 2905 7075 50  0000 C CNN
+F 0 "R88" V 2905 7075 50  0000 C CNN
 F 1 "10k" V 2825 7075 50  0000 C CNN
 F 2 "Resistors_SMD:R_0805" V 2755 7075 50  0001 C CNN
@@
 $EndComp
 $Comp
-L Jumper_NO_Small JP?
+L Jumper_NO_Small JP1
 U 1 1 5791C31D
 P 2825 7325
-F 0 "JP?" H 2825 7405 50  0000 C CNN
+F 0 "JP1" H 2825 7405 50  0000 C CNN
 F 1 "Jumper_NO_Small" H 2835 7265 50  0001 C CNN
 F 2 "" H 2825 7325 50  0000 C CNN
@@
 	2900 7225 2825 7225
 $Comp
-L GND #PWR?
+L GND #PWR078
 U 1 1 5791C4BD
 P 2825 7425
-F 0 "#PWR?" H 2825 7175 50  0001 C CNN
+F 0 "#PWR078" H 2825 7175 50  0001 C CNN
 F 1 "GND" H 2825 7275 50  0001 C CNN
 F 2 "" H 2825 7425 50  0000 C CNN
@@
 Text Notes 7125 5700 0    60   ~ 0
 Decoupling
-Text GLabel 10350 3000 2    60   Input ~ 0
+Text GLabel 10375 3000 2    60   Input ~ 0
 CAN_RX
 Text GLabel 10375 3100 2    60   Input ~ 0
@@
 RightRear_DIAG
 $Comp
-L CAT250_EEPROM U?
+L CAT250_EEPROM U24
 U 1 1 579296D6
 P 4675 7200
-F 0 "U?" H 4375 7450 50  0000 L CNN
+F 0 "U24" H 4375 7450 50  0000 L CNN
 F 1 "CAT250_EEPROM" H 4725 7450 50  0000 L CNN
 F 2 "Housings_SSOP:TSSOP-8_4.4x3mm_Pitch0.65mm" H 4325 7150 50  0001 C CNN
@@
 $EndComp
 $Comp
-L C C?
+L C C43
 U 1 1 579298BC
 P 4275 6725
-F 0 "C?" H 4300 6825 50  0000 L CNN
+F 0 "C43" H 4300 6825 50  0000 L CNN
 F 1 "1n" H 4300 6625 50  0000 L CNN
 F 2 "" H 4313 6575 50  0000 C CNN
@@
 $EndComp
 $Comp
-L C C?
+L C C42
 U 1 1 5792991D
 P 4025 6725
-F 0 "C?" H 4050 6825 50  0000 L CNN
+F 0 "C42" H 4050 6825 50  0000 L CNN
 F 1 "100n" H 4050 6625 50  0000 L CNN
 F 2 "Capacitors_SMD:C_0805" H 4063 6575 50  0001 C CNN
@@
 $EndComp
 $Comp
-L GND #PWR?
+L GND #PWR079
 U 1 1 579299FE
 P 4025 6875
-F 0 "#PWR?" H 4025 6625 50  0001 C CNN
+F 0 "#PWR079" H 4025 6625 50  0001 C CNN
 F 1 "GND" H 4025 6725 50  0001 C CNN
 F 2 "" H 4025 6875 50  0000 C CNN
@@
 +3.3V
 $Comp
-L GND #PWR?
+L GND #PWR080
 U 1 1 57929D36
 P 4675 7500
-F 0 "#PWR?" H 4675 7250 50  0001 C CNN
+F 0 "#PWR080" H 4675 7250 50  0001 C CNN
 F 1 "GND" H 4675 7350 50  0001 C CNN
 F 2 "" H 4675 7500 50  0000 C CNN
@@
 RF_speed_in
 $Comp
-L STM32F373RBTx U?
+L STM32F373RBTx U25
 U 1 1 57934AF3
 P 5925 3050
-F 0 "U?" H 1525 5250 50  0000 L BNN
+F 0 "U25" H 1525 5250 50  0000 L BNN
 F 1 "STM32F373RBTx" H 10275 5225 50  0000 R BNN
 F 2 "Housings_QFP:LQFP-64_10x10mm_Pitch0.5mm" H 10275 5175 50  0001 R TNN
@@
 VREF+
 $Comp
-L C C?
+L C C53
 U 1 1 579360EF
 P 10100 6175
-F 0 "C?" H 10125 6275 50  0000 L CNN
+F 0 "C53" H 10125 6275 50  0000 L CNN
 F 1 "10n" H 10125 6075 50  0000 L CNN
 F 2 "Capacitors_SMD:C_0805" H 10138 6025 50  0001 C CNN
@@
 $EndComp
 $Comp
-L C C?
+L C C54
 U 1 1 579360F5
 P 10350 6175
-F 0 "C?" H 10375 6275 50  0000 L CNN
+F 0 "C54" H 10375 6275 50  0000 L CNN
 F 1 "1u" H 10375 6075 50  0000 L CNN
 F 2 "Capacitors_SMD:C_1206" H 10388 6025 50  0001 C CNN
@@
 $EndComp
 $Comp
-L GND #PWR?
+L GND #PWR081
 U 1 1 579360FB
 P 10350 6325
-F 0 "#PWR?" H 10350 6075 50  0001 C CNN
+F 0 "#PWR081" H 10350 6075 50  0001 C CNN
 F 1 "GND" H 10350 6175 50  0001 C CNN
 F 2 "" H 10350 6325 50  0000 C CNN
@@
 	10350 6025 10100 6025
 Text GLabel 10350 6025 1    60   Input ~ 0
-3.3V
++3.3V
 Text Label 10100 6025 1    60   ~ 0
 VREF+
@@
 Text GLabel 1375 3200 0    60   Input ~ 0
 INDICATOR_ON
+NoConn ~ 1375 1600
 $EndSCHEMATC
